File: hardware/mainboard/pcb/v3.1/v3.1.kicad_pcb (KiCad board)
At the start: 2 copper layers, 110 x 167 mm, 159 parts, among them J1 Conn_01x03_Male, J2 Conn_01x03_Male, SW1 RotaryEncoder_Switch, SW2 RotaryEncoder_Switch, SW3 RotaryEncoder_Switch, SW4 RotaryEncoder_Switch, U1 ATtiny1626, U10 touch_but_square, U11 touch_but_square, U12 touch_but_square, U13 touch_but_square, U14 touch_but_square, U15 touch_but_square, U16 touch_but_square, U17 BU4551BF-E2, U18 BU4551BF-E2, U19 touch_but_square, U2 ATtiny1626, U20 touch_but_square, U21 touch_but_square, U22 touch_but_square, U23 touch_but_square, U24 touch_but_square, U25 touch_but_square, U26 touch_but_square, U27 touch_but_round, U28 touch_but_round, U29 touch_but_round, U3 TPIC6C595, U4 TPIC6C595, U5 TPIC6C595, U6 TPIC6C595, U7 TPIC6C595, U8 TPIC6C595, U9 touch_but_square

Commit message: .
Parts:
- removed the C14 at (67.3, 225.7)
- removed the R73 at (-4.35, 188.4)
- removed the R80 at (79.3, 225.7)
- removed SW1, SW2, SW3, SW4: RotaryEncoder_Switch, 3dAudioFoot:PEC11R4230KS0024
- removed U14: touch_but_square, 3dAudioFoot:But_Velo_Rec_1
- removed the U15 at (109.3, 149.2)
- removed the U16 at (109.3, 177.7)
- removed the U17 at (-32.6, 101.6)
- removed the U18 at (-41.4, 101.6)
- added C11: 100nF, Capacitor_SMD:C_1206_3216Metric_Pad1.33x1.80mm_HandSolder, F.Cu at (230.6, 28.4)
- added C19: 100n, Capacitor_SMD:C_1206_3216Metric_Pad1.33x1.80mm_HandSolder, F.Cu at (119.0, 8.30)
- added C20: 100n, Capacitor_SMD:C_1206_3216Metric_Pad1.33x1.80mm_HandSolder, F.Cu at (109.1, 19.4)
- added D17: RGB_led, 3dAudioFoot:LED_QBLP679E-RGB, F.Cu at (59.8, 63.2)
- added D18: RGB_led, 3dAudioFoot:LED_QBLP679E-RGB, F.Cu at (94.8, 63.2)
- added D19: RGB_led, 3dAudioFoot:LED_QBLP679E-RGB, F.Cu at (129.8, 63.2)
- added MT1: PEC11R-4215F-S0024, 3dAudioFoot:XDCR_PEC11R-4215F-S0024, F.Cu at (51.8, 38.2)
- added MT2: PEC11R-4215F-S0024, 3dAudioFoot:XDCR_PEC11R-4215F-S0024, F.Cu at (80.3, 38.2)
- added MT3: PEC11R-4215F-S0024, 3dAudioFoot:XDCR_PEC11R-4215F-S0024, F.Cu at (108.8, 38.2)
- added MT4: PEC11R-4215F-S0024, 3dAudioFoot:XDCR_PEC11R-4215F-S0024, F.Cu at (137.1, 38.2)
- added R100: 10k, Resistor_SMD:R_1206_3216Metric_Pad1.30x1.75mm_HandSolder, F.Cu at (125.0, 4.92)
- added R60: 4K7, Resistor_SMD:R_1206_3216Metric_Pad1.30x1.75mm_HandSolder, F.Cu at (210.4, 51.3)
- added R61: R, Resistor_SMD:R_1206_3216Metric, F.Cu at (236.4, 28.4)
- added R62: R, Resistor_SMD:R_1206_3216Metric, F.Cu at (244.8, 21.8)
- added R63: R, Resistor_SMD:R_1206_3216Metric, F.Cu at (256.1, 21.8)
- added R76: R, Resistor_SMD:R_1206_3216Metric_Pad1.30x1.75mm_HandSolder, B.Cu at (238.9, 123.6)
- added R88: R, Resistor_SMD:R_1206_3216Metric_Pad1.30x1.75mm_HandSolder, B.Cu at (233.0, 123.6)
- added R90: 10k, Resistor_SMD:R_1206_3216Metric_Pad1.30x1.75mm_HandSolder, F.Cu at (125.0, 8.21)
- added R93: 10k, Resistor_SMD:R_1206_3216Metric_Pad1.30x1.75mm_HandSolder, F.Cu at (150.9, -16.2)
- added R94: 10k, Resistor_SMD:R_1206_3216Metric_Pad1.30x1.75mm_HandSolder, F.Cu at (131.0, 1.57)
- added R95: 10k, Resistor_SMD:R_1206_3216Metric_Pad1.30x1.75mm_HandSolder, F.Cu at (131.0, 4.86)
- added R96: 10k, Resistor_SMD:R_1206_3216Metric_Pad1.30x1.75mm_HandSolder, F.Cu at (150.9, -12.9)
- added R97: 10k, Resistor_SMD:R_1206_3216Metric_Pad1.30x1.75mm_HandSolder, F.Cu at (115.0, 19.3)
- added R98: 10k, Resistor_SMD:R_1206_3216Metric_Pad1.30x1.75mm_HandSolder, F.Cu at (119.0, 11.6)
- added R99: 10k, Resistor_SMD:R_1206_3216Metric_Pad1.30x1.75mm_HandSolder, F.Cu at (119.0, 14.9)
- added U10: TPIC6C595, Package_SO:SOIC-16_3.9x9.9mm_P1.27mm, B.Cu at (137.8, 149.2)
- added U11: touch_but_square, 3dAudioFoot:But_Velo_Rec_1, F.Cu at (109.3, 92.2)
- added U12: touch_but_square, 3dAudioFoot:But_Velo_Rec_1, F.Cu at (109.3, 120.7)
- added U27: touch_but_square, 3dAudioFoot:But_Velo_Rec_1, F.Cu at (80.8, 120.7)
- added U28: touch_but_square, 3dAudioFoot:But_Velo_Rec_1, F.Cu at (80.8, 149.2)
- added U29: touch_but_square, 3dAudioFoot:But_Velo_Rec_1, F.Cu at (80.8, 177.7)
- added U30: 74hc4066, Package_SO:SOIC-14_3.9x8.7mm_P1.27mm, B.Cu at (137.0, 135.2)
- added U31: 74hc4066, Package_SO:SOIC-14_3.9x8.7mm_P1.27mm, B.Cu at (80.2, 134.8)
- added U9: TPIC6C595, Package_SO:SOIC-16_3.9x9.9mm_P1.27mm, B.Cu at (137.8, 92.9)
- added locked: touch_but_square, 3dAudioFoot:But_Velo_Rec_1, F.Cu at (109.3, 177.7)
- C1, C2, C3, C4, C5, C6, C7, R25, R26, R27, R74, R75, U1, U2, U3, U4, U5, U6, U7, U8: moved to B.Cu
- C12: value 100n -> 100nF; moved to B.Cu
- C13: renamed from C11; moved to B.Cu
- C14: renamed from C13; moved to B.Cu
- D1, D10, D11, D12, D13, D14, D15, D16, D2, D3, D4, D5, D6, D7, D8, D9: footprint LED_SMD:LED_Avago_PLCC6_3x2.8mm -> 3dAudioFoot:LED_QBLP679E-RGB
- R1, R10, R11, R12, R13, R14, R15, R16, R17, R18, R19, R2, R20, R21, R22, R23, R24, R3, R31, R32, R33, R34, R35, R36, R37, R38, R39, R4, R40, R41, R42, R43, R44, R45, R46, R47, R48, R49, R5, R50, R51, R52, R53, R54, R6, R64, R65, R66, R67, R68, R69, R7, R8, R9: footprint Resistor_SMD:R_1206_3216Metric_Pad1.30x1.75mm_HandSolder -> Resistor_SMD:R_1206_3216Metric
- R101: renamed from R88; moved to B.Cu
- R102: renamed from R89; moved to B.Cu
- R103: renamed from R90; moved to B.Cu
- R28: renamed from R30; moved to B.Cu
- R29: renamed from R28; moved to B.Cu
- R30: renamed from R29; moved to B.Cu
- R57: value 4K7 -> 0R
- R70: value R -> 0R
- R71: value R -> 4K7
- R72: value R -> 4K7; moved to B.Cu
- R73: renamed from R60; moved to B.Cu
- R77, R81, R82, R83, R84, R85, R86, R87: value 10k -> R; moved to B.Cu
- R78: renamed from R61; moved to B.Cu
- R79: renamed from R62; moved to B.Cu
- R80: renamed from R63; moved to B.Cu
- R89: renamed from R76; moved to B.Cu
- R91: renamed from R78; moved to B.Cu
- R92: renamed from R79; moved to B.Cu
- U19, U20: value touch_but_square -> 74hc4066; footprint 3dAudioFoot:But_Velo_Rec_1 -> Package_SO:SOIC-14_3.9x8.7mm_P1.27mm; moved to B.Cu
- U21: value touch_but_square -> 74hc14d; footprint 3dAudioFoot:But_Velo_Rec_1 -> Package_SO:SOIC-14_3.9x8.7mm_P1.27mm; moved to B.Cu
- moved U4 313.3 mm to (52.2, 149.2), turned to 180 degrees
- moved C2 296.8 mm to (86.0, 51.2), turned to 180 degrees
- moved R68 295.6 mm to (244.3, 41.5)
- moved C1 283.3 mm to (92.9, 55.6), turned to 180 degrees
- moved R69 282.9 mm to (227.4, 48.0)
- moved U3 276.1 mm to (51.8, 92.9), turned to 180 degrees
- moved C4 275.5 mm to (95.0, 119.8), turned to 180 degrees
- moved R66 273.7 mm to (230.4, 35.0)
- moved R70 273.1 mm to (210.0, 48.0)
- moved R67 272.3 mm to (233.0, 44.8)
- moved U1 271.8 mm to (95.0, 62.2), turned to 180 degrees
- moved C3 266.0 mm to (97.3, 126.2), turned to 180 degrees
- moved R65 264.4 mm to (215.8, 48.0)
- moved U6 262.6 mm to (80.8, 149.2), turned to 180 degrees
- moved R64 262.4 mm to (221.4, 57.9)
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- renumbered U9 to U15, U10 to U16, U11 to U17, U12 to U18, U27 to U32, U28 to U33, U29 to U34
Connections:
- C12 pad 1: /Encoder/ENCB3 -> VCC
- C12 pad 2: +5V -> GND
- C14 pad 2: EA1 -> GND
- C15 pad 1: EB2 -> /Encoder/ENCB3
- C16 pad 1: /Encoder/ENCB4 -> +5V
- C16 pad 2: +5V -> GND
- C17 pad 1: +5V -> EB2
- C17 pad 2: EA2 -> +5V
- C18 pad 2: /Encoder/ENCA4 -> GND
- R1 pad 1: +5V -> Net-(D1-Pad4)
- R1 pad 2: Net-(D1-Pad6) -> +5V
- R10 pad 1: +5V -> Net-(D4-Pad4)
- R10 pad 2: Net-(D2-Pad5) -> +5V
- R11 pad 1: +5V -> Net-(D4-Pad5)
- R11 pad 2: Net-(D3-Pad5) -> +5V
- R12 pad 1: +5V -> Net-(D4-Pad6)
- R12 pad 2: Net-(D4-Pad5) -> +5V
- R13 pad 1: +5V -> Net-(D5-Pad4)
- R13 pad 2: Net-(D5-Pad5) -> +5V
- R14 pad 1: +5V -> Net-(D5-Pad5)
- R14 pad 2: Net-(D6-Pad5) -> +5V
- R15 pad 1: +5V -> Net-(D5-Pad6)
- R15 pad 2: Net-(D7-Pad5) -> +5V
- R16 pad 1: +5V -> Net-(D6-Pad4)
- R16 pad 2: Net-(D8-Pad5) -> +5V
- R17 pad 1: +5V -> Net-(D6-Pad5)
- R17 pad 2: Net-(D1-Pad4) -> +5V
- R18 pad 1: +5V -> Net-(D6-Pad6)
- R18 pad 2: Net-(D2-Pad4) -> +5V
- R19 pad 1: +5V -> Net-(D7-Pad4)
- R19 pad 2: Net-(D3-Pad4) -> +5V
- R2 pad 1: +5V -> Net-(D1-Pad5)
- R2 pad 2: Net-(D2-Pad6) -> +5V
- R20 pad 1: +5V -> Net-(D7-Pad5)
- R20 pad 2: Net-(D4-Pad4) -> +5V
- R21 pad 1: +5V -> Net-(D7-Pad6)
- R21 pad 2: Net-(D5-Pad4) -> +5V
- R22 pad 1: +5V -> Net-(D8-Pad4)
- R22 pad 2: Net-(D6-Pad4) -> +5V
- R23 pad 1: +5V -> Net-(D8-Pad5)
- R23 pad 2: Net-(D7-Pad4) -> +5V
- R24 pad 1: +5V -> Net-(D8-Pad6)
- R24 pad 2: Net-(D8-Pad4) -> +5V
- R3 pad 1: +5V -> Net-(D1-Pad6)
- R3 pad 2: Net-(D3-Pad6) -> +5V
- R31 pad 1: +5V -> Net-(D9-Pad4)
- R31 pad 2: Net-(D9-Pad6) -> +5V
- R32 pad 1: +5V -> Net-(D9-Pad5)
- R32 pad 2: Net-(D10-Pad6) -> +5V
- R33 pad 1: +5V -> Net-(D9-Pad6)
- R33 pad 2: Net-(D11-Pad6) -> +5V
- R34 pad 1: +5V -> Net-(D10-Pad4)
- R34 pad 2: Net-(D12-Pad6) -> +5V
- R35 pad 1: +5V -> Net-(D10-Pad5)
- R35 pad 2: Net-(D13-Pad6) -> +5V
- R36 pad 1: +5V -> Net-(D10-Pad6)
- R36 pad 2: Net-(D14-Pad6) -> +5V
- R37 pad 1: +5V -> Net-(D11-Pad4)
- R37 pad 2: Net-(D15-Pad6) -> +5V
- R38 pad 1: +5V -> Net-(D11-Pad5)
- R38 pad 2: Net-(D16-Pad6) -> +5V
- R39 pad 1: +5V -> Net-(D11-Pad6)
- R39 pad 2: Net-(D9-Pad5) -> +5V
- R4 pad 1: +5V -> Net-(D2-Pad4)
- R4 pad 2: Net-(D4-Pad6) -> +5V
- R40 pad 1: +5V -> Net-(D12-Pad4)
- R40 pad 2: Net-(D10-Pad5) -> +5V
- R41 pad 1: +5V -> Net-(D12-Pad5)
- R41 pad 2: Net-(D11-Pad5) -> +5V
- R42 pad 1: +5V -> Net-(D12-Pad6)
- R42 pad 2: Net-(D12-Pad5) -> +5V
- R43 pad 1: +5V -> Net-(D13-Pad4)
- R43 pad 2: Net-(D13-Pad5) -> +5V
- R44 pad 1: +5V -> Net-(D13-Pad5)
- R44 pad 2: Net-(D14-Pad5) -> +5V
- R45 pad 1: +5V -> Net-(D13-Pad6)
- R45 pad 2: Net-(D15-Pad5) -> +5V
- R46 pad 1: +5V -> Net-(D14-Pad4)
- R46 pad 2: Net-(D16-Pad5) -> +5V
- R47 pad 1: +5V -> Net-(D14-Pad5)
- R47 pad 2: Net-(D9-Pad4) -> +5V
- R48 pad 1: +5V -> Net-(D14-Pad6)
- R48 pad 2: Net-(D10-Pad4) -> +5V
- R49 pad 1: +5V -> Net-(D15-Pad4)
- R49 pad 2: Net-(D11-Pad4) -> +5V
- R5 pad 1: +5V -> Net-(D2-Pad5)
- R5 pad 2: Net-(D5-Pad6) -> +5V
- R50 pad 1: +5V -> Net-(D15-Pad5)
- R50 pad 2: Net-(D12-Pad4) -> +5V
- R51 pad 1: +5V -> Net-(D15-Pad6)
- R51 pad 2: Net-(D13-Pad4) -> +5V
- R52 pad 1: +5V -> Net-(D16-Pad4)
- R52 pad 2: Net-(D14-Pad4) -> +5V
- R53 pad 1: +5V -> Net-(D16-Pad5)
- R53 pad 2: Net-(D15-Pad4) -> +5V
- R54 pad 1: +5V -> Net-(D16-Pad6)
- R54 pad 2: Net-(D16-Pad4) -> +5V
- R57 pad 2: VCC -> LED_DATA2
- R6 pad 1: +5V -> Net-(D2-Pad6)
- R6 pad 2: Net-(D6-Pad6) -> +5V
- R64 pad 1: +5V -> Net-(D18-Pad4)
- R64 pad 2: Net-(R64-Pad2) -> +5V
- R65 pad 1: +5V -> Net-(D18-Pad5)
- R65 pad 2: Net-(R65-Pad2) -> +5V
- R66 pad 1: +5V -> Net-(D18-Pad6)
- R66 pad 2: Net-(R66-Pad2) -> +5V
- R67 pad 1: +5V -> Net-(D19-Pad4)
- R67 pad 2: Net-(R67-Pad2) -> +5V
- R68 pad 1: +5V -> Net-(D19-Pad5)
- R68 pad 2: Net-(R68-Pad2) -> +5V
- R69 pad 1: +5V -> Net-(D19-Pad6)
- R69 pad 2: Net-(R69-Pad2) -> +5V
- R7 pad 1: +5V -> Net-(D3-Pad4)
- R7 pad 2: Net-(D7-Pad6) -> +5V
- R70 pad 1: +5V -> Net-(R70-Pad1)
- R71 pad 1: +5V -> Net-(R71-Pad1)
- R71 pad 2: Net-(R71-Pad2) -> VCC
- R72 pad 1: +5V -> Net-(R72-Pad1)
- R72 pad 2: Net-(R72-Pad2) -> VCC
- R73 pad 2: Net-(R60-Pad2) -> Net-(R73-Pad2)
- R77 pad 2: /Encoder/ENSC_SW3 -> Net-(R77-Pad2)
- R78 pad 2: Net-(R61-Pad2) -> Net-(R78-Pad2)
- R79 pad 2: Net-(R62-Pad2) -> Net-(R79-Pad2)
- R8 pad 1: +5V -> Net-(D3-Pad5)
- R8 pad 2: Net-(D8-Pad6) -> +5V
- R80 pad 2: Net-(R63-Pad2) -> Net-(R80-Pad2)
- R81 pad 1: /Encoder/ENCB3 -> +5V
- R81 pad 2: +5V -> Net-(R81-Pad2)
- R82 pad 2: ES2 -> Net-(R82-Pad2)
- R83 pad 2: /Encoder/ENSC_SW4 -> Net-(R83-Pad2)
- R84 pad 2: EA2 -> Net-(R84-Pad2)
- R85 pad 1: EB2 -> +5V
- R85 pad 2: +5V -> Net-(R85-Pad2)
- R86 pad 2: /Encoder/ENCA4 -> Net-(R86-Pad2)
- R87 pad 1: /Encoder/ENCB4 -> +5V
- R87 pad 2: +5V -> Net-(R87-Pad2)
- R9 pad 1: +5V -> Net-(D3-Pad6)
- R9 pad 2: Net-(D1-Pad5) -> +5V
- U13 pad 1: Net-(R64-Pad2) -> Net-(R76-Pad2)
- U15 pad 1: Net-(R60-Pad2) -> Net-(R73-Pad2)
- U16 pad 1: Net-(R61-Pad2) -> Net-(R78-Pad2)
- U17 pad 1: Net-(R62-Pad2) -> Net-(R79-Pad2)
- U18 pad 1: Net-(R63-Pad2) -> Net-(R80-Pad2)
- U19 pad 1: Net-(R68-Pad2) -> Net-(R74-Pad2)
- U19 pad 2: GND -> /Button round/BUTCD1
- U20 pad 1: Net-(R69-Pad2) -> Net-(R73-Pad2)
- U20 pad 2: GND -> /Button round/BUTAB1
- U21 pad 1: Net-(R70-Pad2) -> /Button round/BUT_CTL
- U21 pad 2: GND -> BUT_CTL_I
- U22 pad 1: Net-(R71-Pad2) -> Net-(R82-Pad2)
- U23 pad 1: Net-(R72-Pad2) -> Net-(R83-Pad2)
- U24 pad 1: Net-(R73-Pad2) -> Net-(R84-Pad2)
- U25 pad 1: Net-(R74-Pad2) -> Net-(R85-Pad2)
- U26 pad 1: Net-(R75-Pad2) -> Net-(R81-Pad2)
- U32 pad 1: unconnected-(U27-Pad1) -> BR2
- U32 pad 2: unconnected-(U27-Pad2) -> GND
- U33 pad 1: unconnected-(U28-Pad1) -> BR1
- U33 pad 2: unconnected-(U28-Pad2) -> GND
- U34 pad 1: unconnected-(U29-Pad1) -> BR3
- U34 pad 2: unconnected-(U29-Pad2) -> GND
- U6 pad 7: Net-(R57-Pad1) -> Net-(R59-Pad1)
- U7 pad 7: Net-(R59-Pad1) -> Net-(R60-Pad1)
- U8 pad 9: unconnected-(U8-Pad9) -> Net-(R57-Pad1)
Other:
- board size 110 x 167 mm -> 110 x 175 mm
