File: hardware/mainboard/pcb/v3.1/bottom_pcb/button_matrix.kicad_sch (KiCad schematic)
At the start: 37 parts, among them U11 touch_but_square, U12 touch_but_square, U13 touch_but_square, U14 touch_but_square, U15 touch_but_square, U16 touch_but_square, U17 touch_but_square, U18 touch_but_square, U19 74hc4066, U20 74hc4066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

Commit message: top encoder und zechdraw
Parts:
- renumbered R78 to R74, R79 to R75, R80 to R76, R74 to R77, R75 to R78, R76 to R79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
