File: hardware/mainboard/pcb/v3.1/bottom_pcb/button_matrix_round.kicad_sch (KiCad schematic)
At the start: 6 parts, among them U32 touch_but_round, U33 touch_but_round, U34 touch_but_round

Commit message: top encoder und zechdraw
Parts:
- renumbered R101 to R95, R102 to R96, R103 to R97
Changed lines of the file:
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@@
   (symbol (lib_id "Device:R") (at 81.28 100.33 90) (unit 1)
     (in_bom yes) (on_board yes) (fields_autoplaced)
-    (property "Reference" "R103" (id 0) (at 81.28 93.98 90))
+    (property "Reference" "R97" (id 0) (at 81.28 93.98 90))
     (property "Value" "R" (id 1) (at 81.28 96.52 90))
     (property "Footprint" "Resistor_SMD:R_1206_3216Metric_Pad1.30x1.75mm_HandSolder" (id 2) (at 81.28 102.108 90)
@@
   (symbol (lib_id "Device:R") (at 81.28 54.61 90) (unit 1)
     (in_bom yes) (on_board yes) (fields_autoplaced)
-    (property "Reference" "R101" (id 0) (at 81.28 48.26 90))
+    (property "Reference" "R95" (id 0) (at 81.28 48.26 90))
     (property "Value" "R" (id 1) (at 81.28 50.8 90))
     (property "Footprint" "Resistor_SMD:R_1206_3216Metric_Pad1.30x1.75mm_HandSolder" (id 2) (at 81.28 56.388 90)
@@
   (symbol (lib_id "power:GND") (at 113.03 77.47 0) (unit 1)
     (in_bom yes) (on_board yes) (fields_autoplaced)
-    (property "Reference" "#PWR079" (id 0) (at 113.03 83.82 0)
+    (property "Reference" "#PWR070" (id 0) (at 113.03 83.82 0)
       (effects (font (size 1.27 1.27)) hide)
     )
@@
   (symbol (lib_id "power:GND") (at 114.3 100.33 0) (unit 1)
     (in_bom yes) (on_board yes) (fields_autoplaced)
-    (property "Reference" "#PWR081" (id 0) (at 114.3 106.68 0)
+    (property "Reference" "#PWR072" (id 0) (at 114.3 106.68 0)
       (effects (font (size 1.27 1.27)) hide)
     )
@@
   (symbol (lib_id "power:GND") (at 114.3 54.61 0) (unit 1)
     (in_bom yes) (on_board yes) (fields_autoplaced)
-    (property "Reference" "#PWR080" (id 0) (at 114.3 60.96 0)
+    (property "Reference" "#PWR071" (id 0) (at 114.3 60.96 0)
       (effects (font (size 1.27 1.27)) hide)
     )
@@
   (symbol (lib_id "power:+5V") (at 77.47 100.33 0) (unit 1)
     (in_bom yes) (on_board yes) (fields_autoplaced)
-    (property "Reference" "#PWR078" (id 0) (at 77.47 104.14 0)
+    (property "Reference" "#PWR069" (id 0) (at 77.47 104.14 0)
       (effects (font (size 1.27 1.27)) hide)
     )
@@
   (symbol (lib_id "power:+5V") (at 77.47 77.47 0) (unit 1)
     (in_bom yes) (on_board yes) (fields_autoplaced)
-    (property "Reference" "#PWR077" (id 0) (at 77.47 81.28 0)
+    (property "Reference" "#PWR068" (id 0) (at 77.47 81.28 0)
       (effects (font (size 1.27 1.27)) hide)
     )
@@
   (symbol (lib_id "power:+5V") (at 77.47 54.61 0) (unit 1)
     (in_bom yes) (on_board yes) (fields_autoplaced)
-    (property "Reference" "#PWR076" (id 0) (at 77.47 58.42 0)
+    (property "Reference" "#PWR067" (id 0) (at 77.47 58.42 0)
       (effects (font (size 1.27 1.27)) hide)
     )
@@
   (symbol (lib_id "Device:R") (at 81.28 77.47 90) (unit 1)
     (in_bom yes) (on_board yes) (fields_autoplaced)
-    (property "Reference" "R102" (id 0) (at 81.28 71.12 90))
+    (property "Reference" "R96" (id 0) (at 81.28 71.12 90))
     (property "Value" "R" (id 1) (at 81.28 73.66 90))
     (property "Footprint" "Resistor_SMD:R_1206_3216Metric_Pad1.30x1.75mm_HandSolder" (id 2) (at 81.28 79.248 90)
