File: hardware/mainboard/pcb/v3.1/bottom_pcb/led_arr2.kicad_sch (KiCad schematic)
At the start: 107 parts, among them U10 TPIC6C595, U3 TPIC6C595, U4 TPIC6C595, U5 TPIC6C595, U6 TPIC6C595, U7 TPIC6C595, U8 TPIC6C595, U9 TPIC6C595

Commit message: top encoder und zechdraw
Parts:
- gave numbers to parts that had none: 3
- renumbered D17 to D1, D8 to D10, D19 to D11, D9 to D12, D10 to D13, D11 to D14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
Connections:
- net at R68.1: now also D19.5
- net at R69.1: now also D19.6
- no-connect marks 4 -> 8
Other:
- moved on the sheet: R68, R69
