File: hardware/pcbs/bottom_pcb/v3.1.kicad_pcb (KiCad board)
At the start: 2 copper layers, 125.5 x 163 mm, 188 parts, among them J1 Conn_01x03_Male, J2 Conn_01x03_Male, U1 ATtiny1626, U10 TPIC6C595, U11 touch_but_square, U12 touch_but_square, U13 touch_but_square, U15 touch_but_square, U16 touch_but_square, U17 touch_but_square, U18 touch_but_square, U19 74VHC4053AFT, U2 ATtiny1626, U20 74VHC4053AFT, U21 74VHC4053AFT, U22 touch_but_square, U23 touch_but_square, U24 touch_but_square, U25 touch_but_square, U26 touch_but_square, U27 touch_but_square, U28 touch_but_square, U29 touch_but_square, U3 TPIC6C595, U32 touch_but_round, U33 touch_but_round, U34 touch_but_round, U4 TPIC6C595, U5 TPIC6C595, U6 TPIC6C595, U7 TPIC6C595, U8 TPIC6C595, U9 TPIC6C595

Commit message: started placement
Parts:
- added J3: mount_hole, MountingHole:MountingHole_4.3mm_M4_DIN965_Pad, F.Cu at (181.3, 87.2)
- added J4: mount_hole, MountingHole:MountingHole_4.3mm_M4_DIN965_Pad, F.Cu at (181.3, 96.2)
- added J5: mount_hole, MountingHole:MountingHole_4.3mm_M4_DIN965_Pad, F.Cu at (190.3, 87.2)
- added J6: mount_hole, MountingHole:MountingHole_4.3mm_M4_DIN965_Pad, F.Cu at (190.3, 96.2)
- added J7: mount_hole, MountingHole:MountingHole_4.3mm_M4_DIN965_Pad, F.Cu at (199.4, 87.2)
- added J8: mount_hole, MountingHole:MountingHole_4.3mm_M4_DIN965_Pad, F.Cu at (199.4, 96.2)
- C10, C11, C12, C5, C6, C7, C8, C9, R1, R10, R11, R12, R13, R14, R15, R16, R17, R18, R19, R2, R20, R21, R22, R23, R24, R25, R26, R27, R28, R29, R3, R30, R31, R32, R33, R34, R35, R36, R37, R38, R39, R4, R40, R41, R42, R43, R44, R45, R46, R47, R48, R49, R5, R50, R51, R52, R53, R54, R55, R56, R57, R58, R59, R6, R60, R61, R62, R63, R64, R65, R66, R67, R68, R69, R7, R70, R71, R72, R8, R9, U21: moved to B.Cu
- moved R13 196.7 mm to (64.0, 181.0)
- moved C6 192.5 mm to (63.4, 143.0)
- moved R14 191.9 mm to (64.0, 178.0)
- moved R15 187.0 mm to (64.0, 175.0)
- moved R11 178.2 mm to (63.0, 149.0), turned to 180 degrees
- moved R49 175.0 mm to (121.5, 181.6)
- moved R12 173.7 mm to (63.0, 146.0)
- moved R28 170.9 mm to (91.5, 181.6)
- moved R50 169.2 mm to (121.5, 178.3)
- moved C8 166.4 mm to (92.0, 143.0)
- moved R29 165.6 mm to (91.5, 178.3)
- moved C5 164.6 mm to (63.4, 86.0)
- moved R51 163.4 mm to (121.5, 175.0)
- moved R30 160.4 mm to (91.5, 175.0)
- moved R67 159.2 mm to (149.0, 181.0)
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Connections:
- C2 pad 1: +5V -> VCC
- C3 pad 1: +5V -> VCC
- C4 pad 1: +5V -> VCC
- R1 pad 2: +5V -> VCC
- R10 pad 2: +5V -> VCC
- R101 pad 1: +5V -> VCC
- R102 pad 1: +5V -> VCC
- R103 pad 1: +5V -> VCC
- R105 pad 1: +5V -> VCC
- R11 pad 2: +5V -> VCC
- R12 pad 2: +5V -> VCC
- R13 pad 2: +5V -> VCC
- R14 pad 2: +5V -> VCC
- R15 pad 2: +5V -> VCC
- R16 pad 2: +5V -> VCC
- R17 pad 2: +5V -> VCC
- R18 pad 2: +5V -> VCC
- R19 pad 2: +5V -> VCC
- R2 pad 2: +5V -> VCC
- R20 pad 2: +5V -> VCC
- R21 pad 2: +5V -> VCC
- R22 pad 2: +5V -> VCC
- R23 pad 2: +5V -> VCC
- R24 pad 2: +5V -> VCC
- R25 pad 2: +5V -> VCC
- R26 pad 2: +5V -> VCC
- R27 pad 2: +5V -> VCC
- R28 pad 2: +5V -> VCC
- R29 pad 2: +5V -> VCC
- R3 pad 2: +5V -> VCC
- R30 pad 2: +5V -> VCC
- R37 pad 2: +5V -> VCC
- R38 pad 2: +5V -> VCC
- R39 pad 2: +5V -> VCC
- R4 pad 2: +5V -> VCC
- R40 pad 2: +5V -> VCC
- R41 pad 2: +5V -> VCC
- R42 pad 2: +5V -> VCC
- R43 pad 2: +5V -> VCC
- R44 pad 2: +5V -> VCC
- R45 pad 2: +5V -> VCC
- R46 pad 2: +5V -> VCC
- R47 pad 2: +5V -> VCC
- R48 pad 2: +5V -> VCC
- R49 pad 2: +5V -> VCC
- R5 pad 2: +5V -> VCC
- R50 pad 2: +5V -> VCC
- R51 pad 2: +5V -> VCC
- R58 pad 2: +5V -> VCC
- R59 pad 2: +5V -> VCC
- R6 pad 2: +5V -> VCC
- R60 pad 2: +5V -> VCC
- R61 pad 2: +5V -> VCC
- R62 pad 2: +5V -> VCC
- R63 pad 2: +5V -> VCC
- R64 pad 2: +5V -> VCC
- R65 pad 2: +5V -> VCC
- R66 pad 2: +5V -> VCC
- R67 pad 2: +5V -> VCC
- R68 pad 2: +5V -> VCC
- R69 pad 2: +5V -> VCC
- R7 pad 2: +5V -> VCC
- R73 pad 1: +5V -> VCC
- R74 pad 1: +5V -> VCC
- R75 pad 1: +5V -> VCC
- R76 pad 1: +5V -> VCC
- R77 pad 1: +5V -> VCC
- R78 pad 1: +5V -> VCC
- R79 pad 1: +5V -> VCC
- R8 pad 2: +5V -> VCC
- R80 pad 1: +5V -> VCC
- R81 pad 1: +5V -> VCC
- R82 pad 1: +5V -> VCC
- R83 pad 1: +5V -> VCC
- R84 pad 1: +5V -> VCC
- R85 pad 1: +5V -> VCC
- R86 pad 1: +5V -> VCC
- R87 pad 1: +5V -> VCC
- R88 pad 1: +5V -> VCC
- R89 pad 1: +5V -> VCC
- R9 pad 2: +5V -> VCC
- R90 pad 1: +5V -> VCC
- R91 pad 1: +5V -> VCC
- R92 pad 1: +5V -> VCC
- R93 pad 1: +5V -> VCC
- R94 pad 1: +5V -> VCC
- R95 pad 1: +5V -> VCC
- R96 pad 1: +5V -> VCC
- R97 pad 1: +5V -> VCC
- R98 pad 1: +5V -> VCC
- R99 pad 1: +5V -> VCC
- U1 pad 1: +5V -> VCC
- U19 pad 16: +5V -> VCC
- U2 pad 1: +5V -> VCC
- U20 pad 16: +5V -> VCC
- U21 pad 16: +5V -> VCC
- locked pad 1: +5V -> VCC

Commit message: pcb main fertig
Parts:
- added J9: Conn_01x04_Male, Connector_Molex:Molex_KK-254_AE-6410-04A_1x04_P2.54mm_Vertical, F.Cu at (147.4, 60.0)
- added R112: R, Resistor_SMD:R_1206_3216Metric_Pad1.30x1.75mm_HandSolder, B.Cu at (148.4, 65.1)
- added R113: R, Resistor_SMD:R_1206_3216Metric_Pad1.30x1.75mm_HandSolder, B.Cu at (148.1, 68.8)
- added R114: 0R, Resistor_SMD:R_1206_3216Metric_Pad1.30x1.75mm_HandSolder, B.Cu at (47.3, 86.2)
- added R115: 0R, Resistor_SMD:R_1206_3216Metric_Pad1.30x1.75mm_HandSolder, B.Cu at (46.9, 144.1)
- added R116: 0R, Resistor_SMD:R_1206_3216Metric_Pad1.30x1.75mm_HandSolder, B.Cu at (75.8, 86.2)
- added R117: 0R, Resistor_SMD:R_1206_3216Metric_Pad1.30x1.75mm_HandSolder, B.Cu at (104.3, 86.2)
- added R118: 0R, Resistor_SMD:R_1206_3216Metric_Pad1.30x1.75mm_HandSolder, B.Cu at (104.3, 141.7)
- added R119: 0R, Resistor_SMD:R_1206_3216Metric_Pad1.30x1.75mm_HandSolder, B.Cu at (144.0, 100.7)
- added R120: 0R, Resistor_SMD:R_1206_3216Metric_Pad1.30x1.75mm_HandSolder, B.Cu at (132.8, 141.7)
- added R121: 0R, Resistor_SMD:R_1206_3216Metric_Pad1.30x1.75mm_HandSolder, B.Cu at (57.3, 86.2)
- C1: renamed from locked; footprint Capacitor_THT:CP_Radial_D4.0mm_P1.50mm -> Capacitor_SMD:CP_Elec_4x5.3
- C13, C14, C15, C16, C17, C18, C19, C21, R100, R101, R102, R103, R104, R105, R106, R107, R108, R109, R110, R111, R73, R74, R75, R76, R77, R78, R79, R80, R81, R82, R83, R84, R85, R86, R87, R88, R89, R90, R91, R92, R93, R94, R95, R96, R97, R98, R99, U19, U20: moved to B.Cu
- C3: footprint Capacitor_THT:CP_Radial_D4.0mm_P1.50mm -> Capacitor_SMD:CP_Elec_4x5.3
- moved R76 229.6 mm to (63.0, 186.0), turned to 180 degrees
- moved R75 218.5 mm to (58.2, 159.9), turned to 180 degrees
- moved R84 209.1 mm to (91.0, 185.9), turned to 180 degrees
- moved R74 204.1 mm to (58.2, 131.3)
- moved R80 198.5 mm to (121.5, 184.6), turned to -90 degrees
- moved R83 197.8 mm to (86.3, 160.9), turned to 90 degrees
- moved R73 192.0 mm to (58.2, 102.8)
- moved R104 187.5 mm to (47.0, 49.0)
- moved R79 185.9 mm to (114.9, 159.9), turned to 180 degrees
- moved R106 184.4 mm to (56.0, 49.0), turned to 180 degrees
- moved R88 182.6 mm to (148.5, 186.0), turned to 180 degrees
- moved R82 181.8 mm to (86.5, 131.3), turned to 180 degrees
- moved R90 181.5 mm to (47.0, 53.0)
- moved C13 181.5 mm to (41.0, 49.0), turned to 180 degrees
- moved R89 181.0 mm to (48.0, 27.0)
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- renumbered locked to U14
Connections:
- C14 pad 1: /Encoder/ENCA3 -> EA3
- C17 pad 1: /Encoder/ENCB3 -> EB3
- C18 pad 1: /Encoder/ENCA4 -> EA4
- C19 pad 1: /Encoder/ENCB4 -> EB4
- J1 pad 1: UPDI1 -> VCC
- J1 pad 2: UPDI2 -> UPDI1
- J1 pad 3: unconnected-(J1-Pin_3-Pad3) -> GND
- J2 pad 1: SDA -> VCC
- J2 pad 2: SCL -> UPDI2
- J2 pad 3: unconnected-(J2-Pin_3-Pad3) -> GND
- MT3 pad 1: /Encoder/ENSC_SW3 -> ES3
- MT4 pad 1: /Encoder/ENSC_SW4 -> ES4
- R100 pad 1: /Encoder/ENCA3 -> EA3
- R101 pad 2: /Encoder/ENSC_SW4 -> ES4
- R107 pad 1: /Encoder/ENCB3 -> EB3
- R108 pad 1: /Encoder/ENCA4 -> EA4
- R109 pad 1: /Encoder/ENCB4 -> EB4
- R32 pad 1: Net-(U4-SEROUT) -> Net-(U5-SERIN)
- R36 pad 1: Net-(U6-SEROUT) -> Net-(U7-SERIN)
- R55 pad 1: Net-(U8-SEROUT) -> Net-(U9-SERIN)
- R77 pad 2: BUTB1 -> BUTC1
- R78 pad 2: BUTB2 -> BUTC2
- R79 pad 2: BUTB3 -> BUTC3
- R80 pad 2: BUTB4 -> BUTC4
- R81 pad 2: BUTC1 -> BUTB1
- R82 pad 2: BUTC2 -> BUTB2
- R83 pad 2: BUTC3 -> BUTB3
- R84 pad 2: BUTC4 -> BUTB4
- R91 pad 2: /Encoder/ENSC_SW3 -> ES3
- U1 pad 12: BR1 -> unconnected-(U1-PC0/ADC12/SCK2-Pad12)
- U1 pad 13: BR2 -> unconnected-(U1-PC1/ADC13/DO2-Pad13)
- U1 pad 14: BR3 -> ES4
- U1 pad 18: unconnected-(U1-PA2/ADC2/DI1-Pad18) -> ES3
- U1 pad 2: /Encoder/ENCA3 -> BR1
- U1 pad 3: /Encoder/ENCB3 -> EA1
- U1 pad 4: /Encoder/ENSC_SW3 -> EB1
- U1 pad 5: /Encoder/ENCA4 -> ES1
- U1 pad 6: /Encoder/ENCB4 -> EA2
- U1 pad 7: /Encoder/ENSC_SW4 -> EB2
- U1 pad 8: unconnected-(U1-PB3-Pad8) -> ES2
- U1 pad 9: unconnected-(U1-PB2-Pad9) -> BR2
- U10 pad 15: /LED/LED_CLK -> Net-(U10-SRCK)
- U11 pad 1: BUTB1 -> BUTC1
- U12 pad 1: BUTB2 -> BUTC2
- U13 pad 1: BUTB3 -> BUTC3
- U14 pad 1: BUTB4 -> BUTC4
- U19 pad 10: /Button round/BUTAB2 -> BAB2
- U19 pad 11: /Button round/BUTAB1 -> BCD1
- U19 pad 12: BUTA1 -> BUTC1
- U19 pad 13: BUTB1 -> BUTD1
- U19 pad 14: /Button round/BUT_CTL -> BCNT
- U19 pad 15: /Button round/BUT_CTL -> BCNT
- U19 pad 3: BUTB3 -> BUTB1
- U19 pad 4: /Button round/BUT_CTL -> BCNT
- U19 pad 5: BUTA3 -> BUTA1
- U19 pad 9: /Button round/BUTAB3 -> BAB1
- U2 pad 12: /Button round/BUTCD1 -> EA3
- U2 pad 13: /Button round/BUTCD2 -> EB3
- U2 pad 14: /Button round/BUTCD3 -> unconnected-(U2-PC2/ADC14/DI2-Pad14)
- U2 pad 15: /Button round/BUTCD4 -> BCNT
- U2 pad 17: EA2 -> EA4
- U2 pad 18: EB2 -> EB4
- U2 pad 19: ES2 -> BR3
- U2 pad 2: /Button round/BUT_CTL -> BCD4
- U2 pad 3: /Button round/BUTAB1 -> BAB4
- U2 pad 4: /Button round/BUTAB2 -> BCD3
- U2 pad 5: /Button round/BUTAB3 -> BCD2
- U2 pad 6: /Button round/BUTAB4 -> BAB3
- U2 pad 7: EA1 -> BCD1
- U2 pad 8: EB1 -> BAB2
- U2 pad 9: ES1 -> BAB1
- U20 pad 10: /Button round/BUTCD2 -> BCD2
- U20 pad 11: /Button round/BUTCD1 -> BAB3
- U20 pad 12: BUTC1 -> BUTA3
- U20 pad 13: BUTD1 -> BUTB3
- U20 pad 14: /Button round/BUT_CTL -> BCNT
- U20 pad 15: /Button round/BUT_CTL -> BCNT
- U20 pad 4: /Button round/BUT_CTL -> BCNT
- U20 pad 9: /Button round/BUTCD3 -> BCD3
- U21 pad 11: /Button round/BUTCD4 -> BCD4
- U21 pad 14: /Button round/BUT_CTL -> BCNT
- U21 pad 4: /Button round/BUT_CTL -> BCNT
- U21 pad 9: /Button round/BUTAB4 -> BAB4
- U26 pad 1: BUTC1 -> BUTB1
- U27 pad 1: BUTC2 -> BUTB2
- U28 pad 1: BUTC3 -> BUTB3
- U29 pad 1: BUTC4 -> BUTB4
- U3 pad 15: /LED/LED_CLK -> Net-(U3-SRCK)
- U3 pad 2: /LED/LED_DATA -> Net-(U3-SERIN)
- U4 pad 15: /LED/LED_CLK -> Net-(U4-SRCK)
- U4 pad 9: Net-(U4-SEROUT) -> LED_DATAAB
- U5 pad 15: /LED/LED_CLK -> Net-(U5-SRCK)
- U5 pad 2: LED_DATAAB -> Net-(U5-SERIN)
- U6 pad 9: Net-(U6-SEROUT) -> LED_DATABC
- U7 pad 15: /LED/LED_CLK -> Net-(U7-SRCK)
- U7 pad 2: LED_DATABC -> Net-(U7-SERIN)
- U8 pad 15: /LED/LED_CLK -> Net-(U8-SRCK)
- U8 pad 9: Net-(U8-SEROUT) -> LED_DATACD
- U9 pad 15: /LED/LED_CLK -> Net-(U9-SRCK)
- U9 pad 2: LED_DATACD -> Net-(U9-SERIN)
Routing:
- net VCC: track 0.00 -> 1191.9 mm, vias 0 -> 32
- net /LED/LED_UPDATE: track 0.00 -> 353.0 mm, vias 0 -> 14
- net /LED/LED_CLK: track 0.00 -> 351.4 mm, vias 0 -> 11
- net GND: track 0.00 -> 336.5 mm, vias 0 -> 48
- net BCNT: track 0.00 -> 224.6 mm, vias 0 -> 10
- net LED_DATAAB: track 0.00 -> 118.5 mm, vias 0 -> 4
- net LED_DATABC: track 0.00 -> 113.7 mm, vias 0 -> 4
- net BCD4: track 0.00 -> 112.8 mm
- net BAB4: track 0.00 -> 111.6 mm
- net SDA: track 0.00 -> 91.5 mm, vias 0 -> 4
- net BCD3: track 0.00 -> 90.8 mm, vias 0 -> 2
- net BCD2: track 0.00 -> 84.5 mm, vias 0 -> 2
- net ES4: track 0.00 -> 84.4 mm, vias 0 -> 4
- net BAB3: track 0.00 -> 84.1 mm, vias 0 -> 2
- net LED_DATACD: track 0.00 -> 83.7 mm, vias 0 -> 4
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- added copper zone on B.Cu, net GND
- added copper zone on F.Cu, net GND
