File: hardware/pcbs/bottom_pcb/v3.1.kicad_pcb (KiCad board)
At the start: 2 copper layers, 125.5 x 163 mm, 205 parts, among them J1 Conn_01x03_Male, J2 Conn_01x03_Male, J3 mount_hole, J4 mount_hole, J5 mount_hole, J6 mount_hole, J7 mount_hole, J8 mount_hole, J9 Conn_01x04_Male, U1 ATtiny1626, U10 TPIC6C595, U11 touch_but_square, U12 touch_but_square, U13 touch_but_square, U14 touch_but_square, U15 touch_but_square, U16 touch_but_square, U17 touch_but_square, U18 touch_but_square, U19 74VHC4053AFT, U2 ATtiny1626, U20 74VHC4053AFT, U21 74VHC4053AFT, U22 touch_but_square, U23 touch_but_square, U24 touch_but_square, U25 touch_but_square, U26 touch_but_square, U27 touch_but_square, U28 touch_but_square, U29 touch_but_square, U3 TPIC6C595, U32 touch_but_round, U33 touch_but_round, U34 touch_but_round, U4 TPIC6C595, U5 TPIC6C595, U6 TPIC6C595, U7 TPIC6C595, U8 TPIC6C595, U9 TPIC6C595

Commit message: ,,
Parts:
- added J10: Sec Com, Connector_Molex:Molex_KK-254_AE-6410-04A_1x04_P2.54mm_Vertical, B.Cu at (35.2, 60.2)
- added R122: 0R, Resistor_SMD:R_1206_3216Metric_Pad1.30x1.75mm_HandSolder, B.Cu at (75.2, 144.8)
- J1: value Conn_01x03_Male -> Programming Connector; moved to B.Cu
- J2: value Conn_01x03_Male -> Jumper; footprint Connector_Molex:Molex_KK-254_AE-6410-03A_1x03_P2.54mm_Vertical -> Connector_PinHeader_2.54mm:PinHeader_2x03_P2.54mm_Vertical; moved to B.Cu
- J9: value Conn_01x04_Male -> Main Com; moved to B.Cu
- moved J1 113.6 mm to (153.1, 82.5), turned to -90 degrees
- moved R42 25.0 mm to (96.8, 98.2), turned to 180 degrees
- moved R40 23.4 mm to (96.8, 91.9), turned to 180 degrees
- moved R41 23.4 mm to (96.8, 95.1), turned to 180 degrees
- moved R77 23.1 mm to (96.8, 88.8), turned to 0 degrees
- moved R97 8.15 mm to (137.1, 70.4)
- moved R57 8.10 mm to (112.0, 99.6)
- moved R96 7.63 mm to (102.2, 70.5)
- moved J2 6.85 mm to (154.4, 72.2), turned to 180 degrees
- moved J9 5.66 mm to (153.0, 59.0), turned to -90 degrees
- moved R87 4.71 mm to (148.4, 160.2)
- moved R112 4.66 mm to (145.7, 61.3)
- moved R113 4.65 mm to (145.9, 64.7)
- moved C4 4.41 mm to (131.0, 79.7), turned to 90 degrees
- moved R60 3.25 mm to (148.1, 92.1)
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Connections:
- C1 pad 1: VCC -> VCC_UPDI
- C2 pad 1: VCC -> VCC_UPDI
- C3 pad 1: VCC -> VCC_UPDI
- C4 pad 1: VCC -> VCC_UPDI
- J1 pad 1: VCC -> Net-(J1-Pin_1)
- J1 pad 2: UPDI1 -> VCC_UPDI
- J2 pad 1: VCC -> VCC_UPDI
- J2 pad 2: UPDI2 -> VCC
- J2 pad 3: GND -> Net-(J1-Pin_1)
- U1 pad 1: VCC -> VCC_UPDI
- U2 pad 1: VCC -> VCC_UPDI
- U6 pad 15: /LED/LED_CLK -> Net-(U6-SRCK)
Routing:
- net VCC_UPDI: track 0.00 -> 121.6 mm, vias 0 -> 5
- net /LED/LED_CLK: track 351.4 -> 278.7 mm, vias 11 -> 12
- net SCL: track 83.2 -> 152.9 mm, vias 4 -> 5
- net SDA: track 91.5 -> 147.1 mm, vias 4 -> 5
- net VCC: track 1191.9 -> 1162.5 mm, vias 32 -> 40
- net Net-(D12-Pad6): track 7.61 -> 35.6 mm
- net Net-(D12-Pad5): track 6.97 -> 33.6 mm
- net UPDI1: track 49.7 -> 76.3 mm
- net Net-(D12-Pad4): track 7.46 -> 33.0 mm
- net GND: track 336.5 -> 315.9 mm, vias 48 -> 64
- net BUTC1: track 21.6 -> 38.1 mm, vias 1 -> 3
- net Net-(J1-Pin_1): track 0.00 -> 8.32 mm
- net BR3: track 15.7 -> 23.5 mm
- net Net-(U9-SEROUT): track 71.6 -> 65.1 mm, vias 2 -> 0
- net ES4: track 84.4 -> 88.4 mm, vias 4 -> 2
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Other:
- board size 125.5 x 163 mm -> 125 x 163 mm

Commit message: finished top and main PCB
Parts:
- J1: footprint Connector_Molex:Molex_KK-254_AE-6410-03A_1x03_P2.54mm_Vertical -> 3dAudioFoot:Molex_KK-254_AE-6410-03A_1x03_P2.54mm_Vertical
- moved J4 13.0 mm to (39.0, 164.0)
- moved J7 13.0 mm to (39.0, 106.0)
- moved J6 12.0 mm to (152.0, 164.0)
- moved J8 12.0 mm to (152.0, 106.0)
- moved R87 3.11 mm to (145.3, 160.4)
- moved R85 2.14 mm to (148.3, 100.5)
Routing:
- net GND: track 315.9 -> 275.8 mm, vias 64 -> 66
- net Net-(U3-SEROUT): track 51.1 -> 44.0 mm
- net Net-(U4-DRAIN6): track 35.3 -> 30.1 mm, vias 3 -> 1
- net Net-(U9-DRAIN7): track 68.2 -> 64.4 mm
- net Net-(U4-DARIN5): track 35.2 -> 31.9 mm
- net Net-(U4-DRAIN4): track 35.4 -> 32.5 mm, vias 3 -> 1
- net /LED/LED_CLK: track 278.7 -> 276.7 mm
- net BUTD3: track 62.8 -> 61.1 mm
- net Net-(U9-SEROUT): track 65.1 -> 64.1 mm
- net Net-(U3-DRAIN7): track 41.5 -> 40.6 mm
- net VCC: track 1162.5 -> 1163.0 mm, vias 40 -> 39

Commit message: generated gerber files v31
Parts:
- C1, C3: footprint Capacitor_SMD:CP_Elec_4x5.3 -> Capacitor_THT:CP_Radial_D4.0mm_P1.50mm
- C13, C14, C15, C16, C17, C18, C19, C21: value 10nF -> 100nF
- R1, R10, R11, R13, R14, R16, R17, R19, R2, R20, R22, R23, R25, R26, R28, R29, R37, R38, R4, R40, R41, R43, R44, R46, R47, R49, R5, R50, R58, R59, R61, R62, R64, R65, R67, R68, R7, R8: value R -> 220
- R100, R101, R102, R103, R104, R105, R106, R107, R108, R109, R110, R111, R89, R90, R91, R92, R93, R94, R98, R99: value 10k -> 10K; footprint Resistor_SMD:R_1206_3216Metric_Pad1.30x1.75mm_HandSolder -> Resistor_SMD:R_1206_3216Metric
- R112, R113, R73, R74, R75, R76, R77, R78, R79, R80, R81, R82, R83, R84, R85, R86, R87, R88, R95, R96, R97: value R -> 10K; footprint Resistor_SMD:R_1206_3216Metric_Pad1.30x1.75mm_HandSolder -> Resistor_SMD:R_1206_3216Metric
- R114, R115, R116, R117, R118, R119, R120, R121, R122, R31, R32, R33, R34, R35, R36, R52, R53, R54, R55, R56, R57, R70, R71, R72: footprint Resistor_SMD:R_1206_3216Metric_Pad1.30x1.75mm_HandSolder -> Resistor_SMD:R_1206_3216Metric
- R12, R15, R18, R21, R24, R27, R3, R30, R39, R42, R45, R48, R51, R6, R60, R63, R66, R69, R9: value R -> 160
- moved D6 2.05 mm to (95.0, 61.2), turned to 180 degrees
- moved D1 2.05 mm to (59.8, 61.2), turned to 180 degrees
- moved D11 2.05 mm to (129.8, 61.2), turned to 180 degrees
- moved D13 1.87 mm to (109.5, 118.8), turned to 180 degrees
- moved D16 1.87 mm to (138.0, 90.3), turned to 180 degrees
- moved D17 1.87 mm to (138.0, 118.8), turned to 180 degrees
- moved D2 1.87 mm to (52.5, 90.3), turned to 180 degrees
- moved D3 1.87 mm to (52.5, 118.8), turned to 180 degrees
- moved D7 1.87 mm to (81.0, 90.3), turned to 180 degrees
- moved D8 1.87 mm to (81.0, 118.8), turned to 180 degrees
- moved D10 1.87 mm to (81.0, 175.8), turned to 180 degrees
- moved D14 1.87 mm to (109.5, 147.3), turned to 180 degrees
- moved D15 1.87 mm to (109.5, 175.8), turned to 180 degrees
- moved D18 1.87 mm to (138.0, 147.3), turned to 180 degrees
- moved D19 1.87 mm to (138.0, 175.8), turned to 180 degrees
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Routing:
- net Net-(U5-DRAIN4): track 4.41 -> 5.01 mm
- net Net-(U3-DRAIN4): track 4.41 -> 4.97 mm
- net VCC: vias 39 -> 38

Commit message: before ki
Parts:
- removed C10, C11, C12, C7, C8, C9: 100nF, Capacitor_SMD:C_1206_3216Metric_Pad1.33x1.80mm_HandSolder
- removed J10: Sec Com, Connector_Molex:Molex_KK-254_AE-6410-04A_1x04_P2.54mm_Vertical
- removed J6, J7, J8: mount_hole, MountingHole:MountingHole_4.3mm_M4_DIN965_Pad
- removed J9: Main Com, Connector_Molex:Molex_KK-254_AE-6410-04A_1x04_P2.54mm_Vertical
- removed R10, R11, R13, R14, R16, R17, R19, R20, R22, R23, R25, R26, R28, R29, R37, R38, R40, R41, R43, R44, R46, R47, R49, R50, R58, R59, R61, R62, R64, R65, R67, R68: 220, Resistor_SMD:R_1206_3216Metric
- removed R112, R113: 10K, Resistor_SMD:R_1206_3216Metric
- removed R114, R115, R116, R117, R118, R119, R120, R121, R122, R31, R32, R35, R36, R54, R55, R70: 0R, Resistor_SMD:R_1206_3216Metric
- removed R12, R15, R18, R21, R24, R27, R30, R39, R42, R45, R48, R51, R60, R63, R66, R69: 160, Resistor_SMD:R_1206_3216Metric
- removed R33, R34, R52, R53, R56, R57, R71, R72: 4K7, Resistor_SMD:R_1206_3216Metric
- removed U10, U6, U7, U8, U9: TPIC6C595, Package_SO:SOIC-16_3.9x9.9mm_P1.27mm
- removed U19, U20, U21: 74VHC4053AFT, 3dAudioFoot:74vhc4053aft
- added H1: MountingHole, MountingHole:MountingHole_3.2mm_M3, F.Cu at (43.2, -42.3)
- added H2: MountingHole, MountingHole:MountingHole_3.2mm_M3, F.Cu at (43.2, -34.4)
- added H3: MountingHole, MountingHole:MountingHole_3.2mm_M3, F.Cu at (51.2, -42.3)
- added H4: MountingHole, MountingHole:MountingHole_3.2mm_M3, F.Cu at (51.2, -34.4)
- added H5: MountingHole, MountingHole:MountingHole_3.2mm_M3, F.Cu at (59.1, -42.3)
- added H6: MountingHole, MountingHole:MountingHole_3.2mm_M3, F.Cu at (59.1, -34.4)
- added J3: esp32_voltage_shield, Connector_PinHeader_2.54mm:PinHeader_2x04_P2.54mm_Vertical_SMD, F.Cu at (201.8, 62.1)
- added J4: Con_top_pcb, Connector_JST:JST_PH_B9B-PH-K_1x09_P2.00mm_Vertical, F.Cu at (202.5, 55.9)
- added J5: con_rpi, Connector_JST:JST_PH_B9B-PH-K_1x09_P2.00mm_Vertical, F.Cu at (22.3, -1.26)
- added Q1: BSS138, Package_TO_SOT_SMD:SOT-23, F.Cu at (236.2, 68.9)
- C1, C3: value 10uF -> 100nF; footprint Capacitor_THT:CP_Radial_D4.0mm_P1.50mm -> Capacitor_SMD:C_1206_3216Metric_Pad1.33x1.80mm_HandSolder; moved to F.Cu
- C2, C4, C6: moved to F.Cu
- C5: value 100nF -> 10v/1mF; footprint Capacitor_SMD:C_1206_3216Metric_Pad1.33x1.80mm_HandSolder -> Capacitor_SMD:CP_Elec_10x10; moved to F.Cu
- D1, D10, D11, D12, D13, D14, D15, D16, D17, D18, D19, D2, D3, D4, D5, D6, D7, D8, D9: value RGB_led -> WS2812B-2020; footprint 3dAudioFoot:LED_QBLP679E-RGB -> LED_SMD:LED_WS2812B-2020_PLCC4_2.0x2.0mm
- J1: value Programming Connector -> esp_io_shield1; footprint 3dAudioFoot:Molex_KK-254_AE-6410-03A_1x03_P2.54mm_Vertical -> Connector_PinHeader_2.54mm:PinHeader_2x07_P2.54mm_Vertical_SMD; moved to F.Cu
- J2: value Jumper -> esp_io_shield2; footprint Connector_PinHeader_2.54mm:PinHeader_2x03_P2.54mm_Vertical -> Connector_PinHeader_2.54mm:PinHeader_2x11_P2.54mm_Vertical_SMD; moved to F.Cu
- J3: value mount_hole -> esp32_voltage_shield; footprint MountingHole:MountingHole_4.3mm_M4_DIN965_Pad -> Connector_PinHeader_2.54mm:PinHeader_2x04_P2.54mm_Vertical
- J4: value mount_hole -> Con_top_pcb; footprint MountingHole:MountingHole_4.3mm_M4_DIN965_Pad -> Connector_JST:JST_PH_B6B-PH-K_1x06_P2.00mm_Vertical
- J5: value mount_hole -> con_rpi; footprint MountingHole:MountingHole_4.3mm_M4_DIN965_Pad -> Connector_JST:JST_PH_B6B-PH-K_1x06_P2.00mm_Vertical
- R1, R2, R4, R7, R8: value 220 -> 100; footprint Resistor_SMD:R_1206_3216Metric -> Resistor_SMD:R_1206_3216Metric_Pad1.30x1.75mm_HandSolder; moved to F.Cu
- R100, R104, R106, R107, R108, R109, R110, R111: value 10K -> 1k
- R3, R6: value 160 -> 100; footprint Resistor_SMD:R_1206_3216Metric -> Resistor_SMD:R_1206_3216Metric_Pad1.30x1.75mm_HandSolder; moved to F.Cu
- R5: value 220 -> 1k; footprint Resistor_SMD:R_1206_3216Metric -> Resistor_SMD:R_1206_3216Metric_Pad1.30x1.75mm_HandSolder; moved to F.Cu
- R9: value 160 -> 10k; footprint Resistor_SMD:R_1206_3216Metric -> Resistor_SMD:R_1206_3216Metric_Pad1.30x1.75mm_HandSolder; moved to F.Cu
- U1: value ATtiny1626 -> 74HC4051; footprint 3dAudioFoot:attiny1626 -> Package_SO:SOIC-16_3.9x9.9mm_P1.27mm; moved to F.Cu
- U2: value ATtiny1626 -> ~; footprint 3dAudioFoot:attiny1626 -> esp32:DFR0645
- U3, U4: value TPIC6C595 -> 74HC4051; moved to F.Cu
- U5: value TPIC6C595 -> 74AHCT125; footprint Package_SO:SOIC-16_3.9x9.9mm_P1.27mm -> Capacitor_SMD:CP_Elec_10x10; moved to F.Cu
- moved D5 219.3 mm to (223.9, 39.2), turned to 0 degrees
- moved C5 210.6 mm to (258.8, 32.1), turned to 0 degrees
- moved D4 204.6 mm to (223.9, 35.7), turned to 0 degrees
- moved U3 203.6 mm to (253.3, 60.7), turned to 0 degrees
- moved D10 200.9 mm to (228.2, 39.2), turned to 0 degrees
- moved D3 192.2 mm to (223.9, 32.1), turned to 0 degrees
- moved C6 190.3 mm to (230.7, 68.4), turned to 0 degrees
- moved D9 184.9 mm to (228.2, 35.7), turned to 0 degrees
- moved D15 183.9 mm to (232.6, 39.2), turned to 0 degrees
- moved D2 182.3 mm to (223.9, 28.6), turned to 0 degrees
- moved U4 179.6 mm to (210.9, 65.7), turned to 0 degrees
- moved C2 177.6 mm to (243.6, 71.5), turned to 0 degrees
- moved C1 173.6 mm to (243.6, 68.1), turned to 0 degrees
- moved D19 171.6 mm to (236.9, 35.7), turned to 0 degrees
- moved D8 170.9 mm to (228.2, 32.1), turned to 0 degrees
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Connections:
- C1 pad 1: VCC_UPDI -> +3V3
- C2 pad 1: VCC_UPDI -> +3V3
- C3 pad 1: VCC_UPDI -> +3V3
- C4 pad 1: VCC_UPDI -> MUX_D
- C5 pad 1: VCC -> +5V
- C6 pad 1: VCC -> +5V
- D1 pad 1: Net-(U3-DARIN2) -> Net-(D1-DOUT)
- D1 pad 2: Net-(U3-DRAIN1) -> GND
- D1 pad 3: Net-(U3-DRAIN0) -> led_dat
- D1 pad 4: Net-(D1-Pad4) -> +5V
- D10 pad 1: Net-(U6-DRAIN6) -> Net-(D10-DOUT)
- D10 pad 2: Net-(U6-DARIN5) -> GND
- D10 pad 3: Net-(U6-DRAIN4) -> Net-(D10-DIN)
- D10 pad 4: Net-(D10-Pad4) -> +5V
- D11 pad 1: Net-(U7-DARIN2) -> Net-(D11-DOUT)
- D11 pad 2: Net-(U7-DRAIN1) -> GND
- D11 pad 3: Net-(U7-DRAIN0) -> Net-(D10-DOUT)
- D11 pad 4: Net-(D11-Pad4) -> +5V
- D12 pad 1: Net-(U7-DARIN5) -> Net-(D12-DOUT)
- D12 pad 2: Net-(U7-DRAIN4) -> GND
- D12 pad 3: Net-(U7-DRAIN3) -> Net-(D11-DOUT)
- D12 pad 4: Net-(D12-Pad4) -> +5V
- D13 pad 1: Net-(U8-DRAIN0) -> Net-(D13-DOUT)
- D13 pad 2: Net-(U7-DRAIN7) -> GND
- D13 pad 3: Net-(U7-DRAIN6) -> Net-(D12-DOUT)
- D13 pad 4: Net-(D13-Pad4) -> +5V
- D14 pad 1: Net-(U8-DRAIN3) -> Net-(D14-DOUT)
- D14 pad 2: Net-(U8-DARIN2) -> GND
- D14 pad 3: Net-(U8-DRAIN1) -> Net-(D13-DOUT)
- D14 pad 4: Net-(D14-Pad4) -> +5V
- D15 pad 1: Net-(U8-DRAIN6) -> Net-(D15-DOUT)
- D15 pad 2: Net-(U8-DARIN5) -> GND
- D15 pad 3: Net-(U8-DRAIN4) -> Net-(D14-DOUT)
- D15 pad 4: Net-(D15-Pad4) -> +5V
- D16 pad 1: Net-(U9-DARIN2) -> dat2
- D16 pad 2: Net-(U9-DRAIN1) -> GND
- D16 pad 3: Net-(U9-DRAIN0) -> Net-(D15-DOUT)
- D16 pad 4: Net-(D16-Pad4) -> +5V
- D17 pad 1: Net-(U9-DARIN5) -> Net-(D17-DOUT)
- D17 pad 2: Net-(U9-DRAIN4) -> GND
- D17 pad 3: Net-(U9-DRAIN3) -> dat2
- D17 pad 4: Net-(D17-Pad4) -> +5V
- D18 pad 1: Net-(U10-DRAIN0) -> Net-(D18-DOUT)
- D18 pad 2: Net-(U9-DRAIN7) -> GND
- D18 pad 3: Net-(U9-DRAIN6) -> Net-(D17-DOUT)
- D18 pad 4: Net-(D18-Pad4) -> +5V
- D19 pad 1: Net-(U10-DRAIN3) -> unconnected-(D19-DOUT-Pad1)
- D19 pad 2: Net-(U10-DARIN2) -> GND
- D19 pad 3: Net-(U10-DRAIN1) -> Net-(D18-DOUT)
- D19 pad 4: Net-(D19-Pad4) -> +5V
- D2 pad 1: Net-(U3-DARIN5) -> Net-(D2-DOUT)
- D2 pad 2: Net-(U3-DRAIN4) -> GND
- D2 pad 3: Net-(U3-DRAIN3) -> Net-(D1-DOUT)
- D2 pad 4: Net-(D2-Pad4) -> +5V
- D3 pad 1: Net-(U4-DRAIN0) -> Net-(D3-DOUT)
- D3 pad 2: Net-(U3-DRAIN7) -> GND
- D3 pad 3: Net-(U3-DRAIN6) -> Net-(D2-DOUT)
- D3 pad 4: Net-(D3-Pad4) -> +5V
- D4 pad 1: Net-(U4-DRAIN3) -> Net-(D4-DOUT)
- D4 pad 2: Net-(U4-DARIN2) -> GND
- D4 pad 3: Net-(U4-DRAIN1) -> Net-(D3-DOUT)
- D4 pad 4: Net-(D4-Pad4) -> +5V
- D5 pad 1: Net-(U4-DRAIN6) -> Net-(D5-DOUT)
- D5 pad 2: Net-(U4-DARIN5) -> GND
- D5 pad 3: Net-(U4-DRAIN4) -> Net-(D4-DOUT)
- D5 pad 4: Net-(D5-Pad4) -> +5V
- D6 pad 1: Net-(U5-DARIN2) -> Net-(D6-DOUT)
- D6 pad 2: Net-(U5-DRAIN1) -> GND
- D6 pad 3: Net-(U5-DRAIN0) -> Net-(D5-DOUT)
- D6 pad 4: Net-(D6-Pad4) -> +5V
- D7 pad 1: Net-(U5-DARIN5) -> Net-(D7-DOUT)
- D7 pad 2: Net-(U5-DRAIN4) -> GND
- D7 pad 3: Net-(U5-DRAIN3) -> Net-(D6-DOUT)
- D7 pad 4: Net-(D7-Pad4) -> +5V
- D8 pad 1: Net-(U6-DRAIN0) -> dat1
- D8 pad 2: Net-(U5-DRAIN7) -> GND
- D8 pad 3: Net-(U5-DRAIN6) -> Net-(D7-DOUT)
- D8 pad 4: Net-(D8-Pad4) -> +5V
- D9 pad 1: Net-(U6-DRAIN3) -> Net-(D10-DIN)
- D9 pad 2: Net-(U6-DARIN2) -> GND
- D9 pad 3: Net-(U6-DRAIN1) -> dat1
- D9 pad 4: Net-(D9-Pad4) -> +5V
- J1 pad 1: Net-(J1-Pin_1) -> EA1
- J1 pad 2: VCC_UPDI -> EA1
- J1 pad 3: GND -> led_dat
- J2 pad 1: VCC_UPDI -> SCL
- J2 pad 2: VCC -> SCL
- J2 pad 3: Net-(J1-Pin_1) -> SDA
- J2 pad 4: UPDI2 -> SDA
- J2 pad 5: Net-(J1-Pin_1) -> Net-(J2-Pin_5)
- J2 pad 6: UPDI1 -> Net-(J2-Pin_5)
- J3 pad 1: GND -> +5V
- J4 pad 1: GND -> +3V3
- J5 pad 1: GND -> +5V
- R1 pad 1: Net-(D1-Pad4) -> MUX_A
- R1 pad 2: VCC -> Net-(J2-Pin_5)
- R101 pad 1: VCC -> +3V3
- R102 pad 1: VCC -> +3V3
- R103 pad 1: VCC -> +3V3
- R105 pad 1: VCC -> +3V3
- R2 pad 1: Net-(D1-Pad5) -> MUX_B
- R2 pad 2: VCC -> Net-(J2-Pin_7)
- R3 pad 1: Net-(D1-Pad6) -> MUX_C
- R3 pad 2: VCC -> Net-(J2-Pin_10)
- R4 pad 1: Net-(D2-Pad4) -> MUX_D
- R4 pad 2: VCC -> Net-(J2-Pin_11)
- R5 pad 1: Net-(D2-Pad5) -> +5V
- R5 pad 2: VCC -> led_dat
- R6 pad 1: Net-(D2-Pad6) -> Net-(J4-Pin_3)
- R6 pad 2: VCC -> MUX_S0
- R7 pad 1: Net-(D3-Pad4) -> Net-(J4-Pin_4)
- R7 pad 2: VCC -> MUX_S1
- R73 pad 1: VCC -> +3V3
- R74 pad 1: VCC -> +3V3
- R75 pad 1: VCC -> +3V3
- R76 pad 1: VCC -> +3V3
- R77 pad 1: VCC -> +3V3
- R78 pad 1: VCC -> +3V3
- R79 pad 1: VCC -> +3V3
- R8 pad 1: Net-(D3-Pad5) -> Net-(J4-Pin_5)
- R8 pad 2: VCC -> MUX_S2
- R80 pad 1: VCC -> +3V3
- R81 pad 1: VCC -> +3V3
- R82 pad 1: VCC -> +3V3
- R83 pad 1: VCC -> +3V3
- R84 pad 1: VCC -> +3V3
- R85 pad 1: VCC -> +3V3
- R86 pad 1: VCC -> +3V3
- R87 pad 1: VCC -> +3V3
- R88 pad 1: VCC -> +3V3
- R89 pad 1: VCC -> +3V3
- R9 pad 1: Net-(D3-Pad6) -> +3V3
- R9 pad 2: VCC -> led_dat
- R90 pad 1: VCC -> +3V3
- R91 pad 1: VCC -> +3V3
- R92 pad 1: VCC -> +3V3
- R93 pad 1: VCC -> +3V3
- R94 pad 1: VCC -> +3V3
- R95 pad 1: VCC -> +3V3
- R96 pad 1: VCC -> +3V3
- R97 pad 1: VCC -> +3V3
- R98 pad 1: VCC -> +3V3
- R99 pad 1: VCC -> +3V3
- U1 pad 1: VCC_UPDI -> BUTB1
- U1 pad 10: SDA -> MUX_S1
- U1 pad 11: SCL -> MUX_S0
- U1 pad 12: unconnected-(U1-PC0/ADC12/SCK2-Pad12) -> BUTA4
- U1 pad 13: unconnected-(U1-PC1/ADC13/DO2-Pad13) -> BUTA1
- U1 pad 14: ES4 -> BUTA2
- U1 pad 15: /LED/LED_UPDATE -> BUTA3
- U1 pad 16: UPDI1 -> +3V3
- U1 pad 2: BR1 -> BUTB3
- U1 pad 3: EA1 -> MUX_A
- U1 pad 4: EB1 -> BUTB4
- U1 pad 5: ES1 -> BUTB2
- U1 pad 6: EA2 -> GND
- U1 pad 7: EB2 -> GND
- U1 pad 8: ES2 -> GND
- U1 pad 9: BR2 -> MUX_S2
- U2 pad 1: VCC_UPDI -> +3V3
- U2 pad 10: SDA -> unconnected-(U2-21/SDA-Pad10)
- U2 pad 11: SCL -> unconnected-(U2-2/D9-Pad11)
- U2 pad 12: EA3 -> EA2
- U2 pad 13: EB3 -> EB2
- U2 pad 15: BCNT -> EA3
- U2 pad 16: UPDI2 -> EB3
- U2 pad 17: EA4 -> unconnected-(U2-1/TX-Pad17)
- U2 pad 18: EB4 -> unconnected-(U2-3/RX-Pad18)
- U2 pad 19: BR3 -> MUX_S2
- U2 pad 2: BCD4 -> Net-(J3-Pin_5)
- U2 pad 20: GND -> MUX_S1
- U2 pad 3: BAB4 -> unconnected-(U2-NC-Pad3)
- U2 pad 4: BCD3 -> GND
- U2 pad 5: BCD2 -> unconnected-(U2-EN-Pad5)
- U2 pad 6: BAB3 -> EA1
- U2 pad 7: BCD1 -> led_dat
- U2 pad 8: BAB2 -> EB1
- U2 pad 9: BAB1 -> unconnected-(U2-22/SCL-Pad9)
- U3 pad 1: VCC -> BUTD1
- U3 pad 10: /LED/LED_UPDATE -> MUX_S1
- U3 pad 11: Net-(U3-DRAIN4) -> MUX_S0
- U3 pad 12: Net-(U3-DARIN5) -> BUTC4
- U3 pad 13: Net-(U3-DRAIN6) -> BUTC1
- U3 pad 14: Net-(U3-DRAIN7) -> BUTC2
- U3 pad 15: Net-(U3-SRCK) -> BUTC3
- U3 pad 16: GND -> +3V3
- U3 pad 2: Net-(U3-SERIN) -> BUTD3
- U3 pad 3: Net-(U3-DRAIN0) -> MUX_B
- U3 pad 4: Net-(U3-DRAIN1) -> BUTD4
- U3 pad 5: Net-(U3-DARIN2) -> BUTD2
- U3 pad 6: Net-(U3-DRAIN3) -> GND
- U3 pad 7: Net-(U3-~{CLR}) -> GND
- U3 pad 9: Net-(U3-SEROUT) -> MUX_S2
- U4 pad 1: VCC -> ES2
- U4 pad 10: /LED/LED_UPDATE -> MUX_S1
- U4 pad 11: Net-(U4-DRAIN4) -> MUX_S2
- U4 pad 12: Net-(U4-DARIN5) -> ES1
- U4 pad 13: Net-(U4-DRAIN6) -> BR3
- U4 pad 14: unconnected-(U4-DRAIN7-Pad14) -> BR2
- U4 pad 15: Net-(U4-SRCK) -> BR1
- U4 pad 16: GND -> +3V3
- U4 pad 2: Net-(U4-SERIN) -> ES4
- U4 pad 3: Net-(U4-DRAIN0) -> MUX_C
- U4 pad 4: Net-(U4-DRAIN1) -> unconnected-(U4-A7-Pad4)
- U4 pad 5: Net-(U4-DARIN2) -> ES3
- U4 pad 6: Net-(U4-DRAIN3) -> GND
- U4 pad 7: Net-(U4-~{CLR}) -> GND
- U4 pad 9: LED_DATAAB -> MUX_S0
- U5 pad 1: VCC -> GND
- U5 pad 2: Net-(U5-SERIN) -> led_dat
Routing:
- net VCC: track 1163.0 -> 0.00 mm, vias 38 -> 0
- net /LED/LED_UPDATE: track 351.0 -> 0.00 mm, vias 12 -> 0
- net /LED/LED_CLK: track 276.7 -> 0.00 mm, vias 12 -> 0
- net GND: track 275.8 -> 0.00 mm, vias 66 -> 0
- net BCNT: track 223.7 -> 0.00 mm, vias 10 -> 0
- net SCL: track 152.9 -> 0.00 mm, vias 5 -> 0
- net SDA: track 147.1 -> 0.00 mm, vias 5 -> 0
- net VCC_UPDI: track 122.0 -> 0.00 mm, vias 5 -> 0
- net LED_DATAAB: track 119.5 -> 0.00 mm, vias 2 -> 0
- net LED_DATABC: track 113.9 -> 0.00 mm, vias 4 -> 0
- net BCD4: track 111.8 -> 0.00 mm
- net BAB4: track 111.1 -> 0.00 mm
- net BCD3: track 90.7 -> 0.00 mm, vias 2 -> 0
- net ES4: track 88.4 -> 0.00 mm, vias 2 -> 0
- net BCD2: track 84.7 -> 0.00 mm, vias 2 -> 0
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