File: hardware/pcbs/bottom_pcb/v3.1.kicad_sch (KiCad schematic)
At the start: 8 parts, among them J1 Conn_01x03_Male, J2 Conn_01x03_Male, U1 ATtiny1626, U2 ATtiny1626

Commit message: started placement
Parts:
- added J3, J4, J5, J6, J7, J8: mount_hole, MountingHole:MountingHole_4.3mm_M4_DIN965_Pad, symbol Connector:Conn_01x01_Pin
Connections:
- net GND: now also J3.1 (Pin_1), J4.1 (Pin_1), J5.1 (Pin_1), J6.1 (Pin_1), J7.1 (Pin_1), J8.1 (Pin_1)
Changed lines of the file:
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@@
   (junction (at 176.53 43.18) (diameter 0) (color 0 0 0 0)
   )
+  (junction (at 215.9 30.48) (diameter 0) (color 0 0 0 0)
+  )
   (junction (at 172.72 50.8) (diameter 0) (color 0 0 0 0)
   )
   (junction (at 26.67 25.4) (diameter 0) (color 0 0 0 0)
+  )
+  (junction (at 208.28 45.72) (diameter 0) (color 0 0 0 0)
+  )
+  (junction (at 200.66 40.64) (diameter 0) (color 0 0 0 0)
+  )
+  (junction (at 200.66 30.48) (diameter 0) (color 0 0 0 0)
+  )
+  (junction (at 215.9 40.64) (diameter 0) (color 0 0 0 0)
   )
   (junction (at 20.32 25.4) (diameter 0) (color 0 0 0 0)
@@
     (stroke (width 0) (type default))
   )
+  (wire (pts (xy 200.66 40.64) (xy 200.66 45.72))
+    (stroke (width 0) (type default))
+  )
   (wire (pts (xy 203.2 69.85) (xy 217.17 69.85))
     (stroke (width 0) (type default))
@@
     (stroke (width 0) (type default))
   )
+  (wire (pts (xy 208.28 45.72) (xy 215.9 45.72))
+    (stroke (width 0) (type default))
+  )
   (wire (pts (xy 60.96 44.45) (xy 68.58 44.45))
     (stroke (width 0) (type default))
@@
     (stroke (width 0) (type default))
   )
+  (wire (pts (xy 215.9 30.48) (xy 215.9 40.64))
+    (stroke (width 0) (type default))
+  )
   (wire (pts (xy 203.2 67.31) (xy 217.17 67.31))
     (stroke (width 0) (type default))
@@
     (stroke (width 0) (type default))
   )
+  (wire (pts (xy 60.96 101.6) (xy 66.04 101.6))
+    (stroke (width 0) (type default))
+  )
   (wire (pts (xy 59.69 44.45) (xy 59.69 41.91))
     (stroke (width 0) (type default))
@@
     (stroke (width 0) (type default))
   )
+  (wire (pts (xy 200.66 45.72) (xy 208.28 45.72))
+    (stroke (width 0) (type default))
+  )
+  (wire (pts (xy 200.66 30.48) (xy 200.66 40.64))
+    (stroke (width 0) (type default))
+  )
   (wire (pts (xy 53.34 80.01) (xy 64.77 80.01))
     (stroke (width 0) (type default))
@@
     (stroke (width 0) (type default))
   )
+  (wire (pts (xy 208.28 45.72) (xy 208.28 48.26))
+    (stroke (width 0) (type default))
+  )
   (wire (pts (xy 53.34 44.45) (xy 59.69 44.45))
     (stroke (width 0) (type default))
@@
     (stroke (width 0) (type default))
   )
+  (wire (pts (xy 215.9 40.64) (xy 215.9 45.72))
+    (stroke (width 0) (type default))
+  )
   (wire (pts (xy 26.67 25.4) (xy 33.02 25.4))
     (stroke (width 0) (type default))
   )
+  (wire (pts (xy 215.9 20.32) (xy 215.9 30.48))
+    (stroke (width 0) (type default))
+  )
   (wire (pts (xy 53.34 85.09) (xy 64.77 85.09))
     (stroke (width 0) (type default))
   )
+  (wire (pts (xy 200.66 20.32) (xy 200.66 30.48))
+    (stroke (width 0) (type default))
+  )
   (global_label "ES2" (shape input) (at 68.58 34.29 180) (fields_autoplaced)
     (effects (font (size 1.27 1.27)) (justify right))
@@
     )
   )
+  (global_label "VCC" (shape input) (at 66.04 101.6 90) (fields_autoplaced)
+    (effects (font (size 1.27 1.27)) (justify left))
+    (property "Intersheetrefs" "${INTERSHEET_REFS}" (at 66.04 94.9862 90)
+      (effects (font (size 1.27 1.27)) (justify left) hide)
+    )
+  )
   (global_label "SDA" (shape input) (at 53.34 62.23 0) (fields_autoplaced)
     (effects (font (size 1.27 1.27)) (justify left))
@@
     (property "Intersheetrefs" "${INTERSHEET_REFS}" (at 209.1812 102.7906 0)
       (effects (font (size 1.27 1.27)) (justify left) hide)
+    )
+  )
+  (symbol (lib_id "power:GND") (at 208.28 48.26 0) (unit 1)
+    (in_bom yes) (on_board yes) (dnp no) (fields_autoplaced)
+    (property "Reference" "#PWR092" (at 208.28 54.61 0)
+      (effects (font (size 1.27 1.27)) hide)
+    )
+    (property "Value" "GND" (at 208.28 53.34 0)
+      (effects (font (size 1.27 1.27)))
+    )
+    (property "Footprint" "" (at 208.28 48.26 0)
+      (effects (font (size 1.27 1.27)) hide)
+    )
+    (property "Datasheet" "" (at 208.28 48.26 0)
+      (effects (font (size 1.27 1.27)) hide)
+    )
+    (pin "1")
+    (instances
+      (project "v3.1"
+        (path "/1501dcbd-05c1-4298-b373-c91a1b0991c0"
+          (reference "#PWR092") (unit 1)
+        )
+      )
+    )
+  )
+  (symbol (lib_id "Connector:Conn_01x01_Pin") (at 210.82 30.48 0) (unit 1)
+    (in_bom yes) (on_board yes) (dnp no) (fields_autoplaced)
+    (property "Reference" "J7" (at 211.455 25.4 0)
+      (effects (font (size 1.27 1.27)))
+    )
+    (property "Value" "mount_hole" (at 211.455 27.94 0)
+      (effects (font (size 1.27 1.27)))
+    )
+    (property "Footprint" "MountingHole:MountingHole_4.3mm_M4_DIN965_Pad" (at 210.82 30.48 0)
+      (effects (font (size 1.27 1.27)) hide)
+    )
+    (property "Datasheet" "~" (at 210.82 30.48 0)
+      (effects (font (size 1.27 1.27)) hide)
+    )
+    (pin "1")
+    (instances
+      (project "v3.1"
+        (path "/1501dcbd-05c1-4298-b373-c91a1b0991c0"
+          (reference "J7") (unit 1)
+        )
+      )
+    )
+  )
+  (symbol (lib_id "Connector:Conn_01x01_Pin") (at 210.82 40.64 0) (unit 1)
+    (in_bom yes) (on_board yes) (dnp no) (fields_autoplaced)
+    (property "Reference" "J8" (at 211.455 35.56 0)
+      (effects (font (size 1.27 1.27)))
+    )
+    (property "Value" "mount_hole" (at 211.455 38.1 0)
+      (effects (font (size 1.27 1.27)))
+    )
+    (property "Footprint" "MountingHole:MountingHole_4.3mm_M4_DIN965_Pad" (at 210.82 40.64 0)
+      (effects (font (size 1.27 1.27)) hide)
+    )
+    (property "Datasheet" "~" (at 210.82 40.64 0)
+      (effects (font (size 1.27 1.27)) hide)
+    )
+    (pin "1")
+    (instances
+      (project "v3.1"
+        (path "/1501dcbd-05c1-4298-b373-c91a1b0991c0"
+          (reference "J8") (unit 1)
+        )
+      )
     )
   )
@@
     )
   )
+  (symbol (lib_id "Connector:Conn_01x01_Pin") (at 195.58 40.64 0) (unit 1)
+    (in_bom yes) (on_board yes) (dnp no) (fields_autoplaced)
+    (property "Reference" "J5" (at 196.215 35.56 0)
+      (effects (font (size 1.27 1.27)))
+    )
+    (property "Value" "mount_hole" (at 196.215 38.1 0)
+      (effects (font (size 1.27 1.27)))
+    )
+    (property "Footprint" "MountingHole:MountingHole_4.3mm_M4_DIN965_Pad" (at 195.58 40.64 0)
+      (effects (font (size 1.27 1.27)) hide)
+    )
+    (property "Datasheet" "~" (at 195.58 40.64 0)
+      (effects (font (size 1.27 1.27)) hide)
+    )
+    (pin "1")
+    (instances
+      (project "v3.1"
+        (path "/1501dcbd-05c1-4298-b373-c91a1b0991c0"
+          (reference "J5") (unit 1)
+        )
+      )
+    )
+  )
   (symbol (lib_id "power:GND") (at 68.58 121.92 0) (unit 1)
     (in_bom yes) (on_board yes) (dnp no) (fields_autoplaced)
@@
     )
   )
+  (symbol (lib_id "Connector:Conn_01x01_Pin") (at 195.58 30.48 0) (unit 1)
+    (in_bom yes) (on_board yes) (dnp no) (fields_autoplaced)
+    (property "Reference" "J4" (at 196.215 25.4 0)
+      (effects (font (size 1.27 1.27)))
+    )
+    (property "Value" "mount_hole" (at 196.215 27.94 0)
+      (effects (font (size 1.27 1.27)))
+    )
+    (property "Footprint" "MountingHole:MountingHole_4.3mm_M4_DIN965_Pad" (at 195.58 30.48 0)
+      (effects (font (size 1.27 1.27)) hide)
+    )
+    (property "Datasheet" "~" (at 195.58 30.48 0)
+      (effects (font (size 1.27 1.27)) hide)
+    )
+    (pin "1")
+    (instances
+      (project "v3.1"
+        (path "/1501dcbd-05c1-4298-b373-c91a1b0991c0"
+          (reference "J4") (unit 1)
+        )
+      )
+    )
+  )
   (symbol (lib_id "3dAudioSym:C_Polarized") (at 170.18 46.99 0) (unit 1)
     (in_bom yes) (on_board yes) (dnp no)
@@
         (path "/1501dcbd-05c1-4298-b373-c91a1b0991c0"
           (reference "#FLG01") (unit 1)
+        )
+      )
+    )
+  )
+  (symbol (lib_id "Connector:Conn_01x01_Pin") (at 210.82 20.32 0) (unit 1)
+    (in_bom yes) (on_board yes) (dnp no) (fields_autoplaced)
+    (property "Reference" "J6" (at 211.455 15.24 0)
+      (effects (font (size 1.27 1.27)))
+    )
+    (property "Value" "mount_hole" (at 211.455 17.78 0)
+      (effects (font (size 1.27 1.27)))
+    )
+    (property "Footprint" "MountingHole:MountingHole_4.3mm_M4_DIN965_Pad" (at 210.82 20.32 0)
+      (effects (font (size 1.27 1.27)) hide)
+    )
+    (property "Datasheet" "~" (at 210.82 20.32 0)
+      (effects (font (size 1.27 1.27)) hide)
+    )
+    (pin "1")
+    (instances
+      (project "v3.1"
+        (path "/1501dcbd-05c1-4298-b373-c91a1b0991c0"
+          (reference "J6") (unit 1)
         )
       )
@@
         )
       )
+    )
+  )
+  (symbol (lib_id "power:+5V") (at 60.96 101.6 0) (unit 1)
+    (in_bom yes) (on_board yes) (dnp no) (fields_autoplaced)
+    (property "Reference" "#PWR093" (at 60.96 105.41 0)
+      (effects (font (size 1.27 1.27)) hide)
+    )
+    (property "Value" "+5V" (at 60.96 96.52 0)
+      (effects (font (size 1.27 1.27)))
+    )
+    (property "Footprint" "" (at 60.96 101.6 0)
+      (effects (font (size 1.27 1.27)) hide)
+    )
+    (property "Datasheet" "" (at 60.96 101.6 0)
+      (effects (font (size 1.27 1.27)) hide)
+    )
+    (pin "1")
+    (instances
+      (project "v3.1"
+        (path "/1501dcbd-05c1-4298-b373-c91a1b0991c0"
+          (reference "#PWR093") (unit 1)
+        )
+      )
+    )
+  )
+  (symbol (lib_id "Connector:Conn_01x01_Pin") (at 195.58 20.32 0) (unit 1)
+    (in_bom yes) (on_board yes) (dnp no) (fields_autoplaced)
+    (property "Reference" "J3" (at 196.215 15.24 0)
+      (effects (font (size 1.27 1.27)))
+    )
+    (property "Value" "mount_hole" (at 196.215 17.78 0)
+      (effects (font (size 1.27 1.27)))
+    )
+    (property "Footprint" "MountingHole:MountingHole_4.3mm_M4_DIN965_Pad" (at 195.58 20.32 0)
+      (effects (font (size 1.27 1.27)) hide)
+    )
+    (property "Datasheet" "~" (at 195.58 20.32 0)
+      (effects (font (size 1.27 1.27)) hide)
+    )
+    (pin "1")
+    (instances
+      (project "v3.1"
+        (path "/1501dcbd-05c1-4298-b373-c91a1b0991c0"
+          (reference "J3") (unit 1)
+        )
+      )

Commit message: pcb main fertig
Parts:
- added J2: Conn_01x03_Male, Connector_Molex:Molex_KK-254_AE-6410-03A_1x03_P2.54mm_Vertical, symbol Connector:Conn_01x03_Male
- added R112, R113: R, Resistor_SMD:R_1206_3216Metric_Pad1.30x1.75mm_HandSolder, symbol Device:R
- C1, C3: footprint Capacitor_THT:CP_Radial_D4.0mm_P1.50mm -> Capacitor_SMD:CP_Elec_4x5.3
- J9: renamed from J2; value Conn_01x03_Male -> Conn_01x04_Male; footprint Connector_Molex:Molex_KK-254_AE-6410-03A_1x03_P2.54mm_Vertical -> Connector_Molex:Molex_KK-254_AE-6410-04A_1x04_P2.54mm_Vertical; symbol Connector:Conn_01x03_Male -> Connector:Conn_01x04_Pin
Connections:
- net Encoder/ENCA3 is gone; now on net BR1: U1.2 (PA4/ADC4/SS1)
- net Encoder/ENCA4 is gone; now on net ES1: U1.5 (PA7/ADC7)
- net Encoder/ENCB3 is gone; now on net EA1: U1.3 (PA5/ADC5)
- net Encoder/ENCB4 is gone; now on net EA2: U1.6 (PB5/ADC8/CLKOUT)
- net Encoder/ENSC_SW3 is gone; now on net EB1: U1.4 (PA6/ADC6)
- net Encoder/ENSC_SW4 is gone; now on net EB2: U1.7 (PB4/ADC9/RST)
- net +5V: now also J1.1 (Pin_1), J9.1 (Pin_1), J2.1 (Pin_1), R112.1, R113.1
- net BR1: no longer U1.12 (PC0/ADC12/SCK2)
- net BR2: now also U1.9 (PB2); no longer U1.13 (PC1/ADC13/DO2)
- net BR3: now also U2.19 (PA3/ADC3/SCK1); no longer U1.14 (PC2/ADC14/DI2)
- net EA1: no longer U2.7 (PB4/ADC9/RST)
- net EA2: no longer U2.17 (PA1/ADC1/DO1)
- net EB1: no longer U2.8 (PB3)
- net EB2: no longer U2.18 (PA2/ADC2/DI1)
- net ES1: no longer U2.9 (PB2)
- net ES2: now also U1.8 (PB3); no longer U2.19 (PA3/ADC3/SCK1)
- net GND: now also J1.3 (Pin_3), J9.4 (Pin_4), J2.3 (Pin_3)
- net SCL: now also R112.2
- net SDA: now also J9.3 (Pin_3), R113.2; no longer J9.1 (Pin_1)
- net UPDI1: now also J1.2 (Pin_2); no longer J1.1 (Pin_1)
- net UPDI2: now also J2.2 (Pin_2); no longer J1.2 (Pin_2)
- net ES3: now reaches U1.18 (PA2/ADC2/DI1)
- net Button square/BUTAB1 renamed BAB4
- net Button square/BUTAB2 renamed BCD3
- net Button square/BUTAB3 renamed BCD2
- net Button square/BUTAB4 renamed BAB3
- net Button square/BUTCD1 renamed EA3
- net Button square/BUTCD2 renamed EB3
- net Button square/BUTCD3: no longer names the net of U2.14 (PC2/ADC14/DI2)
- net Button square/BUTCD4 renamed BCNT
- net Button square/BUT_CTL renamed BCD4
- new net BAB1: U2.9 (PB2)
- new net BAB2: U2.8 (PB3)
- new net BCD1: U2.7 (PB4/ADC9/RST)
- new net EA4: U2.17 (PA1/ADC1/DO1)
- new net EB4: U2.18 (PA2/ADC2/DI1)
- new net ES4: U1.14 (PC2/ADC14/DI2)
- no-connect marks 5 -> 3
Other:
- sheet Button round renamed Button square
- sheet Untitled Sheet renamed button round

Commit message: ,,
Parts:
- removed J2: Conn_01x03_Male, Connector_Molex:Molex_KK-254_AE-6410-03A_1x03_P2.54mm_Vertical, symbol Connector:Conn_01x03_Male
- added J10: Sec Com, Connector_Molex:Molex_KK-254_AE-6410-04A_1x04_P2.54mm_Vertical, symbol Connector:Conn_01x04_Pin
- added J2: Jumper, Connector_PinHeader_2.54mm:PinHeader_2x03_P2.54mm_Vertical, symbol Connector_Generic:Conn_02x03_Odd_Even
- J1: value Conn_01x03_Male -> Programming Connector
- J9: value Conn_01x04_Male -> Main Com
Connections:
- net +5V: now also J10.1 (Pin_1), J2.2 (Pin_2); no longer C1.1, C2.1, C3.1, C4.1, J1.1 (Pin_1), U1.1 (VCC), U2.1 (VCC)
- net GND: now also J10.4 (Pin_4)
- net SCL: now also J10.2 (Pin_2)
- net SDA: now also J10.3 (Pin_3)
- net UPDI1: now also J2.6 (Pin_6); no longer J1.2 (Pin_2)
- net UPDI2: now also J2.4 (Pin_4)
- new net: J1.1 (Pin_1), J2.3 (Pin_3), J2.5 (Pin_5)
- new net VCC_UPDI: C1.1, C2.1, C3.1, C4.1, J1.2 (Pin_2), J2.1 (Pin_1), U1.1 (VCC), U2.1 (VCC)
Other:
- moved on the sheet: J1, R113

Commit message: finished top and main PCB
Parts:
- J1: footprint Connector_Molex:Molex_KK-254_AE-6410-03A_1x03_P2.54mm_Vertical -> 3dAudioFoot:Molex_KK-254_AE-6410-03A_1x03_P2.54mm_Vertical; symbol Connector:Conn_01x03_Male -> 3dAudioSym:molex1x03
- J10, J9: symbol Connector:Conn_01x04_Pin -> 3dAudioSym:molex1x04
Changed lines of the file:
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@@
 	)
 	(junction
-		(at 80.01 147.32)
+		(at 40.64 154.94)
 		(diameter 0)
 		(color 0 0 0 0)
 	)
 	(junction
-		(at 20.32 25.4)
+		(at 80.01 147.32)
 		(diameter 0)
 		(color 0 0 0 0)
@@
 	(wire
 		(pts
-			(xy 59.69 158.75) (xy 53.34 158.75)
+			(xy 31.75 158.75) (xy 33.02 158.75)
 		)
 		(stroke
@@
 	(wire
 		(pts
-			(xy 58.42 154.94) (xy 53.34 154.94)
+			(xy 59.69 158.75) (xy 53.34 158.75)
 		)
 		(stroke
@@
 	(wire
 		(pts
-			(xy 19.05 25.4) (xy 20.32 25.4)
+			(xy 58.42 154.94) (xy 53.34 154.94)
 		)
 		(stroke
@@
 	(wire
 		(pts
-			(xy 38.1 165.1) (xy 40.64 165.1)
-		)
-		(stroke
-			(width 0)
-			(type default)
-		)
-	)
-	(wire
-		(pts
 			(xy 34.29 158.75) (xy 40.64 158.75)
 		)
@@
 	(wire
 		(pts
-			(xy 33.02 160.02) (xy 38.1 160.02)
+			(xy 176.53 43.18) (xy 182.88 43.18)
 		)
 		(stroke
@@
 	(wire
 		(pts
-			(xy 176.53 43.18) (xy 182.88 43.18)
+			(xy 33.02 25.4) (xy 33.02 34.29)
 		)
 		(stroke
@@
 	(wire
 		(pts
-			(xy 33.02 25.4) (xy 33.02 34.29)
+			(xy 168.91 43.18) (xy 170.18 43.18)
 		)
 		(stroke
@@
 	(wire
 		(pts
-			(xy 168.91 43.18) (xy 170.18 43.18)
+			(xy 33.02 154.94) (xy 40.64 154.94)
 		)
 		(stroke
@@
 	(wire
 		(pts
-			(xy 83.82 176.53) (xy 88.9 176.53)
+			(xy 33.02 158.75) (xy 33.02 154.94)
 		)
 		(stroke
@@
 	(wire
 		(pts
-			(xy 69.85 149.86) (xy 74.93 149.86)
+			(xy 83.82 176.53) (xy 88.9 176.53)
 		)
 		(stroke
@@
 	(wire
 		(pts
-			(xy 31.75 158.75) (xy 33.02 158.75)
+			(xy 69.85 149.86) (xy 74.93 149.86)
 		)
 		(stroke
@@
 	(wire
 		(pts
-			(xy 74.93 149.86) (xy 87.63 149.86)
+			(xy 40.64 154.94) (xy 40.64 156.21)
 		)
 		(stroke
@@
 	(wire
 		(pts
-			(xy 200.66 45.72) (xy 208.28 45.72)
+			(xy 74.93 149.86) (xy 87.63 149.86)
 		)
 		(stroke
@@
 	(wire
 		(pts
-			(xy 200.66 30.48) (xy 200.66 40.64)
+			(xy 200.66 45.72) (xy 208.28 45.72)
 		)
 		(stroke
@@
 	(wire
 		(pts
-			(xy 53.34 80.01) (xy 72.39 80.01)
+			(xy 200.66 30.48) (xy 200.66 40.64)
 		)
 		(stroke
@@
 	(wire
 		(pts
-			(xy 53.34 74.93) (xy 72.39 74.93)
+			(xy 53.34 80.01) (xy 72.39 80.01)
 		)
 		(stroke
@@
 	(wire
 		(pts
-			(xy 40.64 152.4) (xy 40.64 156.21)
+			(xy 53.34 74.93) (xy 72.39 74.93)
 		)
 		(stroke
@@
 	(wire
 		(pts
-			(xy 38.1 160.02) (xy 38.1 165.1)
+			(xy 40.64 152.4) (xy 40.64 154.94)
 		)
 		(stroke
@@
 	(wire
 		(pts
-			(xy 33.02 158.75) (xy 33.02 160.02)
+			(xy 80.01 137.16) (xy 80.01 139.7)
 		)
 		(stroke
@@
 	(wire
 		(pts
-			(xy 80.01 137.16) (xy 80.01 139.7)
+			(xy 83.82 173.99) (xy 88.9 173.99)
 		)
 		(stroke
@@
 	(wire
 		(pts
-			(xy 83.82 173.99) (xy 88.9 173.99)
+			(xy 27.94 133.35) (xy 31.75 133.35)
 		)
 		(stroke
@@
 	(global_label "VCC_UPDI"
 		(shape input)
-		(at 19.05 25.4 90)
+		(at 22.86 25.4 90)
 		(fields_autoplaced yes)
 		(effects
@@
 		)
 		(property "Intersheetrefs" "${INTERSHEET_REFS}"
-			(at 19.05 13.3433 90)
+			(at 22.86 13.3433 90)
 			(effects
 				(font
@@
 		)
 	)
+	(global_label "VCC_UPDI"
+		(shape input)
+		(at 27.94 133.35 180)
+		(fields_autoplaced yes)
+		(effects
+			(font
+				(size 1.27 1.27)
+			)
+			(justify right)
+		)
+		(property "Intersheetrefs" "${INTERSHEET_REFS}"
+			(at 15.8833 133.35 0)
+			(effects
+				(font
+					(size 1.27 1.27)
+				)
+				(justify right)
+				(hide yes)
+			)
+		)
+	)
 	(global_label "BAB2"
 		(shape input)
@@
 		)
 	)
-	(global_label "VCC_UPDI"
-		(shape input)
-		(at 40.64 165.1 0)
-		(fields_autoplaced yes)
-		(effects
-			(font
-				(size 1.27 1.27)
-			)
-			(justify left)
-		)
-		(property "Intersheetrefs" "${INTERSHEET_REFS}"
-			(at 52.6967 165.1 0)
-			(effects
-				(font
-					(size 1.27 1.27)
-				)
-				(justify left)
-				(hide yes)
-			)
-		)
-	)
 	(global_label "SDA"
 		(shape input)
@@
 	)
 	(symbol
-		(lib_id "Connector:Conn_01x03_Male")
+		(lib_id "3dAudioSym:molex1x03")
 		(at 26.67 158.75 0)
+		(mirror y)
 		(unit 1)
 		(exclude_from_sim no)
@@
 		(dnp no)
 		(property "Reference" "J1"
-			(at 25.146 155.702 0)
+			(at 24.13 151.638 0)
 			(effects
 				(font
@@
 		)
 		(property "Value" "Programming Connector"
-			(at 38.608 168.656 0)
+			(at 14.732 168.656 0)
 			(effects
 				(font
@@
 			)
 		)
-		(property "Footprint" "Connector_Molex:Molex_KK-254_AE-6410-03A_1x03_P2.54mm_Vertical"
+		(property "Footprint" "3dAudioFoot:Molex_KK-254_AE-6410-03A_1x03_P2.54mm_Vertical"
 			(at 26.67 158.75 0)
 			(effects
@@
 			)
 		)
-		(property "Description" ""
+		(property "Description" "Generic connector, single row, 01x03, script generated (kicad-library-utils/schlib/autogen/connector/)"
 			(at 26.67 158.75 0)
 			(effects
@@
 	)
 	(symbol
-		(lib_id "Connector:Conn_01x04_Pin")
+		(lib_id "3dAudioSym:molex1x04")
 		(at 92.71 147.32 0)
-		(mirror y)
 		(unit 1)
 		(exclude_from_sim no)
@@
 		(dnp no)
 		(property "Reference" "J9"
-			(at 91.44 139.7 0)
+			(at 93.98 139.7 0)
 			(effects
 				(font
@@
 		)
 		(property "Value" "Main Com"
-			(at 87.63 156.21 0)
+			(at 97.79 156.21 0)
 			(effects
 				(font
@@
 			)
 		)
-		(property "Description" ""
+		(property "Description" "Generic connector, single row, 01x04, script generated (kicad-library-utils/schlib/autogen/connector/)"
 			(at 92.71 147.32 0)
 			(effects
@@
 	)
 	(symbol
-		(lib_id "Connector:Conn_01x04_Pin")
+		(lib_id "3dAudioSym:molex1x04")
 		(at 93.98 171.45 0)
-		(mirror y)
 		(unit 1)
 		(exclude_from_sim no)
@@
 		(dnp no)
 		(property "Reference" "J10"
-			(at 92.71 163.83 0)
+			(at 95.25 163.83 0)
 			(effects
 				(font
@@
 		)
 		(property "Value" "Sec Com"
-			(at 88.9 180.34 0)
+			(at 99.06 180.34 0)
 			(effects
 				(font
@@
 			)
 		)
-		(property "Description" ""
+		(property "Description" "Generic connector, single row, 01x04, script generated (kicad-library-utils/schlib/autogen/connector/)"
 			(at 93.98 171.45 0)
 			(effects
@@
 					(unit 1)
 				)
+			)
+		)
+	)
+	(symbol
+		(lib_id "power:PWR_FLAG")
+		(at 31.75 133.35 0)
+		(unit 1)
+		(exclude_from_sim no)
+		(in_bom yes)
+		(on_board yes)
+		(dnp no)
+		(fields_autoplaced yes)
+		(property "Reference" "#FLG03"
+			(at 31.75 131.445 0)
+			(effects
+				(font
+					(size 1.27 1.27)
+				)
+				(hide yes)
+			)
+		)
+		(property "Value" "PWR_FLAG"
+			(at 31.75 128.27 0)
+			(effects
+				(font
+					(size 1.27 1.27)
+				)
+			)
+		)
+		(property "Footprint" ""
+			(at 31.75 133.35 0)
+			(effects
+				(font
+					(size 1.27 1.27)
+				)
+				(hide yes)
+			)
+		)
+		(property "Datasheet" "~"
+			(at 31.75 133.35 0)
+			(effects
+				(font
+					(size 1.27 1.27)
+				)
+				(hide yes)
+			)
+		)
+		(property "Description" ""
+			(at 31.75 133.35 0)
+			(effects
+				(font
+					(size 1.27 1.27)
+				)
+				(hide yes)
+			)
+		)
+		(pin "1"
+		)
+		(instances
+			(project "v3.1"
+				(path "/1501dcbd-05c1-4298-b373-c91a1b0991c0"
+					(reference "#FLG03")
+					(unit 1)
+				)
