File: hardware/pcbs/bottom_pcb/v3.1.kicad_sch (KiCad schematic)
At the start: 18 parts, among them J1 Programming Connector, J10 Sec Com, J2 Jumper, J3 mount_hole, J4 mount_hole, J5 mount_hole, J6 mount_hole, J7 mount_hole, J8 mount_hole, J9 Main Com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

Commit message: before ki
Parts:
- removed C1, C3: 10uF, Capacitor_THT:CP_Radial_D4.0mm_P1.50mm, symbol 3dAudioSym:C_Polarized
- removed C2, C4: 100nF, Capacitor_SMD:C_1206_3216Metric_Pad1.33x1.80mm_HandSolder, symbol 3dAudioSym:C
- removed J1: Programming Connector, 3dAudioFoot:Molex_KK-254_AE-6410-03A_1x03_P2.54mm_Vertical, symbol 3dAudioSym:molex1x03
- removed J10: Sec Com, Connector_Molex:Molex_KK-254_AE-6410-04A_1x04_P2.54mm_Vertical, symbol 3dAudioSym:molex1x04
- removed J2: Jumper, Connector_PinHeader_2.54mm:PinHeader_2x03_P2.54mm_Vertical, symbol Connector_Generic:Conn_02x03_Odd_Even
- removed J3, J4, J5, J6, J7, J8: mount_hole, MountingHole:MountingHole_4.3mm_M4_DIN965_Pad, symbol Connector:Conn_01x01_Pin
- removed J9: Main Com, Connector_Molex:Molex_KK-254_AE-6410-04A_1x04_P2.54mm_Vertical, symbol 3dAudioSym:molex1x04
- removed R112, R113: 10K, Resistor_SMD:R_1206_3216Metric, symbol Device:R
- removed U1, U2: ATtiny1626, 3dAudioFoot:attiny1626, symbol 3dAudioSym:ATtiny1626
- added C3, C4: 100nF, Capacitor_SMD:C_1206_3216Metric_Pad1.33x1.80mm_HandSolder, symbol Device:C
- added H1, H2, H3, H4, H5, H6: MountingHole, MountingHole:MountingHole_3.2mm_M3, symbol Mechanical:MountingHole
- added J1: esp_io_shield1, Connector_PinHeader_2.54mm:PinHeader_2x07_P2.54mm_Vertical_SMD, symbol Connector_Generic:Conn_02x07_Odd_Even
- added J2: esp_io_shield2, Connector_PinHeader_2.54mm:PinHeader_2x11_P2.54mm_Vertical_SMD, symbol Connector_Generic:Conn_02x11_Odd_Even
- added J3: esp32_voltage_shield, Connector_PinHeader_2.54mm:PinHeader_2x04_P2.54mm_Vertical_SMD, symbol Connector_Generic:Conn_02x04_Odd_Even
- added J4: Con_top_pcb, Connector_JST:JST_PH_B9B-PH-K_1x09_P2.00mm_Vertical, symbol Connector:Conn_01x09_Pin
- added J5: con_rpi, Connector_JST:JST_PH_B9B-PH-K_1x09_P2.00mm_Vertical, symbol Connector:Conn_01x09_Pin
- added R1, R2, R3, R4, R6, R7, R8: 100, Resistor_SMD:R_1206_3216Metric_Pad1.30x1.75mm_HandSolder, symbol Device:R
- added SW1: SW_Push, symbol Switch:SW_Push
- added U2: ~, esp32:DFR0645, symbol esp32:DFR0654
- added U4: 74HC4051, Package_SO:SOIC-16_3.9x9.9mm_P1.27mm, symbol 74xx:74HC4051
Connections:
- net +5V: now also J3.1 (Pin_1), J3.2 (Pin_2), J5.1 (Pin_1), U2.32 (VCC)
- net BR1: now also U4.15 (A2)
- net BR2: now also U4.14 (A1)
- net BR3: now also U4.13 (A0)
- net EA1: now also J1.1 (Pin_1), J1.2 (Pin_2), U2.6 (18/SCK)
- net EA2: now also J1.7 (Pin_7), J1.8 (Pin_8), U2.12 (13/D7)
- net EA3: now also J1.11 (Pin_11), J1.12 (Pin_12), U2.15 (26/D3)
- net EA4: now also J2.15 (Pin_15), J2.16 (Pin_16), U2.22 (12/D13)
- net EB1: now also J1.5 (Pin_5), J1.6 (Pin_6), U2.8 (19/MISO)
- net EB2: now also J1.10 (Pin_10), J1.9 (Pin_9), U2.13 (14/D6)
- net EB3: now also J1.13 (Pin_13), J1.14 (Pin_14), U2.16 (25/D2)
- net EB4: now also J2.13 (Pin_13), J2.14 (Pin_14), U2.23 (36/A0)
- net ES1: now also U4.12 (A3)
- net ES2: now also U4.1 (A4)
- net ES3: now also U4.5 (A5)
- net ES4: now also U4.2 (A6)
- net GND: now also C3.2, C4.2, J3.7 (Pin_7), J3.8 (Pin_8), J4.6 (Pin_6), J5.3 (Pin_3), J5.5 (Pin_5), U2.30 (GND), U2.4 (GND), U4.6 (~{E}), U4.7 (VEE), U4.8 (GND)
- net SCL: now also J2.1 (Pin_1), J2.2 (Pin_2), J5.4 (Pin_4), U2.29 (22/SCL)
- net SDA: now also J2.3 (Pin_3), J2.4 (Pin_4), J5.2 (Pin_2), U2.28 (21/SDA)
- new net: J3.5 (Pin_5), J3.6 (Pin_6), U2.2 (3v3)
- new net: J2.11 (Pin_11), J2.12 (Pin_12), R4.2, U2.24 (39/A1)
- new net: J2.10 (Pin_10), J2.9 (Pin_9), R3.2, U2.25 (34/A2)
- new net: J2.7 (Pin_7), J2.8 (Pin_8), R2.2, U2.26 (35/A3)
- new net: J2.5 (Pin_5), J2.6 (Pin_6), R1.2, U2.27 (15/A4)
- new net: J4.3 (Pin_3), R6.1
- new net: J4.4 (Pin_4), R7.1
- new net: J4.5 (Pin_5), R8.1
- new net +3V3: C3.1, J3.3 (Pin_3), J3.4 (Pin_4), J4.1 (Pin_1), U2.1 (RST), U2.31 (3V3), U4.16 (VCC)
- new net MUX_A: R1.1
- new net MUX_B: R2.1
- new net MUX_C: R3.1, U4.3 (A)
- new net MUX_D: C4.1, J4.2 (Pin_2), R4.1
- new net MUX_S0: J2.17 (Pin_17), J2.18 (Pin_18), R6.2, U2.21 (4/D12), U4.9 (S2)
- new net MUX_S1: J2.19 (Pin_19), J2.20 (Pin_20), R7.2, U2.20 (16/D11), U4.10 (S1)
- new net MUX_S2: J2.21 (Pin_21), J2.22 (Pin_22), R8.2, U2.19 (17/D10), U4.11 (S0)
- new net led_driver/in: J1.3 (Pin_3), J1.4 (Pin_4), U2.7 (23/MOSI)
- no-connect marks 3 -> 15
Other:
- added sheet led_driver (led_driver.kicad_sch)
- sheet Button square ports: added A, B, S0, S1, S2; removed BUTAB1, BUTAB2, BUTAB3, BUTAB4, BUTCD1, BUTCD2, BUTCD3, BUTCD4, BUT_CTL
- sheet LED ports: added led_dat; removed LED_CLK, LED_DATA, LED_UPDATE
