File: hardware/pcbs/bottom_pcb/button_matrix.kicad_sch (KiCad schematic)
At the start: 35 parts, among them U11 touch_but_square, U12 touch_but_square, U13 touch_but_square, U14 touch_but_square, U15 touch_but_square, U16 touch_but_square, U17 touch_but_square, U18 touch_but_square, U19 74VHC4053AFT, U20 74VHC4053AFT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

Commit message: pcb main fertig
Connections:
- net BUTA1: now also U19.5 (0Z); no longer U19.12 (0X)
- net BUTA3: now also U20.12 (0X); no longer U19.5 (0Z)
- net BUTAB1: now also U19.9 (C); no longer U19.11 (A)
- net BUTAB3: now also U20.11 (A); no longer U19.9 (C)
- net BUTB1: now also R81.2, U19.3 (1Z), U26.1; no longer R77.2, U11.1, U19.13 (1X)
- net BUTB2: now also R82.2, U27.1; no longer R78.2, U12.1
- net BUTB3: now also R83.2, U20.13 (1X), U28.1; no longer R79.2, U13.1, U19.3 (1Z)
- net BUTB4: now also R84.2, U29.1; no longer R80.2, U14.1
- net BUTC1: now also R77.2, U11.1, U19.12 (0X); no longer R81.2, U20.12 (0X), U26.1
- net BUTC2: now also R78.2, U12.1; no longer R82.2, U27.1
- net BUTC3: now also R79.2, U13.1; no longer R83.2, U28.1
- net BUTC4: now also R80.2, U14.1; no longer R84.2, U29.1
- net BUTCD1: now also U19.11 (A); no longer U20.11 (A)
- net BUTD1: now also U19.13 (1X); no longer U20.13 (1X)

Commit message: generated gerber files v31
Parts:
- R73, R74, R75, R76, R77, R78, R79, R80, R81, R82, R83, R84, R85, R86, R87, R88: value R -> 10K; footprint Resistor_SMD:R_1206_3216Metric_Pad1.30x1.75mm_HandSolder -> Resistor_SMD:R_1206_3216Metric

Commit message: before ki
Parts:
- removed U19, U20, U21: 74VHC4053AFT, 3dAudioFoot:74vhc4053aft, symbol 3dAudioSym:74VHC4053AFT
- added C1, C2: 100nF, Capacitor_SMD:C_1206_3216Metric_Pad1.33x1.80mm_HandSolder, symbol Device:C
- added U1, U3: 74HC4051, Package_SO:SOIC-16_3.9x9.9mm_P1.27mm, symbol 74xx:74HC4051
Connections:
- net BUTA1: now also U1.13 (A0)
- net BUTA2: now also U1.14 (A1)
- net BUTA3: now also U1.15 (A2)
- net BUTA4: now also U1.12 (A3)
- net BUTB1: now also U1.1 (A4)
- net BUTB2: now also U1.5 (A5)
- net BUTB3: now also U1.2 (A6)
- net BUTB4: now also U1.4 (A7)
- net BUTC1: now also U3.13 (A0)
- net BUTC2: now also U3.14 (A1)
- net BUTC3: now also U3.15 (A2)
- net BUTC4: now also U3.12 (A3)
- net BUTD1: now also U3.1 (A4)
- net BUTD2: now also U3.5 (A5)
- net BUTD3: now also U3.2 (A6)
- net BUTD4: now also U3.4 (A7)
- net GND: now also C1.2, C2.2, U1.6 (~{E}), U1.7 (VEE), U1.8 (GND), U3.6 (~{E}), U3.7 (VEE), U3.8 (GND)
- net +5V renamed +3V3
- net +3V3: now also C1.1, C2.1, U1.16 (VCC), U3.16 (VCC)
- new net A: U1.3 (A)
- new net B: U3.3 (A)
- new net S0: U1.11 (S0), U3.11 (S0)
- new net S1: U1.10 (S1), U3.10 (S1)
- new net S2: U1.9 (S2), U3.9 (S2)
- no-connect marks 4 -> 0
