File: hardware/pcbs/bottom_pcb/enc_arr.kicad_sch (KiCad schematic)
At the start: 32 parts

Commit message: generated gerber files v31
Parts:
- C13, C14, C15, C16, C17, C18, C19, C21: value 10nF -> 100nF
- R100, R101, R102, R103, R104, R105, R106, R107, R108, R109, R110, R111, R89, R90, R91, R92, R93, R94, R98, R99: value 10k -> 10K; footprint Resistor_SMD:R_1206_3216Metric_Pad1.30x1.75mm_HandSolder -> Resistor_SMD:R_1206_3216Metric

Commit message: before ki
Parts:
- R100, R104, R106, R107, R108, R109, R110, R111: value 10K -> 1k
Connections:
- net +5V renamed +3V3
