File: hardware/pcbs/bottom_pcb/led_arr2.kicad_sch (KiCad schematic)
At the start: 107 parts, among them U10 TPIC6C595, U3 TPIC6C595, U4 TPIC6C595, U5 TPIC6C595, U6 TPIC6C595, U7 TPIC6C595, U8 TPIC6C595, U9 TPIC6C595

Commit message: pcb main fertig
Parts:
- added R114, R115, R116, R117, R118, R119, R120, R121: 0R, Resistor_SMD:R_1206_3216Metric_Pad1.30x1.75mm_HandSolder, symbol Device:R
Connections:
- net LED_CLK: now also R114.1, R115.1, R116.1, R117.1, R118.1, R119.1, R120.1; no longer U10.15 (SRCK), U3.15 (SRCK), U4.15 (SRCK), U5.15 (SRCK), U7.15 (SRCK), U8.15 (SRCK), U9.15 (SRCK)
- net LED_DATA: now also R121.1; no longer U3.2 (SERIN)
- net LED_DATAAB: now also U4.9 (SEROUT); no longer U5.2 (SERIN)
- net LED_DATABC: now also U6.9 (SEROUT); no longer U7.2 (SERIN)
- net LED_DATACD: now also U8.9 (SEROUT); no longer U9.2 (SERIN)
- net at R36.1: now also U7.2 (SERIN); no longer U6.9 (SEROUT)
- net at R55.1: now also U9.2 (SERIN); no longer U8.9 (SEROUT)
- net at R32.1: now also U5.2 (SERIN); no longer U4.9 (SEROUT)
- new net: R116.2, U5.15 (SRCK)
- new net: R119.2, U9.15 (SRCK)
- new net: R118.2, U8.15 (SRCK)
- new net: R121.2, U3.2 (SERIN)
- new net: R114.2, U3.15 (SRCK)
- new net: R120.2, U10.15 (SRCK)
- new net: R117.2, U7.15 (SRCK)
- new net: R115.2, U4.15 (SRCK)
Other:
- moved on the sheet: R31, R32, R35, R36, R54, R55, R70

Commit message: ,,
Parts:
- added R122: 0R, Resistor_SMD:R_1206_3216Metric_Pad1.30x1.75mm_HandSolder, symbol Device:R
Connections:
- net LED_CLK: now also R122.1; no longer U6.15 (SRCK)
- new net: R122.2, U6.15 (SRCK)
Other:
- moved on the sheet: R114, R115, R116, R117, R119, R120, R121, R31, R32, R35, R36, R54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

Commit message: finished top and main PCB
Changed lines of the file:
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@@
-	(wire
-		(pts
-			(xy 90.17 26.67) (xy 88.9 26.67)
-		)
-		(stroke
-			(width 0)
-			(type default)
-		)
-	)
 	(wire
 		(pts
@@
 		)
 		(stroke
-			(width 0)
-			(type default)
-		)
-	)
-	(wire
-		(pts
-			(xy 87.63 25.4) (xy 87.63 24.13)
-		)
-		(stroke

Commit message: generated gerber files v31
Parts:
- R1, R10, R11, R13, R14, R16, R17, R19, R2, R20, R22, R23, R25, R26, R28, R29, R37, R38, R4, R40, R41, R43, R44, R46, R47, R49, R5, R50, R58, R59, R61, R62, R64, R65, R67, R68, R7, R8: value R -> 220
- R114, R115, R116, R117, R118, R119, R120, R121, R122, R31, R32, R33, R34, R35, R36, R52, R53, R54, R55, R56, R57, R70, R71, R72: footprint Resistor_SMD:R_1206_3216Metric_Pad1.30x1.75mm_HandSolder -> Resistor_SMD:R_1206_3216Metric
- R12, R15, R18, R21, R24, R27, R3, R30, R39, R42, R45, R48, R51, R6, R60, R63, R66, R69, R9: value R -> 160

Commit message: before ki
Parts:
- removed C10, C11, C12, C5, C6, C7, C8, C9: 100nF, Capacitor_SMD:C_1206_3216Metric_Pad1.33x1.80mm_HandSolder, symbol Device:C
- removed D1, D10, D11, D12, D13, D14, D15, D16, D17, D18, D19, D2, D3, D4, D5, D6, D7, D8, D9: RGB_led, 3dAudioFoot:LED_QBLP679E-RGB, symbol 3dAudioSym:QBLP679E-RGB
- removed R1, R10, R11, R13, R14, R16, R17, R19, R2, R20, R22, R23, R25, R26, R28, R29, R37, R38, R4, R40, R41, R43, R44, R46, R47, R49, R5, R50, R58, R59, R61, R62, R64, R65, R67, R68, R7, R8: 220, Resistor_SMD:R_1206_3216Metric, symbol Device:R
- removed R114, R115, R116, R117, R118, R119, R120, R121, R122, R31, R32, R35, R36, R54, R55, R70: 0R, Resistor_SMD:R_1206_3216Metric, symbol Device:R
- removed R12, R15, R18, R21, R24, R27, R3, R30, R39, R42, R45, R48, R51, R6, R60, R63, R66, R69, R9: 160, Resistor_SMD:R_1206_3216Metric, symbol Device:R
- removed R33, R34, R52, R53, R56, R57, R71, R72: 4K7, Resistor_SMD:R_1206_3216Metric, symbol Device:R
- removed U10, U3, U4, U5, U6, U7, U8, U9: TPIC6C595, Package_SO:SOIC-16_3.9x9.9mm_P1.27mm, symbol 3dAudioSym:TPIC6C595
- added C5: 10v/1mF, Capacitor_SMD:CP_Elec_10x10, symbol Device:C_Polarized
- added D1, D10, D11, D12, D13, D14, D15, D16, D17, D18, D19, D2, D3, D4, D5, D6, D7, D8, D9: WS2812B-2020, LED_SMD:LED_WS2812B-2020_PLCC4_2.0x2.0mm, symbol LED:WS2812B-2020
- added D20: switches, 3dAudioFoot:A3_CherryMxHybrid_WS2812Led2020, symbol 3dAudioSym:A3_switches_led
Connections:
- net +5V: now also C5.1, D1.4 (VDD), D10.4 (VDD), D11.4 (VDD), D12.4 (VDD), D13.4 (VDD), D14.4 (VDD), D15.4 (VDD), D16.4 (VDD), D17.4 (VDD), D18.4 (VDD), D19.4 (VDD), D2.4 (VDD), D3.4 (VDD), D4.4 (VDD), D5.4 (VDD), D6.4 (VDD), D7.4 (VDD), D8.4 (VDD), D9.4 (VDD)
- net GND: now also C5.2, D1.2 (VSS), D10.2 (VSS), D11.2 (VSS), D12.2 (VSS), D13.2 (VSS), D14.2 (VSS), D15.2 (VSS), D16.2 (VSS), D17.2 (VSS), D18.2 (VSS), D19.2 (VSS), D2.2 (VSS), D3.2 (VSS), D4.2 (VSS), D5.2 (VSS), D6.2 (VSS), D7.2 (VSS), D8.2 (VSS), D9.2 (VSS)
- new net: D13.1 (DOUT), D14.3 (DIN)
- new net: D12.1 (DOUT), D13.3 (DIN)
- new net: D15.1 (DOUT), D16.3 (DIN)
- new net: D14.1 (DOUT), D15.3 (DIN)
- new net: D1.1 (DOUT), D2.3 (DIN)
- new net: D18.1 (DOUT), D19.3 (DIN)
- new net: D17.1 (DOUT), D18.3 (DIN)
- new net: D7.1 (DOUT), D8.3 (DIN)
- new net: D10.1 (DOUT), D11.3 (DIN)
- new net: D10.3 (DIN), D9.1 (DOUT)
- new net: D4.1 (DOUT), D5.3 (DIN)
- new net: D3.1 (DOUT), D4.3 (DIN)
- new net: D11.1 (DOUT), D12.3 (DIN)
- new net: D2.1 (DOUT), D3.3 (DIN)
- new net: D5.1 (DOUT), D6.3 (DIN)
- new net: D6.1 (DOUT), D7.3 (DIN)
- new net dat1: D8.1 (DOUT), D9.3 (DIN)
- new net dat2: D16.1 (DOUT), D17.3 (DIN)
- new net led_dat: D1.3 (DIN)
- no-connect marks 8 -> 1

Commit message: t
Parts:
- D1, D10, D11, D12, D13, D14, D15, D16, D17, D18, D19, D2, D3, D4, D5, D6, D7, D8, D9: symbol LED:WS2812B-2020 -> 3dAudioSym:A3_switches_led
Connections:
- net dat1: no longer D8.1 (DOUT), D9.3 (DIN)
- net dat2: no longer D16.1 (DOUT), D17.3 (DIN)
- net led_dat: no longer D1.3 (DIN)
- net at D13.1 (DOUT): no longer D14.3 (DIN)
- net at D13.3 (DIN): no longer D12.1 (DOUT)
- net at D15.1 (DOUT): no longer D16.3 (DIN)
- net at D15.3 (DIN): no longer D14.1 (DOUT)
- net at D1.1 (DOUT): no longer D2.3 (DIN)
- net at D18.1 (DOUT): no longer D19.3 (DIN)
- net at D18.3 (DIN): no longer D17.1 (DOUT)
- net at D8.3 (DIN): no longer D7.1 (DOUT)
- net at D10.1 (DOUT): no longer D11.3 (DIN)
- net at D10.3 (DIN): no longer D9.1 (DOUT)
- net at D4.1 (DOUT): no longer D5.3 (DIN)
- net at D4.3 (DIN): no longer D3.1 (DOUT)
- net at D11.1 (DOUT): no longer D12.3 (DIN)
- net at D2.1 (DOUT): no longer D3.3 (DIN)
- net at D5.1 (DOUT): no longer D6.3 (DIN)
- net at D7.3 (DIN): no longer D6.1 (DOUT)
Changed lines of the file:
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@@
 	)
 	(symbol
-		(lib_id "LED:WS2812B-2020")
+		(lib_id "3dAudioSym:A3_switches_led")
 		(at 160.02 88.9 0)
 		(unit 1)
@@
 	)
 	(symbol
-		(lib_id "LED:WS2812B-2020")
+		(lib_id "3dAudioSym:A3_switches_led")
 		(at 215.9 88.9 0)
 		(unit 1)
@@
 	)
 	(symbol
-		(lib_id "LED:WS2812B-2020")
+		(lib_id "3dAudioSym:A3_switches_led")
 		(at 48.26 45.72 0)
 		(unit 1)
@@
 	)
 	(symbol
-		(lib_id "LED:WS2812B-2020")
+		(lib_id "3dAudioSym:A3_switches_led")
 		(at 76.2 144.78 0)
 		(unit 1)
@@
 	)
 	(symbol
-		(lib_id "LED:WS2812B-2020")
+		(lib_id "3dAudioSym:A3_switches_led")
 		(at 243.84 45.72 0)
 		(unit 1)
@@
 	)
 	(symbol
-		(lib_id "LED:WS2812B-2020")
+		(lib_id "3dAudioSym:A3_switches_led")
 		(at 76.2 88.9 0)
 		(unit 1)
@@
 	)
 	(symbol
-		(lib_id "LED:WS2812B-2020")
+		(lib_id "3dAudioSym:A3_switches_led")
 		(at 132.08 45.72 0)
 		(unit 1)
@@
 	)
 	(symbol
-		(lib_id "LED:WS2812B-2020")
+		(lib_id "3dAudioSym:A3_switches_led")
 		(at 104.14 144.78 0)
 		(unit 1)
@@
 	)
 	(symbol
-		(lib_id "LED:WS2812B-2020")
+		(lib_id "3dAudioSym:A3_switches_led")
 		(at 104.14 88.9 0)
 		(unit 1)
@@
 	)
 	(symbol
-		(lib_id "LED:WS2812B-2020")
+		(lib_id "3dAudioSym:A3_switches_led")
 		(at 76.2 45.72 0)
 		(unit 1)
@@
 	)
 	(symbol
-		(lib_id "LED:WS2812B-2020")
+		(lib_id "3dAudioSym:A3_switches_led")
 		(at 187.96 88.9 0)
 		(unit 1)
@@
 	)
 	(symbol
-		(lib_id "LED:WS2812B-2020")
+		(lib_id "3dAudioSym:A3_switches_led")
 		(at 160.02 45.72 0)
 		(unit 1)
@@
 	)
 	(symbol
-		(lib_id "LED:WS2812B-2020")
+		(lib_id "3dAudioSym:A3_switches_led")
 		(at 215.9 45.72 0)
 		(unit 1)
@@
 	)
 	(symbol
-		(lib_id "LED:WS2812B-2020")
+		(lib_id "3dAudioSym:A3_switches_led")
 		(at 243.84 88.9 0)
 		(unit 1)
@@
 	)
 	(symbol
-		(lib_id "LED:WS2812B-2020")
+		(lib_id "3dAudioSym:A3_switches_led")
 		(at 48.26 88.9 0)
 		(unit 1)
@@
 	)
 	(symbol
-		(lib_id "LED:WS2812B-2020")
+		(lib_id "3dAudioSym:A3_switches_led")
 		(at 104.14 45.72 0)
 		(unit 1)
@@
 	)
 	(symbol
-		(lib_id "LED:WS2812B-2020")
+		(lib_id "3dAudioSym:A3_switches_led")
 		(at 187.96 45.72 0)
 		(unit 1)
@@
 	)
 	(symbol
-		(lib_id "LED:WS2812B-2020")
+		(lib_id "3dAudioSym:A3_switches_led")
 		(at 48.26 144.78 0)
 		(unit 1)
@@
 	)
 	(symbol
-		(lib_id "LED:WS2812B-2020")
+		(lib_id "3dAudioSym:A3_switches_led")
 		(at 132.08 88.9 0)
 		(unit 1)
