File: hardware/pcbs/top_pcb/encoder_matrix.kicad_sch (KiCad schematic)
At the start: 56 parts, among them U2 74hc4066, U3 74hc4066, U4 74hc4066, U5 74hc4066, U6 74hc4066, U7 74hc4066, U8 74hc4066, U9 74hc4066

Commit message: ,,
Parts:
- removed MT1, MT2, MT3, MT4, MT5, MT6, MT7, MT8: PEC11R-4215F-S0024, 3dAudioFoot:XDCR_PEC11R-4215F-S0024, symbol 3dAudioSym:PEC11R-4215F-S0024
- removed R1, R10, R11, R12, R13, R14, R15, R16, R17, R18, R19, R2, R20, R21, R22, R23, R24, R4, R5, R6, R7, R8, R9: 10k, Resistor_SMD:R_1206_3216Metric_Pad1.30x1.75mm_HandSolder, symbol Device:R
- added R25, R26, R27, R28, R29, R30, R31: 10k, Resistor_SMD:R_1206_3216Metric_Pad1.30x1.75mm_HandSolder, symbol Device:R
- added U10, U11, U12, U13, U14, U15, U16, U17: ~, 3dAudioFoot:Encoder und Endless, symbol 3dAudioSym:Enc_Mix
Connections:
- net +5V: now also R25.1, R26.1, R27.1, R28.1, R29.1, R30.1, R31.1, U10.3 (EP3/PX), U11.3 (EP3/PX), U12.3 (EP3/PX), U13.3 (EP3/PX), U14.3 (EP3/PX), U15.3 (EP3/PX), U16.3 (EP3/PX), U17.3 (EP3/PX); no longer C10.2, C11.1, C12.2, C13.1, C14.2, C15.1, C16.2, C17.1, C18.2, C3.1, C4.2, C5.1, C6.2, C7.1, C8.2, C9.1
- net ENC_A_A: now also R3.2
- net ENC_A_B: now also R28.2
- net ENC_A_SW: now also U4.9 (3Z); no longer U3.9 (3Z)
- net ENC_B_A: now also R25.2
- net ENC_B_B: now also R29.2
- net ENC_B_SW: now also U3.9 (3Z); no longer U4.9 (3Z)
- net ENC_C_A: now also R26.2
- net ENC_C_B: now also R30.2
- net ENC_C_SW: now also U8.9 (3Z); no longer U7.9 (3Z)
- net ENC_D_A: now also R27.2
- net ENC_D_B: now also R31.2
- net ENC_D_SW: now also U7.9 (3Z); no longer U8.9 (3Z)
- net E_A1_A: now also C4.1, U10.2b (EP2b/P3), U10.A2 (EA2); no longer C3.2, R3.2
- net E_A1_B: now also C3.1, U10.2a (EP2a/P1), U10.A1 (EA1); no longer C4.1
- net E_A1_SW: now also U10.d (E_SW2)
- net E_A2_A: now also C6.1, U11.2b (EP2b/P3), U11.A2 (EA2); no longer C5.2
- net E_A2_B: now also C5.1, U11.2a (EP2a/P1), U11.A1 (EA1); no longer C6.1
- net E_A2_SW: now also U11.d (E_SW2)
- net E_B1_A: now also C9.1, U12.2b (EP2b/P3), U12.A2 (EA2); no longer C7.2
- net E_B1_B: now also C7.1, U12.2a (EP2a/P1), U12.A1 (EA1); no longer C8.1
- net E_B1_SW: now also U12.d (E_SW2)
- net E_B2_A: now also C10.1, U13.2b (EP2b/P3), U13.A2 (EA2); no longer C9.2
- net E_B2_B: now also C8.1, U13.2a (EP2a/P1), U13.A1 (EA1); no longer C10.1
- net E_B2_SW: now also U13.d (E_SW2)
- net E_C1_A: now also C13.1, U14.2b (EP2b/P3), U14.A2 (EA2); no longer C11.2
- net E_C1_B: now also C11.1, U14.2a (EP2a/P1), U14.A1 (EA1); no longer C12.1
- net E_C1_SW: now also U14.d (E_SW2)
- net E_C2_A: now also C14.1, U15.2b (EP2b/P3), U15.A2 (EA2); no longer C13.2
- net E_C2_B: now also C12.1, U15.2a (EP2a/P1), U15.A1 (EA1); no longer C14.1
- net E_C2_SW: now also U15.d (E_SW2)
- net E_D1_A: now also C17.1, U16.2b (EP2b/P3), U16.A2 (EA2); no longer C15.2
- net E_D1_B: now also C15.1, U16.2a (EP2a/P1), U16.A1 (EA1); no longer C16.1
- net E_D1_SW: now also U16.d (E_SW2)
- net E_D2_A: now also C18.1, U17.2b (EP2b/P3), U17.A2 (EA2); no longer C17.2
- net E_D2_B: now also C16.1, U17.2a (EP2a/P1), U17.A1 (EA1); no longer C18.1
- net E_D2_SW: now also U17.d (E_SW2)
- net GND: now also C10.2, C11.2, C12.2, C13.2, C14.2, C15.2, C16.2, C17.2, C18.2, C3.2, C4.2, C5.2, C6.2, C7.2, C8.2, C9.2, U10.1 (EP1/P2), U10.B (EB), U10.c (E_SW1), U11.1 (EP1/P2), U11.B (EB), U11.c (E_SW1), U12.1 (EP1/P2), U12.B (EB), U12.c (E_SW1), U13.1 (EP1/P2), U13.B (EB), U13.c (E_SW1), U14.1 (EP1/P2), U14.B (EB), U14.c (E_SW1), U15.1 (EP1/P2), U15.B (EB), U15.c (E_SW1), U16.1 (EP1/P2), U16.B (EB), U16.c (E_SW1), U17.1 (EP1/P2), U17.B (EB), U17.c (E_SW1)
