File: hardware/pcbs/top_pcb/pcb_top.kicad_pcb (KiCad board)
At the start: 2 copper layers, 105 x 47 mm, 20 parts, among them J1 molex1x03, U1 ATtiny1626, U2 74hc4066, U3 74hc4066, U4 74hc4066, U5 74hc4066, U6 74hc4066, U7 74hc4066, U8 74hc4066, U9 74hc4066

Commit message: ,,
Parts:
- removed MT1, MT2, MT3, MT4, MT5, MT6, MT7, MT8: PEC11R-4215F-S0024, 3dAudioFoot:XDCR_PEC11R-4215F-S0024
- added C10: 100n, Capacitor_SMD:C_1206_3216Metric_Pad1.33x1.80mm_HandSolder, B.Cu at (101.3, 83.7)
- added C11: 100n, Capacitor_SMD:C_1206_3216Metric_Pad1.33x1.80mm_HandSolder, B.Cu at (120.0, 60.2)
- added C12: 100n, Capacitor_SMD:C_1206_3216Metric_Pad1.33x1.80mm_HandSolder, B.Cu at (114.9, 82.1)
- added C13: 100n, Capacitor_SMD:C_1206_3216Metric_Pad1.33x1.80mm_HandSolder, B.Cu at (125.2, 60.2)
- added C14: 100n, Capacitor_SMD:C_1206_3216Metric_Pad1.33x1.80mm_HandSolder, B.Cu at (129.8, 83.7)
- added C15: 100n, Capacitor_SMD:C_1206_3216Metric_Pad1.33x1.80mm_HandSolder, B.Cu at (148.5, 60.2)
- added C16: 100n, Capacitor_SMD:C_1206_3216Metric_Pad1.33x1.80mm_HandSolder, B.Cu at (143.4, 82.1)
- added C17: 100n, Capacitor_SMD:C_1206_3216Metric_Pad1.33x1.80mm_HandSolder, B.Cu at (151.6, 62.7)
- added C18: 100n, Capacitor_SMD:C_1206_3216Metric_Pad1.33x1.80mm_HandSolder, B.Cu at (158.3, 83.7)
- added C3: 100n, Capacitor_SMD:C_1206_3216Metric_Pad1.33x1.80mm_HandSolder, B.Cu at (63.0, 60.2)
- added C4: 100n, Capacitor_SMD:C_1206_3216Metric_Pad1.33x1.80mm_HandSolder, B.Cu at (66.1, 62.7)
- added C5: 100n, Capacitor_SMD:C_1206_3216Metric_Pad1.33x1.80mm_HandSolder, B.Cu at (57.9, 82.1)
- added C6: 100n, Capacitor_SMD:C_1206_3216Metric_Pad1.33x1.80mm_HandSolder, B.Cu at (72.8, 83.7)
- added C7: 100n, Capacitor_SMD:C_1206_3216Metric_Pad1.33x1.80mm_HandSolder, B.Cu at (87.3, 56.9)
- added C8: 100n, Capacitor_SMD:C_1206_3216Metric_Pad1.33x1.80mm_HandSolder, B.Cu at (86.4, 82.1)
- added C9: 100n, Capacitor_SMD:C_1206_3216Metric_Pad1.33x1.80mm_HandSolder, B.Cu at (94.2, 60.0)
- added R25: 10k, Resistor_SMD:R_1206_3216Metric_Pad1.30x1.75mm_HandSolder, B.Cu at (85.4, 51.8)
- added R26: 10k, Resistor_SMD:R_1206_3216Metric_Pad1.30x1.75mm_HandSolder, B.Cu at (133.5, 62.0)
- added R27: 10k, Resistor_SMD:R_1206_3216Metric_Pad1.30x1.75mm_HandSolder, B.Cu at (142.9, 52.6)
- added R28: 10k, Resistor_SMD:R_1206_3216Metric_Pad1.30x1.75mm_HandSolder, B.Cu at (57.0, 53.2)
- added R29: 10k, Resistor_SMD:R_1206_3216Metric_Pad1.30x1.75mm_HandSolder, B.Cu at (81.8, 51.8)
- added R3: 10k, Resistor_SMD:R_1206_3216Metric_Pad1.30x1.75mm_HandSolder, B.Cu at (59.5, 53.2)
- added R30: 10k, Resistor_SMD:R_1206_3216Metric_Pad1.30x1.75mm_HandSolder, B.Cu at (130.2, 62.1)
- added R31: 10k, Resistor_SMD:R_1206_3216Metric_Pad1.30x1.75mm_HandSolder, B.Cu at (140.1, 52.6)
- added U10: ~, 3dAudioFoot:Encoder und Endless, F.Cu at (65.8, 47.5)
- added U11: ~, 3dAudioFoot:Encoder und Endless, F.Cu at (65.8, 76.0)
- added U12: ~, 3dAudioFoot:Encoder und Endless, F.Cu at (94.3, 47.5)
- added U13: ~, 3dAudioFoot:Encoder und Endless, F.Cu at (94.3, 76.0)
- added U14: ~, 3dAudioFoot:Encoder und Endless, F.Cu at (122.8, 47.5)
- added U15: ~, 3dAudioFoot:Encoder und Endless, F.Cu at (122.8, 76.0)
- added U16: ~, 3dAudioFoot:Encoder und Endless, F.Cu at (151.3, 47.5)
- added U17: ~, 3dAudioFoot:Encoder und Endless, F.Cu at (151.3, 76.0)
- moved J1 35.4 mm to (110.8, 43.5)
- moved C1 34.4 mm to (109.1, 77.3)
- moved C2 24.1 mm to (108.4, 73.3)
- moved U3 3.50 mm to (65.8, 77.5), turned to 0 degrees
- moved U5 3.50 mm to (94.3, 77.5), turned to 0 degrees
- moved U7 3.50 mm to (122.8, 77.5), turned to 0 degrees
- moved U9 3.40 mm to (151.3, 77.5), turned to 0 degrees
- moved U1 2.35 mm to (108.2, 63.6), turned to 0 degrees
- moved U4 0.20 mm to (94.3, 49.0), turned to 0 degrees
- turned U2 to 0 degrees
- turned U6 to 0 degrees
- turned U8 to 0 degrees
Connections:
- U3 pad 9: /Untitled Sheet/ENC_A_SW -> /Untitled Sheet/ENC_B_SW
- U4 pad 9: /Untitled Sheet/ENC_B_SW -> /Untitled Sheet/ENC_A_SW
- U7 pad 9: /Untitled Sheet/ENC_C_SW -> /Untitled Sheet/ENC_D_SW
- U8 pad 9: /Untitled Sheet/ENC_D_SW -> /Untitled Sheet/ENC_C_SW
Routing:
- added copper zone on B.Cu, net GND
- added copper zone on F.Cu, net GND
Other:
- board size 105 x 47 mm -> 123.8 x 50.7 mm

Commit message: finished top and main PCB
Parts:
- added H1: MountingHole_Pad-Mechanical, MountingHole:MountingHole_4.3mm_M4_DIN965_Pad, F.Cu at (141.3, 64.5)
- added H2: MountingHole_Pad-Mechanical, MountingHole:MountingHole_4.3mm_M4_DIN965_Pad, F.Cu at (76.8, 64.5)
- added J2: molex1x03, 3dAudioFoot:Molex_KK-254_AE-6410-03A_1x03_P2.54mm_Vertical, B.Cu at (111.0, 41.7)
- J1: value molex1x03 -> molex1x04; footprint 3dAudioFoot:Molex_KK-254_AE-6410-03A_1x03_P2.54mm_Vertical -> Connector_Molex:Molex_KK-254_AE-6410-04A_1x04_P2.54mm_Vertical
- moved R28 13.2 mm to (58.8, 66.3)
- moved R26 10.2 mm to (133.5, 51.8)
- moved J1 6.34 mm to (112.3, 49.7)
- moved C7 4.01 mm to (86.0, 60.8)
- moved C12 2.75 mm to (114.9, 84.8)
- moved C16 2.75 mm to (143.4, 84.8)
- moved C8 2.75 mm to (86.4, 84.8)
- moved C5 2.59 mm to (58.8, 84.5)
- moved U3 1.90 mm to (65.8, 75.6)
- moved U5 1.90 mm to (94.3, 75.6)
- moved U7 1.90 mm to (122.8, 75.6)
- moved U9 1.90 mm to (151.3, 75.6)
- moved U2 1.74 mm to (65.8, 47.3)
- moved U4 1.74 mm to (94.3, 47.3)
- moved U6 1.54 mm to (122.8, 47.3)
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Connections:
- C1 pad 1: +5V -> VCC
- C2 pad 1: +5V -> VCC
- J1 pad 1: SDA -> VCC
- J1 pad 3: UPDI -> SDA
- R25 pad 1: +5V -> VCC
- R26 pad 1: +5V -> VCC
- R27 pad 1: +5V -> VCC
- R28 pad 1: +5V -> VCC
- R29 pad 1: +5V -> VCC
- R3 pad 1: +5V -> VCC
- R30 pad 1: +5V -> VCC
- R31 pad 1: +5V -> VCC
- U1 pad 1: +5V -> VCC
- U1 pad 12: /Untitled Sheet/ENC_C_A -> /Untitled Sheet/ENC_C_B
- U1 pad 13: /Untitled Sheet/ENC_C_B -> /Untitled Sheet/ENC_C_A
- U1 pad 2: /Untitled Sheet/ENC_CTL_1 -> /Untitled Sheet/ENC_CTL_2
- U1 pad 3: /Untitled Sheet/ENC_CTL_2 -> /Untitled Sheet/ENC_B_SW
- U1 pad 4: /Untitled Sheet/ENC_A_A -> /Untitled Sheet/ENC_B_A
- U1 pad 5: /Untitled Sheet/ENC_A_B -> /Untitled Sheet/ENC_B_B
- U1 pad 6: /Untitled Sheet/ENC_A_SW -> /Untitled Sheet/ENC_A_A
- U1 pad 7: /Untitled Sheet/ENC_B_A -> /Untitled Sheet/ENC_A_B
- U1 pad 8: /Untitled Sheet/ENC_B_B -> /Untitled Sheet/ENC_CTL_1
- U1 pad 9: /Untitled Sheet/ENC_B_SW -> /Untitled Sheet/ENC_A_SW
- U10 pad 3: +5V -> VCC
- U11 pad 3: +5V -> VCC
- U12 pad 3: +5V -> VCC
- U13 pad 3: +5V -> VCC
- U14 pad 3: +5V -> VCC
- U15 pad 3: +5V -> VCC
- U16 pad 3: +5V -> VCC
- U17 pad 3: +5V -> VCC
- U2 pad 14: +5V -> VCC
- U3 pad 14: +5V -> VCC
- U4 pad 14: +5V -> VCC
- U5 pad 14: +5V -> VCC
- U6 pad 14: +5V -> VCC
- U7 pad 14: +5V -> VCC
- U8 pad 14: +5V -> VCC
- U9 pad 14: +5V -> VCC
Routing:
- net GND: track 0.00 -> 401.1 mm, vias 0 -> 22
- net VCC: track 0.00 -> 374.8 mm, vias 0 -> 3
- net /Untitled Sheet/ENC_CTL_1: track 0.00 -> 124.2 mm, vias 0 -> 2
- net /Untitled Sheet/ENC_CTL_2: track 0.00 -> 122.6 mm, vias 0 -> 2
- net /Untitled Sheet/ENC_A_B: track 0.00 -> 93.7 mm, vias 0 -> 2
- net /Untitled Sheet/ENC_A_A: track 0.00 -> 88.8 mm, vias 0 -> 3
- net /Untitled Sheet/ENC_D_B: track 0.00 -> 80.4 mm, vias 0 -> 3
- net /Untitled Sheet/ENC_D_A: track 0.00 -> 78.0 mm, vias 0 -> 3
- net /Untitled Sheet/ENC_B_B: track 0.00 -> 63.9 mm
- net /Untitled Sheet/ENC_B_A: track 0.00 -> 62.8 mm, vias 0 -> 3
- net /Untitled Sheet/ENC_C_B: track 0.00 -> 62.7 mm, vias 0 -> 2
- net /Untitled Sheet/ENC_C_A: track 0.00 -> 59.1 mm, vias 0 -> 4
- net /Untitled Sheet/ENC_A_SW: track 0.00 -> 54.0 mm
- net /Untitled Sheet/ENC_C_SW: track 0.00 -> 51.9 mm, vias 0 -> 2
- net /Untitled Sheet/ENC_D_SW: track 0.00 -> 49.5 mm
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Other:
- board size 123.8 x 50.7 mm -> 109 x 50.7 mm

Commit message: generated gerber files v31
Parts:
- added R1: 10k, Resistor_SMD:R_1206_3216Metric_Pad1.30x1.75mm_HandSolder, B.Cu at (111.0, 54.5)
- added R2: 10k, Resistor_SMD:R_1206_3216Metric_Pad1.30x1.75mm_HandSolder, B.Cu at (105.5, 54.5)
- moved C17 0.79 mm to (151.6, 63.5)
- moved C15 0.59 mm to (148.6, 60.8)
Routing:
- net VCC: track 374.8 -> 381.6 mm, vias 3 -> 4
- net E_C1_A: track 14.6 -> 13.3 mm
- net E_D1_A: track 15.1 -> 15.9 mm
- net GND: track 401.1 -> 401.8 mm, vias 22 -> 29
- net E_D1_B: track 16.3 -> 16.9 mm
- net /Untitled Sheet/ENC_D_A: track 78.0 -> 78.5 mm
Other:
- board size 109 x 50.7 mm -> 109 x 52.2 mm
