File: hardware/pcbs/top_pcb/pcb_top.kicad_sch (KiCad schematic)
At the start: 4 parts, among them J1 molex1x03, U1 ATtiny1626

Commit message: finished top and main PCB
Parts:
- removed J1: molex1x03, 3dAudioFoot:Molex_KK-254_AE-6410-03A_1x03_P2.54mm_Vertical, symbol 3dAudioSym:molex1x03
- added H1, H2: MountingHole_Pad-Mechanical, MountingHole:MountingHole_4.3mm_M4_DIN965_Pad, symbol 3dAudioSym:MountingHole_Pad-Mechanical
- added J1: molex1x04, Connector_Molex:Molex_KK-254_AE-6410-04A_1x04_P2.54mm_Vertical, symbol 3dAudioSym:molex1x04
- added J2: molex1x03, 3dAudioFoot:Molex_KK-254_AE-6410-03A_1x03_P2.54mm_Vertical, symbol 3dAudioSym:molex1x03
Connections:
- net +5V: now also J1.1 (Pin_1), J2.2 (Pin_2)
- net GND: now also H1.1, H2.1, J1.4 (Pin_4), J2.3 (Pin_3)
- net SCL: now also J1.2 (Pin_2)
- net SDA: now also J1.3 (Pin_3)
- net UPDI: now also J2.1 (Pin_1)
- net Untitled Sheet/ENC_A_A: now also U1.6 (PB5/ADC8/CLKOUT); no longer U1.4 (PA6/ADC6)
- net Untitled Sheet/ENC_A_B: now also U1.7 (PB4/ADC9/RST); no longer U1.5 (PA7/ADC7)
- net Untitled Sheet/ENC_A_SW: now also U1.9 (PB2); no longer U1.6 (PB5/ADC8/CLKOUT)
- net Untitled Sheet/ENC_B_A: now also U1.4 (PA6/ADC6); no longer U1.7 (PB4/ADC9/RST)
- net Untitled Sheet/ENC_B_B: now also U1.5 (PA7/ADC7); no longer U1.8 (PB3)
- net Untitled Sheet/ENC_B_SW: now also U1.3 (PA5/ADC5); no longer U1.9 (PB2)
- net Untitled Sheet/ENC_CTL_1: now also U1.8 (PB3); no longer U1.2 (PA4/ADC4/SS1)
- net Untitled Sheet/ENC_CTL_2: now also U1.2 (PA4/ADC4/SS1); no longer U1.3 (PA5/ADC5)
- net Untitled Sheet/ENC_C_A: now also U1.13 (PC1/ADC13/DO2); no longer U1.12 (PC0/ADC12/SCK2)
- net Untitled Sheet/ENC_C_B: now also U1.12 (PC0/ADC12/SCK2); no longer U1.13 (PC1/ADC13/DO2)

Commit message: generated gerber files v31
Parts:
- added R1, R2: 10k, Resistor_SMD:R_1206_3216Metric_Pad1.30x1.75mm_HandSolder, symbol Device:R
- C2: value 100nF -> 100n
Connections:
- net +5V: now also R1.1, R2.1
- net SCL: now also R1.2
- net SDA: now also R2.2
Other:
- moved on the sheet: J1
