File: hardware/pcbs/motion_pcb/button_matrix.kicad_sch (KiCad schematic)
At the start: 36 parts, among them U1 74HC4051, U11 touch_but_square, U12 touch_but_square, U13 touch_but_square, U14 touch_but_square, U15 touch_but_square, U16 touch_but_square, U17 touch_but_square, U18 touch_but_square, U22 touch_but_square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

Commit message: finished schematic
Parts:
- removed C2: 100nF, Capacitor_SMD:C_1206_3216Metric_Pad1.33x1.80mm_HandSolder, symbol Device:C
- removed R73, R74, R75, R76, R77, R78, R79, R80, R81, R82, R83, R84, R85, R86, R87, R88: 10K, Resistor_SMD:R_1206_3216Metric, symbol Device:R
- removed U1, U3: 74HC4051, Package_SO:SOIC-16_3.9x9.9mm_P1.27mm, symbol 74xx:74HC4051
- removed U11, U12, U13, U14, U15, U16, U17, U18, U22, U23, U24, U25, U26, U27, U28, U29: touch_but_square, 3dAudioFoot:But_Velo_Rec_1, symbol 3dAudioSym:touch_but_square
- added C4, C7: 100nF, Capacitor_SMD:C_1206_3216Metric_Pad1.33x1.80mm_HandSolder, symbol Device:C
- added U1, U7, U8: 74HC4051, symbol 3dAudioSym:74HC4051
Connections:
- net +3V3: now also C4.1, C7.1, U1.16 (VCC), U7.16 (VCC), U8.16 (VCC)
- net A: now also U7.3 (A)
- net B: now also U8.3 (A)
- net GND: now also C4.2, C7.2, U1.6 (~{E}), U1.7 (VEE), U1.8 (GND), U7.6 (~{E}), U7.7 (VEE), U7.8 (GND), U8.6 (~{E}), U8.7 (VEE), U8.8 (GND)
- net S0: now also U1.11 (S0), U7.11 (S0), U8.11 (S0)
- net S1: now also U1.10 (S1), U7.10 (S1), U8.10 (S1)
- net S2: now also U1.9 (S2), U7.9 (S2), U8.9 (S2)
- new net B11: U7.13 (A0)
- new net B12: U7.4 (A7)
- new net B13: U8.13 (A0)
- new net B14: U8.4 (A7)
- new net B21: U7.12 (A3)
- new net B22: U7.5 (A5)
- new net B23: U8.12 (A3)
- new net B24: U8.5 (A5)
- new net B31: U7.15 (A2)
- new net B32: U7.1 (A4)
- new net B33: U8.15 (A2)
- new net B34: U8.1 (A4)
- new net B41: U7.14 (A1)
- new net B42: U7.2 (A6)
- new net B43: U8.14 (A1)
- new net B44: U8.2 (A6)
- new net BR1: U1.13 (A0)
- new net BR2: U1.12 (A3)
- new net BR3: U1.15 (A2)
- new net C: U1.3 (A)
- new net ES1: U1.5 (A5)
- new net ES2: U1.4 (A7)
- new net ES3: U1.2 (A6)
- new net ES4: U1.1 (A4)
- no-connect marks 0 -> 1
