File: hardware/pcbs/motion_pcb/button_matrix_round.kicad_sch (KiCad schematic)
At the start: 6 parts, among them U32 touch_but_round, U33 touch_but_round, U34 touch_but_round

Commit message: finished schematic
Parts:
- removed R95, R96, R97: 10K, Resistor_SMD:R_1206_3216Metric, symbol Device:R
- removed U32, U33, U34: touch_but_round, 3dAudioFoot:But_Velo_Rnd_1, symbol 3dAudioSym:touch_but_round
Connections:
- no-connect marks 0 -> 1
Other:
- added sheet LED_Button (led_button_h.kicad_sch)
- added sheet LED_Button1 (led_button_h.kicad_sch)
- added sheet LED_Button2 (led_button_h.kicad_sch)
