File: hardware/pcbs/motion_pcb/enc_arr.kicad_sch (KiCad schematic)
At the start: 32 parts

Commit message: finished schematic
Parts:
- removed C13, C14, C15, C16, C17, C18, C19, C21: 100nF, Capacitor_SMD:C_1206_3216Metric_Pad1.33x1.80mm_HandSolder, symbol Device:C
- removed MT1, MT2, MT3, MT4: PEC11R-4215F-S0024, 3dAudioFoot:XDCR_PEC11R-4215F-S0024, symbol 3dAudioSym:PEC11R-4215F-S0024
- removed R100, R104, R106, R107, R108, R109, R110, R111: 1k, Resistor_SMD:R_1206_3216Metric, symbol Device:R
- removed R101, R102, R103, R105, R89, R90, R91, R92, R93, R94, R98, R99: 10K, Resistor_SMD:R_1206_3216Metric, symbol Device:R
Other:
- added sheet encoder_h (encoder_h.kicad_sch)
- added sheet encoder_h1 (encoder_h.kicad_sch)
- added sheet encoder_h2 (encoder_h.kicad_sch)
- added sheet encoder_h3 (encoder_h.kicad_sch)
