File: hardware/pcbs/motion_pcb/led_driver.kicad_sch (KiCad schematic)
At the start: 6 parts, among them Q1 BSS138, U5 74AHCT125, U6 SN74LVC1T45DBV

Commit message: cleanup led driver
Parts:
- added R1: 0, symbol Device:R
- U6: now not fitted
Connections:
- net in: now also R1.1, R1.2
Changed lines of the file:
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@@
+	)
+	(junction
+		(at 156.21 62.23)
+		(diameter 0)
+		(color 0 0 0 0)
+	)
+	(junction
+		(at 163.83 62.23)
+		(diameter 0)
+		(color 0 0 0 0)
 	)
 	(junction
@@
 	(wire
 		(pts
-			(xy 151.13 62.23) (xy 170.18 62.23)
+			(xy 156.21 62.23) (xy 163.83 62.23)
+		)
+		(stroke
+			(width 0)
+			(type default)
+		)
+	)
+	(wire
+		(pts
+			(xy 163.83 62.23) (xy 170.18 62.23)
 		)
 		(stroke
@@
 		(pts
 			(xy 143.51 111.76) (xy 143.51 114.3)
+		)
+		(stroke
+			(width 0)
+			(type default)
+		)
+	)
+	(wire
+		(pts
+			(xy 151.13 62.23) (xy 156.21 62.23)
 		)
 		(stroke
@@
 		(dnp yes)
 		(property "Reference" "Q1"
-			(at 158.75 57.15 90)
+			(at 164.084 65.532 90)
 			(effects
 				(font
@@
 		)
 		(property "Value" "BSS138"
-			(at 158.75 59.69 90)
+			(at 158.242 65.278 90)
 			(effects
 				(font
@@
 		(in_bom yes)
 		(on_board yes)
-		(dnp no)
+		(dnp yes)
 		(fields_autoplaced yes)
 		(property "Reference" "U6"
@@
 					(unit 1)
 				)
+			)
+		)
+	)
+	(symbol
+		(lib_id "Device:R")
+		(at 160.02 62.23 270)
+		(unit 1)
+		(exclude_from_sim no)
+		(in_bom yes)
+		(on_board yes)
+		(dnp yes)
+		(fields_autoplaced yes)
+		(property "Reference" "R1"
+			(at 160.02 55.88 90)
+			(effects
+				(font
+					(size 1.27 1.27)
+				)
+			)
+		)
+		(property "Value" "0"
+			(at 160.02 58.42 90)
+			(effects
+				(font
+					(size 1.27 1.27)
+				)
+			)
+		)
+		(property "Footprint" ""
+			(at 160.02 60.452 90)
+			(effects
+				(font
+					(size 1.27 1.27)
+				)
+				(hide yes)
+			)
+		)
+		(property "Datasheet" "~"
+			(at 160.02 62.23 0)
+			(effects
+				(font
+					(size 1.27 1.27)
+				)
+				(hide yes)
+			)
+		)
+		(property "Description" "Resistor"
+			(at 160.02 62.23 0)
+			(effects
+				(font
+					(size 1.27 1.27)
+				)
+				(hide yes)
+			)
+		)
+		(pin "1"
+		)
+		(pin "2"
+		)
+		(instances
+			(project ""
+				(path "/1501dcbd-05c1-4298-b373-c91a1b0991c0/81d46fee-d0bf-42e9-8f0a-4693b92a3414"
+					(reference "R1")
+					(unit 1)
+				)
