File: hardware/pcbs/motion_pcb/led_button_h.kicad_sch (KiCad schematic)
At the start: 3 parts

Commit message: changing labels
Parts:
- removed R3: 100, symbol Device:R
- renumbered D1 to D9, R4 to R22
Connections:
- net SW: now also D9.5 (sw1), R22.2
