File: hardware/pcbs/motion_pcb/motion_pcb.kicad_pcb (KiCad board)
At the start: 2 copper layers, 125 x 163 mm, 124 parts, among them J1 esp_io_shield1, J2 esp_io_shield2, J3 esp32_voltage_shield, J4 Con_top_pcb, J5 con_rpi, Q1 BSS138, U1 74HC4051, U11 touch_but_square, U12 touch_but_square, U13 touch_but_square, U14 touch_but_square, U15 touch_but_square, U16 touch_but_square, U17 touch_but_square, U18 touch_but_square, U22 touch_but_square, U23 touch_but_square, U24 touch_but_square, U25 touch_but_square, U26 touch_but_square, U27 touch_but_square, U28 touch_but_square, U29 touch_but_square, U3 74HC4051, U32 touch_but_round, U33 touch_but_round, U34 touch_but_round, U4 74HC4051, U5 74AHCT125

Commit message: changing labels
Parts:
- removed the J3 at (201.8, 62.1)
- removed the J3 at (39.0, 32.0)
- removed the J4 at (202.5, 55.9)
- removed the J4 at (39.0, 164.0)
- removed J5: con_rpi, Connector_JST:JST_PH_B6B-PH-K_1x06_P2.00mm_Vertical
- removed J5: con_rpi, Connector_JST:JST_PH_B9B-PH-K_1x09_P2.00mm_Vertical
- removed MT1, MT2, MT3, MT4: PEC11R-4215F-S0024, 3dAudioFoot:XDCR_PEC11R-4215F-S0024
- removed R101, R96, R98: 10K, Resistor_SMD:R_1206_3216Metric
- removed R111: 1k, Resistor_SMD:R_1206_3216Metric
- added C10: 100nF, Capacitor_SMD:C_1206_3216Metric_Pad1.33x1.80mm_HandSolder, B.Cu at (138.0, 80.1)
- added C11: 100nF, Capacitor_SMD:C_1206_3216Metric_Pad1.33x1.80mm_HandSolder, B.Cu at (148.4, 69.1)
- added C12: 100nF, Capacitor_SMD:C_1206_3216Metric_Pad1.33x1.80mm_HandSolder, B.Cu at (195.2, 108.7)
- added C20: 100nF, Capacitor_SMD:C_1206_3216Metric_Pad1.33x1.80mm_HandSolder, B.Cu at (212.3, 80.1)
- added C22: 100nF, Capacitor_SMD:C_1206_3216Metric_Pad1.33x1.80mm_HandSolder, B.Cu at (214.2, 137.2)
- added C23: 100nF, Capacitor_SMD:C_1206_3216Metric_Pad1.33x1.80mm_HandSolder, B.Cu at (224.6, 126.2)
- added C24: 100nF, Capacitor_SMD:C_1206_3216Metric_Pad1.33x1.80mm_HandSolder, B.Cu at (244.2, 166.4)
- added C25: 100nF, Capacitor_SMD:C_1206_3216Metric_Pad1.33x1.80mm_HandSolder, B.Cu at (167.1, 166.8)
- added C26: 100nF, Capacitor_SMD:C_1206_3216Metric_Pad1.33x1.80mm_HandSolder, B.Cu at (271.4, 108.7)
- added C27: 100nF, Capacitor_SMD:C_1206_3216Metric_Pad1.33x1.80mm_HandSolder, B.Cu at (281.8, 97.7)
- added C28: 100nF, Capacitor_SMD:C_1206_3216Metric_Pad1.33x1.80mm_HandSolder, B.Cu at (129.0, 167.3)
- added C29: 100nF, Capacitor_SMD:C_1206_3216Metric_Pad1.33x1.80mm_HandSolder, B.Cu at (282.4, 166.5)
- added C30: 100nF, Capacitor_SMD:C_1206_3216Metric_Pad1.33x1.80mm_HandSolder, F.Cu at (153.1, -14.7)
- added C31: 100nF, Capacitor_SMD:C_1206_3216Metric_Pad1.33x1.80mm_HandSolder, F.Cu at (153.1, -11.3)
- added C32: 100nF, Capacitor_SMD:C_1206_3216Metric_Pad1.33x1.80mm_HandSolder, F.Cu at (153.1, -7.98)
- added C33: 100nF, Capacitor_SMD:C_1206_3216Metric_Pad1.33x1.80mm_HandSolder, B.Cu at (205.4, 166.5)
- added C35: 100nF, Capacitor_SMD:C_1206_3216Metric_Pad1.33x1.80mm_HandSolder, F.Cu at (79.9, 77.2)
- added C36: 100nF, Capacitor_SMD:C_1206_3216Metric_Pad1.33x1.80mm_HandSolder, F.Cu at (79.9, 80.5)
- added C7: 100nF, Capacitor_SMD:C_1206_3216Metric_Pad1.33x1.80mm_HandSolder, B.Cu at (186.5, 69.1)
- added C8: 100nF, Capacitor_SMD:C_1206_3216Metric_Pad1.33x1.80mm_HandSolder, B.Cu at (176.1, 137.2)
- added C9: 100nF, Capacitor_SMD:C_1206_3216Metric_Pad1.33x1.80mm_HandSolder, B.Cu at (186.5, 126.3)
- added D20: WS2812B-2020, 3dAudioFoot:A3_CherryMxHybrid_WS2812Led2020, F.Cu at (218.4, 190.6)
- added D21: WS2812B-2020, 3dAudioFoot:A3_CherryMxHybrid_WS2812Led2020, F.Cu at (218.4, 209.6)
- added D22: WS2812B-2020, 3dAudioFoot:A3_CherryMxHybrid_WS2812Led2020, F.Cu at (161.3, 171.5)
- added D23: WS2812B-2020, 3dAudioFoot:A3_CherryMxHybrid_WS2812Led2020, F.Cu at (161.3, 190.6)
- added D24: WS2812B-2020, 3dAudioFoot:A3_CherryMxHybrid_WS2812Led2020, F.Cu at (161.3, 209.6)
- added D25: WS2812B-2020, 3dAudioFoot:A3_CherryMxHybrid_WS2812Led2020, F.Cu at (180.3, 171.5)
- added D26: WS2812B-2020, 3dAudioFoot:A3_CherryMxHybrid_WS2812Led2020, F.Cu at (180.3, 190.6)
- added D27: WS2812B-2020, 3dAudioFoot:A3_CherryMxHybrid_WS2812Led2020, F.Cu at (180.3, 209.6)
- added D28: WS2812B-2020, 3dAudioFoot:A3_CherryMxHybrid_WS2812Led2020, F.Cu at (123.2, 171.5)
- added D29: WS2812B-2020, 3dAudioFoot:A3_CherryMxHybrid_WS2812Led2020, F.Cu at (123.2, 190.6)
- added D30: WS2812B-2020, 3dAudioFoot:A3_CherryMxHybrid_WS2812Led2020, F.Cu at (123.2, 209.6)
- added D31: WS2812B-2020, 3dAudioFoot:A3_CherryMxHybrid_WS2812Led2020, F.Cu at (123.2, 152.4)
- added D32: WS2812B-2020, 3dAudioFoot:A3_CherryMxHybrid_WS2812Led2020, F.Cu at (142.2, 171.5)
- added D33: WS2812B-2020, 3dAudioFoot:A3_CherryMxHybrid_WS2812Led2020, F.Cu at (142.2, 190.6)
- added D34: WS2812B-2020, 3dAudioFoot:A3_CherryMxHybrid_WS2812Led2020, F.Cu at (142.2, 209.6)
- added D35: WS2812B-2020, 3dAudioFoot:A3_CherryMxHybrid_WS2812Led2020, F.Cu at (275.6, 152.4)
- added D36: WS2812B-2020, 3dAudioFoot:A3_CherryMxHybrid_WS2812Led2020, F.Cu at (256.6, 152.4)
- added D37: WS2812B-2020, 3dAudioFoot:A3_CherryMxHybrid_WS2812Led2020, F.Cu at (237.5, 152.4)
- added D38: WS2812B-2020, 3dAudioFoot:A3_CherryMxHybrid_WS2812Led2020, F.Cu at (218.4, 152.4)
- added D39: WS2812B-2020, 3dAudioFoot:A3_CherryMxHybrid_WS2812Led2020, F.Cu at (123.2, 114.3)
- added D40: WS2812B-2020, 3dAudioFoot:A3_CherryMxHybrid_WS2812Led2020, F.Cu at (199.4, 152.4)
- added D41: WS2812B-2020, 3dAudioFoot:A3_CherryMxHybrid_WS2812Led2020, F.Cu at (123.2, 133.4)
- added D42: WS2812B-2020, 3dAudioFoot:A3_CherryMxHybrid_WS2812Led2020, F.Cu at (180.3, 152.4)
- added D43: WS2812B-2020, 3dAudioFoot:A3_CherryMxHybrid_WS2812Led2020, F.Cu at (161.3, 152.4)
- added D44: WS2812B-2020, 3dAudioFoot:A3_CherryMxHybrid_WS2812Led2020, F.Cu at (142.2, 152.4)
- added IC1: ~, 3dAudioFoot:ESP32-S3-DevKitC-1, F.Cu at (202.6, 49.4)
- added J3: Conn_02x16_Odd_Even, Connector_PinHeader_2.54mm:PinHeader_2x16_P2.54mm_Vertical, F.Cu at (362.2, 56.3)
- added J4: Conn_02x01, Connector_PinHeader_2.54mm:PinHeader_1x02_P2.54mm_Vertical, F.Cu at (376.5, 75.3)
- added R10: 1k, Resistor_SMD:R_1206_3216Metric_Pad1.30x1.75mm_HandSolder, B.Cu at (135.3, 140.2)
- added R11: 1k, Resistor_SMD:R_1206_3216Metric_Pad1.30x1.75mm_HandSolder, B.Cu at (148.4, 129.4)
- added R12: 10k, Resistor_SMD:R_1206_3216Metric_Pad1.30x1.75mm_HandSolder, B.Cu at (269.4, 165.4)
- added R13: 10k, Resistor_SMD:R_1206_3216Metric_Pad1.30x1.75mm_HandSolder, B.Cu at (269.4, 184.5)
- added R14: 10k, Resistor_SMD:R_1206_3216Metric_Pad1.30x1.75mm_HandSolder, B.Cu at (269.4, 203.6)
- added R15: 10k, Resistor_SMD:R_1206_3216Metric_Pad1.30x1.75mm_HandSolder, B.Cu at (193.2, 165.4)
- added R16: 10k, Resistor_SMD:R_1206_3216Metric_Pad1.30x1.75mm_HandSolder, B.Cu at (193.2, 184.5)
- added R17: 10k, Resistor_SMD:R_1206_3216Metric_Pad1.30x1.75mm_HandSolder, B.Cu at (155.1, 97.9)
- added R18: 10K, Resistor_SMD:R_1206_3216Metric_Pad1.30x1.75mm_HandSolder, B.Cu at (158.6, 100.9)
- added R19: 10K, Resistor_SMD:R_1206_3216Metric_Pad1.30x1.75mm_HandSolder, B.Cu at (166.5, 110.5)
- added R20: 1k, Resistor_SMD:R_1206_3216Metric_Pad1.30x1.75mm_HandSolder, B.Cu at (154.6, 111.8)
- added R21: 1k, Resistor_SMD:R_1206_3216Metric_Pad1.30x1.75mm_HandSolder, B.Cu at (167.7, 101.0)
- added R22: 10k, Resistor_SMD:R_1206_3216Metric_Pad1.30x1.75mm_HandSolder, B.Cu at (250.4, 165.4)
- added R23: 10k, Resistor_SMD:R_1206_3216Metric_Pad1.30x1.75mm_HandSolder, B.Cu at (250.4, 184.5)
- added R24: 10k, Resistor_SMD:R_1206_3216Metric_Pad1.30x1.75mm_HandSolder, B.Cu at (250.4, 203.6)
- added R25: 10k, Resistor_SMD:R_1206_3216Metric_Pad1.30x1.75mm_HandSolder, B.Cu at (231.3, 165.4)
- added R26: 10k, Resistor_SMD:R_1206_3216Metric_Pad1.30x1.75mm_HandSolder, B.Cu at (231.3, 184.5)
- added R27: 10k, Resistor_SMD:R_1206_3216Metric_Pad1.30x1.75mm_HandSolder, B.Cu at (231.3, 203.6)
- added R28: 10k, Resistor_SMD:R_1206_3216Metric_Pad1.30x1.75mm_HandSolder, B.Cu at (173.9, 69.1)
- added R29: 10K, Resistor_SMD:R_1206_3216Metric_Pad1.30x1.75mm_HandSolder, B.Cu at (177.4, 72.1)
- added R30: 10K, Resistor_SMD:R_1206_3216Metric_Pad1.30x1.75mm_HandSolder, B.Cu at (185.3, 81.7)
- added R31: 1k, Resistor_SMD:R_1206_3216Metric_Pad1.30x1.75mm_HandSolder, B.Cu at (173.4, 83.0)
- added R32: 1k, Resistor_SMD:R_1206_3216Metric_Pad1.30x1.75mm_HandSolder, B.Cu at (186.5, 72.2)
- added R33: 10k, Resistor_SMD:R_1206_3216Metric_Pad1.30x1.75mm_HandSolder, B.Cu at (173.9, 126.3)
- added R34: 10K, Resistor_SMD:R_1206_3216Metric_Pad1.30x1.75mm_HandSolder, B.Cu at (177.4, 129.2)
- added R35: 10K, Resistor_SMD:R_1206_3216Metric_Pad1.30x1.75mm_HandSolder, B.Cu at (185.3, 138.8)
- added R36: 1k, Resistor_SMD:R_1206_3216Metric_Pad1.30x1.75mm_HandSolder, B.Cu at (173.4, 140.1)
- added R37: 1k, Resistor_SMD:R_1206_3216Metric_Pad1.30x1.75mm_HandSolder, B.Cu at (186.5, 129.3)
- added R38: 10k, Resistor_SMD:R_1206_3216Metric_Pad1.30x1.75mm_HandSolder, B.Cu at (212.3, 165.4)
- added R39: 10k, Resistor_SMD:R_1206_3216Metric_Pad1.30x1.75mm_HandSolder, B.Cu at (193.2, 203.6)
- added R40: 10k, Resistor_SMD:R_1206_3216Metric_Pad1.30x1.75mm_HandSolder, B.Cu at (135.8, 69.1)
- added R41: 10K, Resistor_SMD:R_1206_3216Metric_Pad1.30x1.75mm_HandSolder, B.Cu at (139.3, 72.1)
- added R42: 10K, Resistor_SMD:R_1206_3216Metric_Pad1.30x1.75mm_HandSolder, B.Cu at (147.2, 81.7)
- added R43: 1k, Resistor_SMD:R_1206_3216Metric_Pad1.30x1.75mm_HandSolder, B.Cu at (135.3, 83.0)
- added R44: 1k, Resistor_SMD:R_1206_3216Metric_Pad1.30x1.75mm_HandSolder, B.Cu at (148.4, 72.2)
- added R45: 10k, Resistor_SMD:R_1206_3216Metric_Pad1.30x1.75mm_HandSolder, B.Cu at (212.3, 184.5)
- added R46: 10k, Resistor_SMD:R_1206_3216Metric_Pad1.30x1.75mm_HandSolder, B.Cu at (212.3, 203.6)
- added R47: 10k, Resistor_SMD:R_1206_3216Metric_Pad1.30x1.75mm_HandSolder, B.Cu at (193.0, 97.7)
- added R48: 10K, Resistor_SMD:R_1206_3216Metric_Pad1.30x1.75mm_HandSolder, B.Cu at (196.5, 100.7)
- added R49: 10K, Resistor_SMD:R_1206_3216Metric_Pad1.30x1.75mm_HandSolder, B.Cu at (204.4, 110.3)
- added R50: 1k, Resistor_SMD:R_1206_3216Metric_Pad1.30x1.75mm_HandSolder, B.Cu at (192.5, 111.6)
- added R51: 1k, Resistor_SMD:R_1206_3216Metric_Pad1.30x1.75mm_HandSolder, B.Cu at (205.6, 100.8)
- added R52: 10k, Resistor_SMD:R_1206_3216Metric_Pad1.30x1.75mm_HandSolder, B.Cu at (155.1, 165.4)
- added R53: 10k, Resistor_SMD:R_1206_3216Metric_Pad1.30x1.75mm_HandSolder, B.Cu at (155.1, 184.5)
- added R54: 10k, Resistor_SMD:R_1206_3216Metric_Pad1.30x1.75mm_HandSolder, B.Cu at (155.1, 203.6)
- added R55: 10k, Resistor_SMD:R_1206_3216Metric_Pad1.30x1.75mm_HandSolder, B.Cu at (248.9, 69.1)
- added R56: 10K, Resistor_SMD:R_1206_3216Metric_Pad1.30x1.75mm_HandSolder, B.Cu at (252.4, 72.1)
- added R57: 10K, Resistor_SMD:R_1206_3216Metric_Pad1.30x1.75mm_HandSolder, B.Cu at (260.3, 81.7)
- added R58: 1k, Resistor_SMD:R_1206_3216Metric_Pad1.30x1.75mm_HandSolder, B.Cu at (248.4, 83.0)
- added R59: 1k, Resistor_SMD:R_1206_3216Metric_Pad1.30x1.75mm_HandSolder, B.Cu at (261.5, 72.2)
- added R60: 10k, Resistor_SMD:R_1206_3216Metric_Pad1.30x1.75mm_HandSolder, B.Cu at (174.2, 165.4)
- added R61: 10k, Resistor_SMD:R_1206_3216Metric_Pad1.30x1.75mm_HandSolder, B.Cu at (174.2, 184.5)
- added R62: 10k, Resistor_SMD:R_1206_3216Metric_Pad1.30x1.75mm_HandSolder, B.Cu at (174.2, 203.6)
- added R63: 10k, Resistor_SMD:R_1206_3216Metric_Pad1.30x1.75mm_HandSolder, B.Cu at (250.1, 126.2)
- added R64: 10K, Resistor_SMD:R_1206_3216Metric_Pad1.30x1.75mm_HandSolder, B.Cu at (253.6, 129.2)
- added R65: 10K, Resistor_SMD:R_1206_3216Metric_Pad1.30x1.75mm_HandSolder, B.Cu at (261.5, 138.8)
- added R66: 1k, Resistor_SMD:R_1206_3216Metric_Pad1.30x1.75mm_HandSolder, B.Cu at (249.6, 140.1)
- added R67: 1k, Resistor_SMD:R_1206_3216Metric_Pad1.30x1.75mm_HandSolder, B.Cu at (262.7, 129.3)
- added R68: 10k, Resistor_SMD:R_1206_3216Metric_Pad1.30x1.75mm_HandSolder, B.Cu at (117.0, 165.4)
- added R69: 10k, Resistor_SMD:R_1206_3216Metric_Pad1.30x1.75mm_HandSolder, B.Cu at (117.0, 184.5)
- added R70: 10k, Resistor_SMD:R_1206_3216Metric_Pad1.30x1.75mm_HandSolder, B.Cu at (117.0, 203.6)
- added R71: 10k, Resistor_SMD:R_1206_3216Metric_Pad1.30x1.75mm_HandSolder, B.Cu at (117.0, 146.4)
- added R72: 10k, Resistor_SMD:R_1206_3216Metric_Pad1.30x1.75mm_HandSolder, B.Cu at (231.1, 97.7)
- added U10: ~, 3dAudioFoot:a3_jumper_fix, B.Cu at (171.8, 73.8)
- added U19: ~, 3dAudioFoot:a3_jumper_fix, B.Cu at (150.6, 82.0)
- added U20: ~, 3dAudioFoot:a3_jumper_fix, B.Cu at (135.6, 85.9)
- added U21: ~, 3dAudioFoot:A3_ENC_POT_mix, F.Cu at (199.2, 104.7)
- added U30: ~, 3dAudioFoot:a3_jumper_fix, B.Cu at (248.0, 130.9)
- added U31: ~, 3dAudioFoot:a3_jumper_fix, B.Cu at (264.9, 139.1)
- added U35: ~, 3dAudioFoot:a3_jumper_fix, B.Cu at (245.9, 110.6)
- added U36: ~, 3dAudioFoot:a3_jumper_fix, B.Cu at (230.9, 114.5)
- added U37: ~, 3dAudioFoot:A3_ENC_POT_mix, F.Cu at (216.4, 76.1)
- added U38: ~, 3dAudioFoot:a3_jumper_fix, B.Cu at (208.0, 73.8)
- added U39: ~, 3dAudioFoot:a3_jumper_fix, B.Cu at (224.9, 82.0)
- added U40: ~, 3dAudioFoot:a3_jumper_fix, B.Cu at (209.9, 85.9)
- added U41: ~, 3dAudioFoot:A3_ENC_POT_mix, F.Cu at (218.3, 133.2)
- added U42: SN74LVC1T45DBV, Package_TO_SOT_SMD:SOT-23-6, F.Cu at (164.1, 47.1)
- added U43: 74HC4051, Package_SO:SOIC-16_3.9x9.9mm_P1.27mm, B.Cu at (243.2, 178.6)
- added U44: ~, 3dAudioFoot:a3_jumper_fix, B.Cu at (209.9, 130.9)
- added U45: ~, 3dAudioFoot:a3_jumper_fix, B.Cu at (226.8, 139.1)
- added U46: ~, 3dAudioFoot:a3_jumper_fix, B.Cu at (211.8, 143.0)
- added U47: 74HC4051, Package_SO:SOIC-16_3.9x9.9mm_P1.27mm, B.Cu at (167.3, 178.4)
- added U48: 74HC4051, Package_SO:SOIC-16_3.9x9.9mm_P1.27mm, B.Cu at (129.0, 178.6)
- added U49: ~, 3dAudioFoot:A3_ENC_POT_mix, F.Cu at (275.5, 104.7)
- added U50: ~, 3dAudioFoot:a3_jumper_fix, B.Cu at (267.1, 102.4)
- added U51: ~, 3dAudioFoot:a3_jumper_fix, B.Cu at (284.0, 110.6)
- added U52: ~, 3dAudioFoot:a3_jumper_fix, B.Cu at (269.0, 114.5)
- added U53: 74HC4051, Package_SO:SOIC-16_3.9x9.9mm_P1.27mm, B.Cu at (280.1, 178.6)
- added U54: 74HC4051, Package_SO:SOIC-16_3.9x9.9mm_P1.27mm, B.Cu at (180.3, 114.4)
- added U55: 74HC4051, Package_SO:SOIC-16_3.9x9.9mm_P1.27mm, B.Cu at (142.1, 114.4)
- added U56: 74HC4051, Package_SO:SOIC-16_3.9x9.9mm_P1.27mm, B.Cu at (256.6, 114.4)
- added U57: 74HC4051, Package_SO:SOIC-16_3.9x9.9mm_P1.27mm, B.Cu at (205.3, 178.6)
- added U59: 74HC4051, Package_SO:SOIC-16_3.9x9.9mm_P1.27mm, F.Cu at (161.3, 86.9)
- added U6: ~, 3dAudioFoot:a3_jumper_fix, B.Cu at (153.0, 102.6)
- added U60: 74HC4051, Package_SO:SOIC-16_3.9x9.9mm_P1.27mm, F.Cu at (237.5, 86.9)
- added U7: ~, 3dAudioFoot:a3_jumper_fix, B.Cu at (169.9, 110.8)
- added U8: ~, 3dAudioFoot:a3_jumper_fix, B.Cu at (154.9, 114.7)
- added U9: ~, 3dAudioFoot:A3_ENC_POT_mix, F.Cu at (180.2, 76.1)
- C1: value 100nF -> 10v/1mF; footprint Capacitor_SMD:C_1206_3216Metric_Pad1.33x1.80mm_HandSolder -> Capacitor_SMD:CP_Elec_10x10
- C2, C3, C4, C6: moved to B.Cu
- C5: value 10v/1mF -> 100nF; footprint Capacitor_SMD:CP_Elec_10x10 -> Capacitor_SMD:C_1206_3216Metric_Pad1.33x1.80mm_HandSolder; moved to B.Cu
- D1, D10, D11, D12, D13, D14, D15, D16, D17, D18, D19, D2, D3, D4, D5, D6, D7, D8, D9: footprint LED_SMD:LED_WS2812B-2020_PLCC4_2.0x2.0mm -> 3dAudioFoot:A3_CherryMxHybrid_WS2812Led2020
- J1: value esp_io_shield1 -> Conn_02x02_Odd_Even; footprint Connector_PinHeader_2.54mm:PinHeader_2x07_P2.54mm_Vertical_SMD -> Connector_PinHeader_2.54mm:PinHeader_2x02_P2.54mm_Vertical
- J2: value esp_io_shield2 -> Conn_02x06_Odd_Even; footprint Connector_PinHeader_2.54mm:PinHeader_2x11_P2.54mm_Vertical_SMD -> Connector_PinHeader_2.54mm:PinHeader_2x06_P2.54mm_Vertical
- R1, R2, R3, R4, R6, R7: value 100 -> 10k; moved to B.Cu
- R100, R106: value 1k -> 10k; footprint Resistor_SMD:R_1206_3216Metric -> Resistor_SMD:R_1206_3216Metric_Pad1.30x1.75mm_HandSolder
- R102, R103, R104, R109, R110, R73, R74, R90, R91: footprint Resistor_SMD:R_1206_3216Metric -> Resistor_SMD:R_1206_3216Metric_Pad1.30x1.75mm_HandSolder
- R105, R75, R76, R92, R93: value 10K -> 1k; footprint Resistor_SMD:R_1206_3216Metric -> Resistor_SMD:R_1206_3216Metric_Pad1.30x1.75mm_HandSolder
- R107, R108: value 1k -> 10K; footprint Resistor_SMD:R_1206_3216Metric -> Resistor_SMD:R_1206_3216Metric_Pad1.30x1.75mm_HandSolder
- R5: value 1k -> 10k; moved to B.Cu
- R77, R78, R79, R80, R81, R82, R83, R84, R85, R86, R87, R88, R89, R94: value 10K -> 10k; footprint Resistor_SMD:R_1206_3216Metric -> Resistor_SMD:R_1206_3216Metric_Pad1.30x1.75mm_HandSolder
- R8: value 100 -> 10K; moved to B.Cu
- R9: value 10k -> 10K; moved to B.Cu
- R95: value 10K -> 1k; footprint Resistor_SMD:R_1206_3216Metric -> Resistor_SMD:R_1206_3216Metric_Pad1.30x1.75mm_HandSolder; moved to F.Cu
- R97: value 10K -> 10k; footprint Resistor_SMD:R_1206_3216Metric -> Resistor_SMD:R_1206_3216Metric_Pad1.30x1.75mm_HandSolder; moved to F.Cu
- R99: value 10K -> 0; footprint Resistor_SMD:R_1206_3216Metric -> Resistor_SMD:R_1206_3216Metric_Pad1.30x1.75mm_HandSolder; moved to F.Cu
- U1: value 74HC4051 -> ~; footprint Package_SO:SOIC-16_3.9x9.9mm_P1.27mm -> 3dAudioFoot:A3_ENC_POT_mix
- U11, U12, U14, U15, U16, U18, U22, U23, U24, U26, U27, U28: value touch_but_square -> ~; footprint 3dAudioFoot:But_Velo_Rec_1 -> 3dAudioFoot:a3_jumper_fix; moved to B.Cu
- U13, U17, U25, U29: value touch_but_square -> ~; footprint 3dAudioFoot:But_Velo_Rec_1 -> 3dAudioFoot:A3_ENC_POT_mix
- U2: footprint esp32:DFR0645 -> 3dAudioFoot:a3_jumper_fix
- U3, U4: value 74HC4051 -> ~; footprint Package_SO:SOIC-16_3.9x9.9mm_P1.27mm -> 3dAudioFoot:a3_jumper_fix; moved to B.Cu
- U32, U34: value touch_but_round -> ~; footprint 3dAudioFoot:But_Velo_Rnd_1 -> 3dAudioFoot:a3_jumper_fix; moved to B.Cu
- U33: value touch_but_round -> ~; footprint 3dAudioFoot:But_Velo_Rnd_1 -> 3dAudioFoot:A3_ENC_POT_mix
- U5: value 74AHCT125 -> ~; footprint Capacitor_SMD:CP_Elec_10x10 -> 3dAudioFoot:A3_ENC_POT_mix
- moved H4 331.6 mm to (371.9, 50.0)
- moved H3 254.8 mm to (291.3, 43.1)
- moved R106 218.7 mm to (269.2, 97.7)
- moved H5 217.7 mm to (199.9, 123.8)
- moved R110 211.2 mm to (281.8, 100.8)
- moved R76 199.7 mm to (243.7, 100.8), turned to 0 degrees
- moved D6 196.2 mm to (294.6, 209.6)
- moved C15 191.6 mm to (261.5, 69.1)
- moved R104 188.1 mm to (211.5, 140.1), turned to 180 degrees
- moved U27 187.0 mm to (263.7, 82.0), turned to 180 degrees
- moved C16 185.6 mm to (252.3, 137.2), turned to 180 degrees
- moved R74 185.4 mm to (242.5, 110.3), turned to 90 degrees
- moved R105 185.1 mm to (224.6, 129.3), turned to 0 degrees
- moved R6 183.2 mm to (288.5, 203.6)
- moved U33 182.3 mm to (237.3, 104.7)
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Connections:
- net Net-(D1-DOUT) renamed /LED/LedBut1/LED_OUT
- net Net-(D12-DOUT) renamed /LED/LedBut13/LED_OUT
- net Net-(D13-DOUT) renamed /LED/LedBut14/LED_OUT
- net Net-(D2-DOUT) renamed /LED/LedBut2/LED_OUT
- net Net-(D3-DOUT) renamed /LED/LedBut3/LED_OUT
- net Net-(D4-DOUT) renamed /LED/LedBut4/LED_OUT
- net Net-(D5-DOUT) renamed /LED/LedBut5/LED_OUT
- C1 pad 1: +3V3 -> +5V
- C13 pad 1: EA1 -> /poti_arr/EB14
- C14 pad 1: EA3 -> POT_H
- C15 pad 1: EA2 -> /poti_arr/EB07
- C16 pad 1: EB2 -> POT_H
- C17 pad 1: EB3 -> /poti_arr/EB27
- C18 pad 1: EA4 -> POT_H
- C19 pad 1: EB4 -> /poti_arr/EB16
- C2 pad 1: +3V3 -> POT_H
- C21 pad 1: EB1 -> /poti_arr/EB05
- C3 pad 1: +3V3 -> /poti_arr/EB21
- C4 pad 1: MUX_D -> POT_H
- C5 pad 1: +5V -> /poti_arr/EB12
- C6 pad 1: +5V -> POT_H
- D1 pad 3: led_dat -> /LED/LED_DAT
- D10 pad 1: Net-(D10-DOUT) -> /LED/LedBut22/LED_OUT
- D10 pad 3: Net-(D10-DIN) -> /LED/LedBut22/LED_IN
- D11 pad 1: Net-(D11-DOUT) -> /LED/LedBut22/LED_IN
- D11 pad 3: Net-(D10-DOUT) -> /LED/LedBut25/LED_IN
- D12 pad 3: Net-(D11-DOUT) -> /LED/LedBut13/LED_IN
- D14 pad 1: Net-(D14-DOUT) -> /LED/LedBut15/LED_OUT
- D15 pad 1: Net-(D15-DOUT) -> /LED/LedBut16/LED_OUT
- D15 pad 3: Net-(D14-DOUT) -> /LED/LedBut16/LED_IN
- D16 pad 1: dat2 -> /LED/LedBut16/LED_IN
- D16 pad 3: Net-(D15-DOUT) -> /LED/LedBut17/LED_IN
- D17 pad 1: Net-(D17-DOUT) -> /LED/LedBut17/LED_IN
- D17 pad 3: dat2 -> /LED/LedBut15/LED_OUT
- D18 pad 1: Net-(D18-DOUT) -> /LED/LedBut21/LED_OUT
- D18 pad 3: Net-(D17-DOUT) -> /LED/LedBut21/LED_IN
- D19 pad 1: unconnected-(D19-DOUT-Pad1) -> /LED/LedBut25/LED_IN
- D19 pad 3: Net-(D18-DOUT) -> /LED/LedBut24/LED_OUT
- D6 pad 1: Net-(D6-DOUT) -> /LED/LedBut10/LED_IN
- D7 pad 1: Net-(D7-DOUT) -> /LED/LedBut55/LED_IN
- D7 pad 3: Net-(D6-DOUT) -> /LED/LedBut8/LED_IN
- D8 pad 1: dat1 -> /LED/LedBut8/LED_IN
- D8 pad 3: Net-(D7-DOUT) -> /LED/LedBut10/LED_OUT
- D9 pad 1: Net-(D10-DIN) -> /LED/LedBut10/LED_OUT
- D9 pad 3: dat1 -> /LED/LedBut10/LED_IN
- J1 pad 1: EA1 -> +3V3
- J1 pad 2: EA1 -> +3V3
- J1 pad 3: led_dat -> GND
- J1 pad 4: led_dat -> Net-(IC1-RST)
- J2 pad 1: SCL -> MUX_S2
- J2 pad 10: Net-(J2-Pin_10) -> MUX_B
- J2 pad 11: Net-(J2-Pin_11) -> MUX_C
- J2 pad 12: Net-(J2-Pin_11) -> MUX_C
- J2 pad 2: SCL -> MUX_S2
- J2 pad 3: SDA -> MUX_S1
- J2 pad 4: SDA -> MUX_S1
- J2 pad 5: Net-(J2-Pin_5) -> MUX_S0
- J2 pad 6: Net-(J2-Pin_5) -> MUX_S0
- J2 pad 7: Net-(J2-Pin_7) -> MUX_A
- J2 pad 8: Net-(J2-Pin_7) -> MUX_A
- J2 pad 9: Net-(J2-Pin_10) -> MUX_B
- Q1 pad 2: led_dat -> /led_driver/in
- Q1 pad 3: led_dat -> /led_driver/in
- R1 pad 1: MUX_A -> +3V3
- R1 pad 2: Net-(J2-Pin_5) -> /LED/SW00
- R100 pad 1: EA3 -> +3V3
- R100 pad 2: Net-(MT3-PadA) -> /LED/SW28
- R102 pad 2: Net-(MT4-PadA) -> Net-(R102-Pad2)
- R103 pad 2: Net-(MT4-PadB) -> Net-(R103-Pad2)
- R104 pad 1: EA1 -> POT_H
- R104 pad 2: Net-(MT1-PadA) -> Net-(R102-Pad2)
- R105 pad 1: +3V3 -> /poti_arr/EB25
- R105 pad 2: Net-(MT1-PadB) -> Net-(R103-Pad2)
- R106 pad 1: EB1 -> /poti_arr/ES18
- R106 pad 2: Net-(MT1-PadB) -> +3V3
- R107 pad 1: EB3 -> +3V3
- R107 pad 2: Net-(MT3-PadB) -> Net-(R107-Pad2)
- R108 pad 1: EA4 -> +3V3
- R108 pad 2: Net-(MT4-PadA) -> Net-(R108-Pad2)
- R109 pad 1: EB4 -> POT_H
- R109 pad 2: Net-(MT4-PadB) -> Net-(R107-Pad2)
- R110 pad 1: EA2 -> /poti_arr/EB18
- R110 pad 2: Net-(MT2-PadA) -> Net-(R108-Pad2)
- R2 pad 1: MUX_B -> +3V3
- R2 pad 2: Net-(J2-Pin_7) -> /LED/SW10
- R3 pad 1: MUX_C -> +3V3
- R3 pad 2: Net-(J2-Pin_10) -> /LED/SW20
- R4 pad 1: MUX_D -> +3V3
- R4 pad 2: Net-(J2-Pin_11) -> /LED/SW30
- R5 pad 1: +5V -> +3V3
- R5 pad 2: led_dat -> /LED/SW40
- R6 pad 1: Net-(J4-Pin_3) -> +3V3
- R6 pad 2: MUX_S0 -> /LED/SW50
- R7 pad 1: Net-(J4-Pin_4) -> /poti_arr/ES21
- R7 pad 2: MUX_S1 -> +3V3
- R73 pad 2: BUTA1 -> Net-(R73-Pad2)
- R74 pad 2: BUTA2 -> Net-(R74-Pad2)
- R75 pad 1: +3V3 -> POT_H
- R75 pad 2: BUTA3 -> Net-(R73-Pad2)
- R76 pad 1: +3V3 -> /poti_arr/EB16
- R76 pad 2: BUTA4 -> Net-(R74-Pad2)
- R77 pad 2: BUTC1 -> /LED/SW38
- R78 pad 2: BUTC2 -> /LED/SW48
- R79 pad 2: BUTC3 -> /LED/SW58
- R8 pad 1: Net-(J4-Pin_5) -> +3V3
- R8 pad 2: MUX_S2 -> Net-(R10-Pad2)
- R80 pad 2: BUTC4 -> /LED/SW21
- R81 pad 2: BUTB1 -> /LED/SW22
- R82 pad 2: BUTB2 -> /LED/SW23
- R83 pad 2: BUTB3 -> /LED/SW24
- R84 pad 2: BUTB4 -> /LED/SW09
- R85 pad 2: BUTD1 -> /LED/SW25
- R86 pad 2: BUTD2 -> /LED/SW19
- R87 pad 2: BUTD3 -> /LED/SW26
- R88 pad 1: +3V3 -> /poti_arr/ES05
- R88 pad 2: BUTD4 -> +3V3
- R89 pad 2: ES1 -> /LED/SW27
- R9 pad 2: led_dat -> Net-(R11-Pad2)
- R90 pad 2: Net-(MT1-PadA) -> Net-(R90-Pad2)
- R91 pad 2: ES3 -> Net-(R91-Pad2)
- R92 pad 1: +3V3 -> POT_H
- R92 pad 2: ES2 -> Net-(R90-Pad2)
- R93 pad 1: +3V3 -> /poti_arr/EB05
- R93 pad 2: Net-(MT2-PadA) -> Net-(R91-Pad2)
- R94 pad 1: +3V3 -> /poti_arr/ES25
- R94 pad 2: Net-(MT2-PadB) -> +3V3
- R95 pad 1: +3V3 -> +5V
- R95 pad 2: BR1 -> /led_driver/in
- R97 pad 2: BR3 -> /led_driver/in
- R99 pad 1: +3V3 -> /led_driver/in
- R99 pad 2: Net-(MT3-PadB) -> /led_driver/in
Routing:
- net GND: track 0.00 -> 2156.5 mm, vias 0 -> 1
- net +3V3: track 0.00 -> 1201.4 mm
- net +5V: track 0.00 -> 1097.2 mm, vias 0 -> 8
- net /mux/S2: track 0.00 -> 138.2 mm, vias 0 -> 5
- net /mux/S1: track 0.00 -> 128.3 mm, vias 0 -> 5
- net /mux/S0: track 0.00 -> 119.0 mm, vias 0 -> 5
- net POT_H: track 0.00 -> 118.4 mm
- net /mux/A: track 0.00 -> 75.9 mm, vias 0 -> 4
- net /LED/SW53: track 0.00 -> 32.5 mm
- net /LED/SW55: track 0.00 -> 32.1 mm
- net /LED/SW57: track 0.00 -> 32.0 mm
- net /LED/SW23: track 0.00 -> 31.9 mm
- net /LED/SW25: track 0.00 -> 31.9 mm
- net /LED/SW29: track 0.00 -> 31.4 mm
- net /LED/SW27: track 0.00 -> 31.3 mm
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- removed copper zone on B.Cu, net GND
- removed copper zone on F.Cu, net GND
Other:
- board size 125 x 163 mm -> 488.6 x 432.7 mm
- board text added: "E"
- board text added: "P"

Commit message: finished pcb motion.
Parts:
- removed C36: 100nF, Capacitor_SMD:C_1206_3216Metric_Pad1.33x1.80mm_HandSolder
- removed J1: Conn_02x02_Odd_Even, Connector_PinHeader_2.54mm:PinHeader_2x02_P2.54mm_Vertical
- removed J2: Conn_02x06_Odd_Even, Connector_PinHeader_2.54mm:PinHeader_2x06_P2.54mm_Vertical
- removed J3: Conn_02x16_Odd_Even, Connector_PinHeader_2.54mm:PinHeader_2x16_P2.54mm_Vertical
- removed J4: Conn_02x01, Connector_PinHeader_2.54mm:PinHeader_1x02_P2.54mm_Vertical
- removed U60: 74HC4051, Package_SO:SOIC-16_3.9x9.9mm_P1.27mm
- C1, C30, C31, C32, C35, Q1, R95, R97, R99, U42, U59: moved to B.Cu
- moved C32 145.0 mm to (252.6, 97.5), turned to 90 degrees
- moved R95 135.1 mm to (292.7, 62.8), turned to -90 degrees
- moved R97 128.9 mm to (286.1, 68.9), turned to 180 degrees
- moved C30 128.4 mm to (216.0, 97.3), turned to 90 degrees
- moved R99 127.6 mm to (285.9, 60.2)
- moved Q1 123.0 mm to (286.2, 64.6), turned to 90 degrees
- moved U42 122.2 mm to (286.1, 54.4)
- moved C31 116.4 mm to (138.0, 104.1), turned to 90 degrees
- moved C35 78.9 mm to (158.8, 78.7), turned to 90 degrees
- moved U54 39.8 mm to (219.2, 106.0)
- moved H5 13.7 mm to (212.6, 118.9)
- moved U56 8.44 mm to (256.6, 106.0)
- moved IC1 6.83 mm to (208.8, 46.6), turned to -90 degrees
- moved C1 6.57 mm to (136.6, 43.4)
- moved R83 3.17 mm to (215.4, 145.9)
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Connections:
- C10 pad 1: POT_H -> MEA01
- C11 pad 1: /poti_arr/EB01 -> /mux/EB01
- C12 pad 1: POT_H -> MEA14
- C13 pad 1: /poti_arr/EB14 -> /mux/EB14
- C14 pad 1: POT_H -> MEA07
- C15 pad 1: /poti_arr/EB07 -> /mux/EB07
- C16 pad 1: POT_H -> MEA27
- C17 pad 1: /poti_arr/EB27 -> /mux/EB27
- C18 pad 1: POT_H -> MEA16
- C19 pad 1: /poti_arr/EB16 -> /mux/EB16
- C2 pad 1: POT_H -> MEA21
- C20 pad 1: POT_H -> MEA05
- C21 pad 1: /poti_arr/EB05 -> /mux/EB05
- C22 pad 1: POT_H -> MEA25
- C23 pad 1: /poti_arr/EB25 -> /mux/EB25
- C26 pad 1: POT_H -> MEA18
- C27 pad 1: /poti_arr/EB18 -> /mux/EB18
- C3 pad 1: /poti_arr/EB21 -> /mux/EB21
- C4 pad 1: POT_H -> MEA12
- C5 pad 1: /poti_arr/EB12 -> /mux/EB12
- C6 pad 1: POT_H -> MEA03
- C7 pad 1: /poti_arr/EB03 -> /mux/EB03
- C8 pad 1: POT_H -> MEA23
- C9 pad 1: /poti_arr/EB23 -> /mux/EB23
- D1 pad 3: /LED/LED_DAT -> led_dat
- D1 pad 5: /LED/SW00 -> /LED/SW09
- D10 pad 5: /LED/SW35 -> /LED/SW34
- D11 pad 5: /LED/SW45 -> /LED/SW44
- D12 pad 5: /LED/SW32 -> /LED/SW37
- D13 pad 5: /LED/SW42 -> /LED/SW47
- D14 pad 5: /LED/SW52 -> /LED/SW57
- D15 pad 5: /LED/SW33 -> /LED/SW36
- D16 pad 5: /LED/SW43 -> /LED/SW46
- D17 pad 5: /LED/SW53 -> /LED/SW56
- D18 pad 5: /LED/SW34 -> /LED/SW35
- D19 pad 5: /LED/SW55 -> /LED/SW54
- D2 pad 5: /LED/SW10 -> /LED/SW19
- D20 pad 5: /LED/SW44 -> /LED/SW45
- D21 pad 5: /LED/SW54 -> /LED/SW55
- D22 pad 5: /LED/SW37 -> /LED/SW32
- D23 pad 5: /LED/SW47 -> /LED/SW42
- D24 pad 5: /LED/SW57 -> /LED/SW52
- D25 pad 5: /LED/SW36 -> /LED/SW33
- D26 pad 5: /LED/SW46 -> /LED/SW43
- D27 pad 5: /LED/SW56 -> /LED/SW53
- D28 pad 5: /LED/SW39 -> /LED/SW30
- D29 pad 5: /LED/SW49 -> /LED/SW40
- D3 pad 5: /LED/SW20 -> /LED/SW29
- D30 pad 5: /LED/SW59 -> /LED/SW50
- D31 pad 5: /LED/SW29 -> /LED/SW20
- D32 pad 5: /LED/SW38 -> /LED/SW31
- D33 pad 5: /LED/SW48 -> /LED/SW41
- D34 pad 5: /LED/SW58 -> /LED/SW51
- D35 pad 5: /LED/SW21 -> /LED/SW28
- D36 pad 5: /LED/SW22 -> /LED/SW27
- D37 pad 5: /LED/SW23 -> /LED/SW26
- D38 pad 5: /LED/SW24 -> /LED/SW25
- D39 pad 5: /LED/SW09 -> /LED/SW00
- D4 pad 5: /LED/SW30 -> /LED/SW39
- D40 pad 5: /LED/SW25 -> /LED/SW24
- D41 pad 5: /LED/SW19 -> /LED/SW10
- D42 pad 5: /LED/SW26 -> /LED/SW23
- D43 pad 5: /LED/SW27 -> /LED/SW22
- D44 pad 5: /LED/SW28 -> /LED/SW21
- D5 pad 5: /LED/SW40 -> /LED/SW49
- D6 pad 5: /LED/SW50 -> /LED/SW59
- D7 pad 5: /LED/SW31 -> /LED/SW38
- D8 pad 5: /LED/SW41 -> /LED/SW48
- D9 pad 5: /LED/SW51 -> /LED/SW58
- IC1 pad 10: PT23 -> MEA07
- IC1 pad 11: PT13 -> MC
- IC1 pad 12: PT12 -> MEA14
- IC1 pad 13: PT22 -> MEA05
- IC1 pad 15: EA2 -> MEA03
- IC1 pad 16: EB2 -> MB
- IC1 pad 17: PT11 -> MEA23
- IC1 pad 18: PT21 -> MEA21
- IC1 pad 19: EA1 -> MEA12
- IC1 pad 20: EB1 -> MEA01
- IC1 pad 3: Net-(IC1-RST) -> GND
- IC1 pad 4: EA4 -> led_dat
- IC1 pad 5: EB4 -> MEA18
- IC1 pad 6: PT24 -> MEA27
- IC1 pad 7: PT14 -> MEA25
- IC1 pad 8: EA3 -> MEA16
- IC1 pad 9: EB3 -> MD
- Q1 pad 2: /led_driver/in -> led_dat
- Q1 pad 3: /led_driver/in -> led_dat
- R1 pad 2: /LED/SW00 -> /LED/SW09
- R10 pad 1: POT_H -> MEA21
- R100 pad 2: /LED/SW28 -> /LED/SW21
- R104 pad 1: POT_H -> MEA25
- R105 pad 1: /poti_arr/EB25 -> /mux/EB25
- R106 pad 1: /poti_arr/ES18 -> /mux/ES18
- R109 pad 1: POT_H -> MEA18
- R11 pad 1: /poti_arr/EB21 -> /mux/EB21
- R110 pad 1: /poti_arr/EB18 -> /mux/EB18
- R12 pad 2: /LED/SW31 -> /LED/SW38
- R13 pad 2: /LED/SW41 -> /LED/SW48
- R14 pad 2: /LED/SW51 -> /LED/SW58
- R15 pad 2: /LED/SW35 -> /LED/SW34
- R16 pad 2: /LED/SW45 -> /LED/SW44
- R17 pad 1: /poti_arr/ES12 -> /mux/ES12
- R2 pad 2: /LED/SW10 -> /LED/SW19
- R20 pad 1: POT_H -> MEA12
- R21 pad 1: /poti_arr/EB12 -> /mux/EB12
- R22 pad 2: /LED/SW32 -> /LED/SW37
- R23 pad 2: /LED/SW42 -> /LED/SW47
- R24 pad 2: /LED/SW52 -> /LED/SW57
- R25 pad 2: /LED/SW33 -> /LED/SW36
- R26 pad 2: /LED/SW43 -> /LED/SW46
- R27 pad 2: /LED/SW53 -> /LED/SW56
- R28 pad 1: /poti_arr/ES03 -> /mux/ES03
- R3 pad 2: /LED/SW20 -> /LED/SW29
- R31 pad 1: POT_H -> MEA03
- R32 pad 1: /poti_arr/EB03 -> /mux/EB03
- R33 pad 1: /poti_arr/ES23 -> /mux/ES23
- R36 pad 1: POT_H -> MEA23
- R37 pad 1: /poti_arr/EB23 -> /mux/EB23
- R38 pad 2: /LED/SW34 -> /LED/SW35
- R39 pad 2: /LED/SW55 -> /LED/SW54
- R4 pad 2: /LED/SW30 -> /LED/SW39
- R40 pad 1: /poti_arr/ES01 -> /mux/ES01
- R43 pad 1: POT_H -> MEA01
- R44 pad 1: /poti_arr/EB01 -> /mux/EB01
- R45 pad 2: /LED/SW44 -> /LED/SW45
- R46 pad 2: /LED/SW54 -> /LED/SW55
- R47 pad 1: /poti_arr/ES14 -> /mux/ES14
- R5 pad 2: /LED/SW40 -> /LED/SW49
- R50 pad 1: POT_H -> MEA14
- R51 pad 1: /poti_arr/EB14 -> /mux/EB14
- R52 pad 2: /LED/SW37 -> /LED/SW32
- R53 pad 2: /LED/SW47 -> /LED/SW42
- R54 pad 2: /LED/SW57 -> /LED/SW52
- R55 pad 1: /poti_arr/ES07 -> /mux/ES07
- R58 pad 1: POT_H -> MEA07
- R59 pad 1: /poti_arr/EB07 -> /mux/EB07
- R6 pad 2: /LED/SW50 -> /LED/SW59
- R60 pad 2: /LED/SW36 -> /LED/SW33
- R61 pad 2: /LED/SW46 -> /LED/SW43
- R62 pad 2: /LED/SW56 -> /LED/SW53
- R63 pad 1: /poti_arr/ES27 -> /mux/ES27
- R66 pad 1: POT_H -> MEA27
- R67 pad 1: /poti_arr/EB27 -> /mux/EB27
- R68 pad 2: /LED/SW39 -> /LED/SW30
- R69 pad 2: /LED/SW49 -> /LED/SW40
- R7 pad 1: /poti_arr/ES21 -> /mux/ES21
- R70 pad 2: /LED/SW59 -> /LED/SW50
- R71 pad 2: /LED/SW29 -> /LED/SW20
- R72 pad 1: /poti_arr/ES16 -> /mux/ES16
- R75 pad 1: POT_H -> MEA16
- R76 pad 1: /poti_arr/EB16 -> /mux/EB16
- R77 pad 2: /LED/SW38 -> /LED/SW31
- R78 pad 2: /LED/SW48 -> /LED/SW41
- R79 pad 2: /LED/SW58 -> /LED/SW51
- R80 pad 2: /LED/SW21 -> /LED/SW28
- R81 pad 2: /LED/SW22 -> /LED/SW27
- R82 pad 2: /LED/SW23 -> /LED/SW26
- R83 pad 2: /LED/SW24 -> /LED/SW25
- R84 pad 2: /LED/SW09 -> /LED/SW00
- R85 pad 2: /LED/SW25 -> /LED/SW24
- R86 pad 2: /LED/SW19 -> /LED/SW10
- R87 pad 2: /LED/SW26 -> /LED/SW23
- R88 pad 1: /poti_arr/ES05 -> /mux/ES05
- R89 pad 2: /LED/SW27 -> /LED/SW22
- R92 pad 1: POT_H -> MEA05
- R93 pad 1: /poti_arr/EB05 -> /mux/EB05
- R94 pad 1: /poti_arr/ES25 -> /mux/ES25
- R95 pad 2: /led_driver/in -> led_dat
- R97 pad 2: /led_driver/in -> led_dat
- R99 pad 1: /led_driver/in -> led_dat
- R99 pad 2: /led_driver/in -> led_dat
- U1 pad S2: /poti_arr/ES21 -> /mux/ES21
- U12 pad S1: POT_H -> MEA03
- U13 pad S2: /poti_arr/ES23 -> /mux/ES23
- U16 pad S1: POT_H -> MEA23
- U17 pad S2: /poti_arr/ES01 -> /mux/ES01
- U20 pad S1: POT_H -> MEA01
- U21 pad S2: /poti_arr/ES14 -> /mux/ES14
- U24 pad S1: POT_H -> MEA14
- U25 pad S2: /poti_arr/ES07 -> /mux/ES07
- U28 pad S1: POT_H -> MEA07
- U29 pad S2: /poti_arr/ES27 -> /mux/ES27
- U32 pad S1: POT_H -> MEA27
- U33 pad S2: /poti_arr/ES16 -> /mux/ES16
- U36 pad S1: POT_H -> MEA16
- U37 pad S2: /poti_arr/ES05 -> /mux/ES05
- U4 pad S1: POT_H -> MEA21
- U40 pad S1: POT_H -> MEA05
- U41 pad S2: /poti_arr/ES25 -> /mux/ES25
- U42 pad 3: /led_driver/in -> led_dat
- U42 pad 4: /led_driver/in -> led_dat
- U43 pad 1: /mux/A4 -> /LED/SW27
- U43 pad 10: /mux/S1 -> MS1
- U43 pad 11: /mux/S0 -> MS0
- U43 pad 12: /mux/A3 -> /LED/SW56
- U43 pad 13: /mux/A0 -> /LED/SW46
- U43 pad 14: /mux/A1 -> /LED/SW36
- U43 pad 15: /mux/A2 -> /LED/SW26
- U43 pad 2: /mux/A6 -> /LED/SW37
- U43 pad 3: /mux/A -> MAA67
- U43 pad 4: /mux/A7 -> /LED/SW47
- U43 pad 5: /mux/A5 -> /LED/SW57
- U43 pad 9: /mux/S2 -> MS2
- U46 pad S1: POT_H -> MEA25
- U47 pad 1: /mux/A4 -> /LED/SW23
- U47 pad 10: /mux/S1 -> MS1
- U47 pad 11: /mux/S0 -> MS0
- U47 pad 12: /mux/A3 -> /LED/SW52
- U47 pad 13: /mux/A0 -> /LED/SW42
- U47 pad 14: /mux/A1 -> /LED/SW32
- U47 pad 15: /mux/A2 -> /LED/SW22
- U47 pad 2: /mux/A6 -> /LED/SW33
- U47 pad 3: /mux/A -> MAA23
- U47 pad 4: /mux/A7 -> /LED/SW43
- U47 pad 5: /mux/A5 -> /LED/SW53
- U47 pad 9: /mux/S2 -> MS2
- U48 pad 1: /mux/A4 -> /LED/SW21
- U48 pad 10: /mux/S1 -> MS1
- U48 pad 11: /mux/S0 -> MS0
- U48 pad 12: /mux/A3 -> /LED/SW50
- U48 pad 13: /mux/A0 -> /LED/SW40
- U48 pad 14: /mux/A1 -> /LED/SW30
- U48 pad 15: /mux/A2 -> /LED/SW20
- U48 pad 2: /mux/A6 -> /LED/SW31
- U48 pad 3: /mux/A -> MAA01
- U48 pad 4: /mux/A7 -> /LED/SW41
- U48 pad 5: /mux/A5 -> /LED/SW51
- U48 pad 9: /mux/S2 -> MS2
- U49 pad S2: /poti_arr/ES18 -> /mux/ES18
- U5 pad S2: /poti_arr/ES12 -> /mux/ES12
- U52 pad S1: POT_H -> MEA18
- U53 pad 1: /mux/A4 -> /LED/SW29
- U53 pad 10: /mux/S1 -> MS1
- U53 pad 11: /mux/S0 -> MS0
- U53 pad 12: /mux/A3 -> /LED/SW58
- U53 pad 13: /mux/A0 -> /LED/SW48
- U53 pad 14: /mux/A1 -> /LED/SW38
- U53 pad 15: /mux/A2 -> /LED/SW28
- U53 pad 2: /mux/A6 -> /LED/SW39
- U53 pad 3: /mux/A -> MAA89
- U53 pad 4: /mux/A7 -> /LED/SW49
- U53 pad 5: /mux/A5 -> /LED/SW59
- U53 pad 9: /mux/S2 -> MS2
- U54 pad 1: /mux/A4 -> /mux/EB05
- U54 pad 10: /mux/S1 -> MS1
- U54 pad 11: /mux/S0 -> MS0
- U54 pad 12: /mux/A3 -> /mux/EB25
- U54 pad 13: /mux/A0 -> /mux/ES25
- U54 pad 14: /mux/A1 -> /mux/EB14
- U54 pad 15: /mux/A2 -> /mux/ES14
- U54 pad 2: /mux/A6 -> /mux/ES05
- U54 pad 3: /mux/A -> MC
- U54 pad 4: /mux/A7 -> /mux/EB16
- U54 pad 5: /mux/A5 -> /mux/ES16
- U54 pad 9: /mux/S2 -> MS2
- U55 pad 1: /mux/A4 -> unconnected-(U55-A4-Pad1)
- U55 pad 10: /mux/S1 -> MS1
- U55 pad 11: /mux/S0 -> MS0
- U55 pad 12: /mux/A3 -> unconnected-(U55-A3-Pad12)
- U55 pad 13: /mux/A0 -> /mux/ES21
- U55 pad 14: /mux/A1 -> /LED/SW10
- U55 pad 15: /mux/A2 -> /LED/SW00
- U55 pad 2: /mux/A6 -> /mux/EB23
- U55 pad 3: /mux/A -> MA
- U55 pad 4: /mux/A7 -> /mux/ES23
- U55 pad 5: /mux/A5 -> /mux/EB21
- U55 pad 9: /mux/S2 -> MS2
- U56 pad 1: /mux/A4 -> /mux/EB18
- U56 pad 10: /mux/S1 -> MS1
- U56 pad 11: /mux/S0 -> MS0
- U56 pad 12: /mux/A3 -> /mux/EB27
- U56 pad 13: /mux/A0 -> /mux/ES27
- U56 pad 14: /mux/A1 -> /mux/EB07
- U56 pad 15: /mux/A2 -> /mux/ES07
- U56 pad 2: /mux/A6 -> /mux/ES18
- U56 pad 3: /mux/A -> MD
- U56 pad 4: /mux/A7 -> /LED/SW09
- U56 pad 5: /mux/A5 -> /LED/SW19
- U56 pad 9: /mux/S2 -> MS2
- U57 pad 1: /mux/A4 -> /LED/SW25
- U57 pad 10: /mux/S1 -> MS1
- U57 pad 11: /mux/S0 -> MS0
- U57 pad 12: /mux/A3 -> /LED/SW54
- U57 pad 13: /mux/A0 -> /LED/SW44
- U57 pad 14: /mux/A1 -> /LED/SW34
- U57 pad 15: /mux/A2 -> /LED/SW24
- U57 pad 2: /mux/A6 -> /LED/SW35
- U57 pad 3: /mux/A -> MAA45
- U57 pad 4: /mux/A7 -> /LED/SW45
- U57 pad 5: /mux/A5 -> /LED/SW55
- U57 pad 9: /mux/S2 -> MS2
- U59 pad 1: /mux/A4 -> /mux/ES03
- U59 pad 10: /mux/S1 -> MS1
- U59 pad 11: /mux/S0 -> MS0
- U59 pad 12: /mux/A3 -> unconnected-(U59-A3-Pad12)
- U59 pad 13: /mux/A0 -> unconnected-(U59-A0-Pad13)
- U59 pad 14: /mux/A1 -> /mux/EB01
- U59 pad 15: /mux/A2 -> /mux/ES01
- U59 pad 2: /mux/A6 -> /mux/EB03
- U59 pad 3: /mux/A -> MB
- U59 pad 4: /mux/A7 -> /mux/EB12
- U59 pad 5: /mux/A5 -> /mux/ES12
- U59 pad 9: /mux/S2 -> MS2
- U8 pad S1: POT_H -> MEA12
- U9 pad S2: /poti_arr/ES03 -> /mux/ES03
Routing:
- net GND: track 2156.5 -> 3495.3 mm, vias 1 -> 20
- net +3V3: track 1201.4 -> 1888.9 mm, vias 0 -> 27
- net MS2: track 0.00 -> 577.6 mm, vias 0 -> 17
- net MS1: track 0.00 -> 564.7 mm, vias 0 -> 17
- net MS0: track 0.00 -> 558.9 mm, vias 0 -> 16
- net +5V: track 1097.2 -> 1378.4 mm, vias 8 -> 15
- net MAA89: track 0.00 -> 247.4 mm, vias 0 -> 2
- net MAA01: track 0.00 -> 213.2 mm, vias 0 -> 2
- net MAA67: track 0.00 -> 202.5 mm, vias 0 -> 2
- net led_dat: track 0.00 -> 191.9 mm, vias 0 -> 3
- net MEA25: track 0.00 -> 185.1 mm
- net MEA23: track 0.00 -> 182.7 mm, vias 0 -> 2
- net MEA21: track 0.00 -> 174.9 mm
- net MAA23: track 0.00 -> 174.4 mm, vias 0 -> 2
- net MEA27: track 0.00 -> 173.7 mm
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- added copper zone on B.Cu, net GND
- added copper zone on F.Cu, net GND
Other:
- board size 488.6 x 432.7 mm -> 201.2 x 190.3 mm

Commit message: finished design
Parts:
- IC1: moved to B.Cu
Connections:
- IC1 pad 10: MEA07 -> MEA05
- IC1 pad 11: MC -> MEA14
- IC1 pad 12: MEA14 -> MC
- IC1 pad 13: MEA05 -> MEA07
- IC1 pad 15: MEA03 -> MD
- IC1 pad 16: MB -> MEA16
- IC1 pad 17: MEA23 -> MEA25
- IC1 pad 18: MEA21 -> MEA27
- IC1 pad 19: MEA12 -> MEA18
- IC1 pad 20: MEA01 -> led_dat
- IC1 pad 27: MA -> MAA67
- IC1 pad 28: MAA23 -> MAA89
- IC1 pad 29: MAA01 -> MS2
- IC1 pad 35: unconnected-(IC1-IO38/LED-Pad35) -> MS1
- IC1 pad 36: unconnected-(IC1-IO39-Pad36) -> MS0
- IC1 pad 38: unconnected-(IC1-IO41-Pad38) -> MAA01
- IC1 pad 39: MS0 -> MAA23
- IC1 pad 4: led_dat -> MEA01
- IC1 pad 40: MS1 -> MA
- IC1 pad 41: MS2 -> unconnected-(IC1-IO1/AD1_0-Pad41)
- IC1 pad 42: MAA89 -> unconnected-(IC1-IO44-Pad42)
- IC1 pad 43: MAA67 -> unconnected-(IC1-IO43-Pad43)
- IC1 pad 5: MEA18 -> MEA12
- IC1 pad 6: MEA27 -> MEA21
- IC1 pad 7: MEA25 -> MEA23
- IC1 pad 8: MEA16 -> MB
- IC1 pad 9: MD -> MEA03
Routing:
- net +3V3: track 1888.9 -> 2000.6 mm, vias 27 -> 30
- net GND: track 3495.3 -> 3519.9 mm, vias 20 -> 62
- net MS1: track 564.7 -> 543.4 mm
- net MAA89: track 247.4 -> 229.2 mm
- net MS0: track 558.9 -> 541.0 mm
- net MEA23: track 182.7 -> 169.9 mm, vias 2 -> 0
- net MAA45: track 158.4 -> 146.8 mm
- net MAA67: track 202.5 -> 191.2 mm
- net MS2: track 577.6 -> 568.6 mm
- net MAA01: track 213.2 -> 219.0 mm
- net /mux/ES05: track 55.9 -> 50.3 mm
- net MC: track 100.4 -> 106.0 mm
- net MAA23: track 174.4 -> 179.7 mm
- net MEA01: track 108.7 -> 111.8 mm
- net MEA18: track 119.3 -> 116.4 mm
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